File: HARDWARE/STM32XP/STM32XP.kicad_pcb (KiCad board)
At the start: 2 copper layers, 99.1 x 53.3 mm, 34 parts, among them J1 USB_C_Receptacle_USB2.0_16P, J2 Micro_SD_Card, J3 Conn_01x20_Socket, J4 Conn_01x20_Socket, J5 Jack-DC, J9 Conn_02x05_Odd_Even, SW1 SW_Push, SW2 SW_Push, SW3 RST, U1 STM32F411RETx, U2 ADS1115IDGS, U3 LM324, Y1 32.768kHz, Y2 8MHz xpF

Commit message: Continuing schematic design and preliminary placement of components.
Parts:
- added C12: 10uF 25V, Capacitor_SMD:C_0805_2012Metric_Pad1.18x1.45mm_HandSolder, F.Cu at (170.3, 91.1)
- added C13: 100nF 50V, Capacitor_SMD:C_0603_1608Metric_Pad1.08x0.95mm_HandSolder, F.Cu at (139.8, 101.9)
- added C14: 100nF 50V, Capacitor_SMD:C_0603_1608Metric_Pad1.08x0.95mm_HandSolder, F.Cu at (153.8, 109.5)
- added C15: 100nF 50V, Capacitor_SMD:C_0603_1608Metric_Pad1.08x0.95mm_HandSolder, F.Cu at (162.7, 91.1)
- added C16: 100nF 50V, Capacitor_SMD:C_0603_1608Metric_Pad1.08x0.95mm_HandSolder, F.Cu at (188.1, 94.3)
- added C17: 10uF 25V, Capacitor_SMD:C_0805_2012Metric_Pad1.18x1.45mm_HandSolder, F.Cu at (189.4, 121.0)
- added C18: 100nF 50V, Capacitor_SMD:C_0603_1608Metric_Pad1.08x0.95mm_HandSolder, F.Cu at (191.3, 121.0)
- added R10: 10K 1%, Resistor_SMD:R_0603_1608Metric_Pad0.98x0.95mm_HandSolder, F.Cu at (139.8, 100.0)
- added R11: 51R 1%, Resistor_SMD:R_0603_1608Metric_Pad0.98x0.95mm_HandSolder, F.Cu at (161.4, 81.0)
- added R12: 51R 1%, Resistor_SMD:R_0603_1608Metric_Pad0.98x0.95mm_HandSolder, F.Cu at (151.9, 88.6)
- added R13: 51R 1%, Resistor_SMD:R_0603_1608Metric_Pad0.98x0.95mm_HandSolder, F.Cu at (154.4, 88.6)
- added R14: 10K 1%, Resistor_SMD:R_0603_1608Metric_Pad0.98x0.95mm_HandSolder, F.Cu at (169.7, 115.2)
- added R15: 10K 1%, Resistor_SMD:R_0603_1608Metric_Pad0.98x0.95mm_HandSolder, F.Cu at (181.8, 115.2)
- added R16: 51R 1%, Resistor_SMD:R_0603_1608Metric_Pad0.98x0.95mm_HandSolder, F.Cu at (160.8, 101.3)
- added R17: 51R 1%, Resistor_SMD:R_0603_1608Metric_Pad0.98x0.95mm_HandSolder, F.Cu at (160.8, 103.2)
- added R18: 51R 1%, Resistor_SMD:R_0603_1608Metric_Pad0.98x0.95mm_HandSolder, F.Cu at (160.8, 107.0)
- added R19: 51R 1%, Resistor_SMD:R_0603_1608Metric_Pad0.98x0.95mm_HandSolder, F.Cu at (183.7, 109.5)
- added R20: 10K 1%, Resistor_SMD:R_0603_1608Metric_Pad0.98x0.95mm_HandSolder, F.Cu at (182.7, 103.8)
- added R21: 10K 1%, Resistor_SMD:R_0603_1608Metric_Pad0.98x0.95mm_HandSolder, F.Cu at (182.7, 106.3)
- added R3: 51R 1%, Resistor_SMD:R_0603_1608Metric_Pad0.98x0.95mm_HandSolder, F.Cu at (148.1, 88.6)
- added R4: 51R 1%, Resistor_SMD:R_0603_1608Metric_Pad0.98x0.95mm_HandSolder, F.Cu at (146.2, 88.6)
- added R5: 2.2K 1%, Resistor_SMD:R_0603_1608Metric_Pad0.98x0.95mm_HandSolder, F.Cu at (148.1, 84.8)
- added R6: 2.2K 1%, Resistor_SMD:R_0603_1608Metric_Pad0.98x0.95mm_HandSolder, F.Cu at (146.2, 84.8)
- added R7: 51R 1%, Resistor_SMD:R_0603_1608Metric_Pad0.98x0.95mm_HandSolder, F.Cu at (169.1, 81.0)
- added R8: 51R 1%, Resistor_SMD:R_0603_1608Metric_Pad0.98x0.95mm_HandSolder, F.Cu at (166.5, 81.0)
- added R9: 51R 1%, Resistor_SMD:R_0603_1608Metric_Pad0.98x0.95mm_HandSolder, F.Cu at (164.0, 81.0)
- added U4: AMS1117-3.3, Package_TO_SOT_SMD:SOT-223-3_TabPin2, F.Cu at (175.4, 91.1)
- added U5: USBLC6-2SC6, Package_TO_SOT_SMD:SOT-23-6, F.Cu at (188.2, 97.0)
- moved SW3 25.7 mm to (133.5, 102.5)
- moved SW2 12.5 mm to (181.8, 112.7)
- moved SW1 9.86 mm to (169.7, 112.7)
- moved Y1 3.58 mm to (138.6, 93.7)
- moved R1 2.06 mm to (150.0, 88.6)
- moved C5 1.94 mm to (140.1, 104.4)
- moved C6 1.94 mm to (137.0, 106.4)
- moved C7 1.94 mm to (137.0, 109.9)
- moved L1 1.94 mm to (140.1, 107.9)
- moved C2 1.63 mm to (158.3, 94.9)
- moved C3 1.57 mm to (155.1, 107.0), turned to 90 degrees
- moved C4 1.31 mm to (145.3, 108.5)
- moved C1 0.73 mm to (144.9, 92.4)
- moved C11 0.68 mm to (154.4, 111.4)
- turned D1 to 180 degrees
Connections:
- net Net-(J1-VBUS-PadA4) renamed VBUS
- D1 pad 1: unconnected-(D1-VDD-Pad1) -> +5V
- D1 pad 2: unconnected-(D1-DOUT-Pad2) -> NEOPIXEL DOUT
- D1 pad 3: unconnected-(D1-VSS-Pad3) -> GND
- D1 pad 4: unconnected-(D1-DIN-Pad4) -> NEOPIXEL DIN
- J1 pad A1: Net-(J1-GND-PadA1) -> GND
- J1 pad A12: Net-(J1-GND-PadA1) -> GND
- J1 pad A6: unconnected-(J1-D+-PadA6) -> Net-(J1-D+-PadA6)
- J1 pad A7: unconnected-(J1-D--PadA7) -> Net-(J1-D--PadA7)
- J1 pad B1: Net-(J1-GND-PadA1) -> GND
- J1 pad B12: Net-(J1-GND-PadA1) -> GND
- J1 pad B6: unconnected-(J1-D+-PadB6) -> Net-(J1-D+-PadA6)
- J1 pad B7: unconnected-(J1-D--PadB7) -> Net-(J1-D--PadA7)
- J2 pad 1: unconnected-(J2-DAT2-Pad1) -> Net-(J2-DAT2)
- J2 pad 2: unconnected-(J2-DAT3/CD-Pad2) -> SPI NSS
- J2 pad 3: unconnected-(J2-CMD-Pad3) -> SPI MOSI
- J2 pad 4: unconnected-(J2-VDD-Pad4) -> +3.3V
- J2 pad 5: unconnected-(J2-CLK-Pad5) -> SPI SCK
- J2 pad 6: unconnected-(J2-VSS-Pad6) -> GND
- J2 pad 7: unconnected-(J2-DAT0-Pad7) -> Net-(J2-DAT0)
- J2 pad 8: unconnected-(J2-DAT1-Pad8) -> Net-(J2-DAT1)
- J3 pad 10: unconnected-(J3-Pin_10-Pad10) -> AIN7
- J3 pad 3: unconnected-(J3-Pin_3-Pad3) -> AIN0
- J3 pad 4: unconnected-(J3-Pin_4-Pad4) -> AIN1
- J3 pad 5: unconnected-(J3-Pin_5-Pad5) -> AIN2
- J3 pad 6: unconnected-(J3-Pin_6-Pad6) -> AIN3
- J3 pad 7: unconnected-(J3-Pin_7-Pad7) -> AIN4
- J3 pad 8: unconnected-(J3-Pin_8-Pad8) -> AIN5
- J3 pad 9: unconnected-(J3-Pin_9-Pad9) -> AIN6
- J4 pad 1: unconnected-(J4-Pin_1-Pad1) -> +3.3V
- J4 pad 10: unconnected-(J4-Pin_10-Pad10) -> I2C SDA
- J4 pad 2: unconnected-(J4-Pin_2-Pad2) -> GND
- J4 pad 3: unconnected-(J4-Pin_3-Pad3) -> Net-(J4-Pin_3)
- J4 pad 4: unconnected-(J4-Pin_4-Pad4) -> Net-(J4-Pin_4)
- J4 pad 5: unconnected-(J4-Pin_5-Pad5) -> Net-(J4-Pin_5)
- J4 pad 6: unconnected-(J4-Pin_6-Pad6) -> Net-(J4-Pin_6)
- J4 pad 7: unconnected-(J4-Pin_7-Pad7) -> DEBUG TX
- J4 pad 8: unconnected-(J4-Pin_8-Pad8) -> DEBUG RX
- J4 pad 9: unconnected-(J4-Pin_9-Pad9) -> I2C SCL
- R1 pad 1: unconnected-(R1-Pad1) -> GND
- SW1 pad 1: unconnected-(SW1-Pad1) -> GND
- SW1 pad 2: unconnected-(SW1-Pad2) -> BUTTON 1
- SW2 pad 1: unconnected-(SW2-Pad1) -> GND
- SW2 pad 2: unconnected-(SW2-Pad2) -> BUTTON 2
- SW3 pad 1: unconnected-(SW3-Pad1) -> GND
- SW3 pad 2: unconnected-(SW3-Pad2) -> NRST
- U1 pad 14: unconnected-(U1-PA0-Pad14) -> AIN0
- U1 pad 15: unconnected-(U1-PA1-Pad15) -> AIN1
- U1 pad 16: unconnected-(U1-PA2-Pad16) -> AIN2
- U1 pad 17: unconnected-(U1-PA3-Pad17) -> AIN3
- U1 pad 20: unconnected-(U1-PA4-Pad20) -> AIN4
- U1 pad 21: unconnected-(U1-PA5-Pad21) -> AIN5
- U1 pad 22: unconnected-(U1-PA6-Pad22) -> AIN6
- U1 pad 23: unconnected-(U1-PA7-Pad23) -> AIN7
- U1 pad 24: unconnected-(U1-PC4-Pad24) -> BUTTON LEFT
- U1 pad 25: unconnected-(U1-PC5-Pad25) -> BUTTON RIGHT
- U1 pad 26: unconnected-(U1-PB0-Pad26) -> BUTTON UP
- U1 pad 27: unconnected-(U1-PB1-Pad27) -> BUTTON DOWN
- U1 pad 28: unconnected-(U1-PB2-Pad28) -> BUTTON CENTER
- U1 pad 33: unconnected-(U1-PB12-Pad33) -> Net-(U1-PB12)
- U1 pad 34: unconnected-(U1-PB13-Pad34) -> SPI MISO
- U1 pad 35: unconnected-(U1-PB14-Pad35) -> Net-(U1-PB14)
- U1 pad 36: unconnected-(U1-PB15-Pad36) -> Net-(U1-PB15)
- U1 pad 41: unconnected-(U1-PA8-Pad41) -> BUTTON 1
- U1 pad 42: unconnected-(U1-PA9-Pad42) -> BUTTON 2
- U1 pad 44: unconnected-(U1-PA11-Pad44) -> USB D-
- U1 pad 45: unconnected-(U1-PA12-Pad45) -> USB D+
- U1 pad 46: unconnected-(U1-PA13-Pad46) -> SWDIO
- U1 pad 49: unconnected-(U1-PA14-Pad49) -> SWCLK
- U1 pad 50: unconnected-(U1-PA15-Pad50) -> Net-(U1-PA15)
- U1 pad 55: unconnected-(U1-PB3-Pad55) -> SWO
- U1 pad 58: unconnected-(U1-PB6-Pad58) -> Net-(U1-PB6)
- U1 pad 59: unconnected-(U1-PB7-Pad59) -> DEBUG RX
- U1 pad 61: unconnected-(U1-PB8-Pad61) -> /MCU PB8
- U1 pad 62: unconnected-(U1-PB9-Pad62) -> /MCU PB9
- U1 pad 7: unconnected-(U1-NRST-Pad7) -> NRST
- U2 pad 10: unconnected-(U2-SCL-Pad10) -> I2C SCL
- U2 pad 3: unconnected-(U2-GND-Pad3) -> GND
- U2 pad 8: unconnected-(U2-VDD-Pad8) -> +3.3V
- U2 pad 9: unconnected-(U2-SDA-Pad9) -> I2C SDA

Commit message: Added libraries for custom components. Added OLED display. Started draft of routing.
Parts:
- added L2: CMF3216F-900-2P-T, Inductor_SMD:L_CommonModeChoke_TDK_ACM2520-2P, F.Cu at (183.7, 95.9)
- added U6: OLED 128x64 1.3", STM32XP:OLED 128x64 1.3in, F.Cu at (150.0, 87.3)
- moved SW3 33.1 mm to (158.9, 81.3), turned to -90 degrees
- moved D1 19.1 mm to (177.0, 100.0)
- moved C15 18.9 mm to (177.0, 103.5)
- moved R21 10.2 mm to (183.7, 116.5), turned to 180 degrees
- moved R6 6.99 mm to (150.6, 90.2), turned to -90 degrees
- moved R5 5.84 mm to (145.9, 90.2), turned to -90 degrees
- moved U4 4.96 mm to (171.6, 87.9)
- moved C10 4.18 mm to (137.3, 96.5), turned to -90 degrees
- moved R1 3.84 mm to (153.5, 90.2)
- moved C9 3.83 mm to (137.3, 100.0), turned to 90 degrees
- moved R12 3.55 mm to (155.1, 90.2)
- moved R13 2.73 mm to (156.7, 90.2)
- moved R14 2.56 mm to (172.2, 114.9), turned to 0 degrees
- moved C12 2.54 mm to (170.3, 93.7), turned to 0 degrees
- moved SW1 2.54 mm to (172.2, 112.7), turned to 180 degrees
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Connections:
- net Net-(J2-DAT0) renamed /SD DAT0 SPI
- net Net-(J2-DAT1) renamed /SD DAT1 SPI
- net Net-(J2-DAT2) renamed /SD DAT2 SPI
- net Net-(U1-PA15) renamed /MCU PA15
- net Net-(U1-PB12) renamed /MCU PB12 SPI
- net Net-(U1-PB14) renamed /MCU PB14 SPI
- net Net-(U1-PB15) renamed /MCU PB15 SPI
- C16 pad 1: GND -> VBUS
- C16 pad 2: VBUS -> GND
- J3 pad 2: unconnected-(J3-Pin_2-Pad2) -> GND
- J4 pad 10: I2C SDA -> I2C SCL
- J4 pad 9: I2C SCL -> I2C SDA
- J5 pad 1: unconnected-(J5-Pad1) -> +VEXT
- J5 pad 2: unconnected-(J5-Pad2) -> GND
- R7 pad 1: SWCLK -> SWDIO
- R8 pad 1: SWDIO -> SWCLK
- U1 pad 43: unconnected-(U1-PA10-Pad43) -> USB OTG ID
- U5 pad 1: Net-(J1-D+-PadA6) -> Net-(L2-Pad4)
- U5 pad 3: Net-(J1-D--PadA7) -> Net-(L2-Pad3)
- U5 pad 4: Net-(L2-Pad4) -> Net-(J1-D--PadA7)
- U5 pad 6: Net-(L2-Pad3) -> Net-(J1-D+-PadA6)
Routing:
- net SPI SCK: track 0.00 -> 38.9 mm
- net SPI NSS: track 0.00 -> 38.2 mm
- net SPI MOSI: track 0.00 -> 38.0 mm, vias 0 -> 2
- net NRST: track 0.00 -> 35.8 mm, vias 0 -> 2
- net BUTTON 2: track 0.00 -> 32.8 mm, vias 0 -> 2
- net GND: track 0.00 -> 31.7 mm, vias 0 -> 1
- net +3.3V: track 0.00 -> 30.1 mm, vias 0 -> 2
- net SPI MISO: track 0.00 -> 29.7 mm
- net USB D-: track 0.00 -> 28.2 mm
- net USB D+: track 0.00 -> 27.9 mm
- net NEOPIXEL DIN: track 0.00 -> 25.5 mm, vias 0 -> 2
- net BUTTON 1: track 0.00 -> 23.6 mm, vias 0 -> 2
- net SWDIO: track 0.00 -> 22.4 mm
- net DEBUG RX: track 0.00 -> 21.6 mm, vias 0 -> 2
- net SWO: track 0.00 -> 21.6 mm, vias 0 -> 2
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