File: HARDWARE/STM32XP/STM32XP.kicad_sch (KiCad schematic)
At the start: 35 parts, among them J1 USB_C_Receptacle_USB2.0_16P, J2 Micro_SD_Card, J3 Conn_01x20_Socket, J4 Conn_01x20_Socket, J5 Jack-DC, J9 Conn_02x05_Odd_Even, SW1 SW_Push, SW2 SW_Push, SW3 RST, U1 STM32F411RETx, U2 ADS1115IDGS, U3 LM324, U4 AMS1117-3.3, Y1 32.768kHz, Y2 8MHz xpF

Commit message: Continuing schematic design and preliminary placement of components.
Parts:
- added C12, C17: 10uF 25V, Capacitor_SMD:C_0805_2012Metric_Pad1.18x1.45mm_HandSolder, symbol Device:C_Small
- added C13, C14, C15, C16, C18: 100nF 50V, Capacitor_SMD:C_0603_1608Metric_Pad1.08x0.95mm_HandSolder, symbol Device:C_Small
- added L2: CMF3216F-900-2P-T, PhilsLab_Footprints_KiCad6:CMC-1206, symbol Device:EMI_Filter_LL_1423
- added R10, R14, R15, R20, R21: 10K 1%, Resistor_SMD:R_0603_1608Metric_Pad0.98x0.95mm_HandSolder, symbol Device:R_US
- added R11, R12, R13, R16, R17, R18, R19, R3, R4, R7, R8, R9: 51R 1%, Resistor_SMD:R_0603_1608Metric_Pad0.98x0.95mm_HandSolder, symbol Device:R_US
- added R5, R6: 2.2K 1%, Resistor_SMD:R_0603_1608Metric_Pad0.98x0.95mm_HandSolder, symbol Device:R_US
- added U5: USBLC6-2SC6, Package_TO_SOT_SMD:SOT-23-6, symbol Power_Protection:USBLC6-2SC6
Connections:
- net +3.3V: now also J2.4 (VDD), J4.1 (Pin_1), U2.8 (VDD), U4.2 (VO), C12.2, C17.2, C18.2, R10.2, R14.2, R15.2, R20.2, R21.2, R5.2, R6.2
- net GND: now also D1.3 (VSS), J1.A1 (GND), J1.A12 (GND), J1.B1 (GND), J1.B12 (GND), J2.6 (VSS), J4.2 (Pin_2), R1.1, SW1.1, SW2.1, SW3.1, U2.3 (GND), U4.1 (GND), C12.1, C13.1, C14.1, C15.1, C16.1, C17.1, C18.1, U5.2 (GND)
- net VCORE: now also C14.2
- net I2C SCL: now reaches U2.10 (SCL)
- net I2C SCL: now also J4.9 (Pin_9), R3.2, R5.1
- net I2C SDA: now reaches U2.9 (SDA)
- net I2C SDA: now also J4.10 (Pin_10), R4.2, R6.1
- net BUTTON 2: now reaches SW2.2
- net BUTTON 2: now also U1.42 (PA9), R15.1
- net at J2.1 (DAT2): now also R20.1
- net SPI NSS: now reaches J2.2 (DAT3/CD)
- net SPI NSS: now also R16.2
- net SPI MOSI: now reaches J2.3 (CMD)
- net SPI MOSI: now also R18.2
- net SPI SCK: now reaches J2.5 (CLK)
- net SPI SCK: now also R17.2
- net at J2.7 (DAT0): now also R19.2
- net at J2.8 (DAT1): now also R21.1
- net NRST: now reaches SW3.2
- net NRST: now also U1.7 (NRST), C13.2, R10.1, R11.1
- net VBUS: now reaches J1.A4 (VBUS), J1.A9 (VBUS), J1.B4 (VBUS), J1.B9 (VBUS)
- net VBUS: now also C16.2, U5.5 (VBUS)
- net at J1.A6 (D+): now also J1.B6 (D+), U5.1 (I/O1)
- net at J1.A7 (D-): now also J1.B7 (D-), U5.3 (I/O2)
- net AIN7: now reaches J3.10 (Pin_10)
- net AIN7: now also U1.23 (PA7)
- net AIN0: now reaches J3.3 (Pin_3)
- net AIN0: now also U1.14 (PA0)
- net AIN1: now reaches J3.4 (Pin_4)
- net AIN1: now also U1.15 (PA1)
- net AIN2: now reaches J3.5 (Pin_5)
- net AIN2: now also U1.16 (PA2)
- net AIN3: now reaches J3.6 (Pin_6)
- net AIN3: now also U1.17 (PA3)
- net AIN4: now reaches J3.7 (Pin_7)
- net AIN4: now also U1.20 (PA4)
- net AIN5: now reaches J3.8 (Pin_8)
- net AIN5: now also U1.21 (PA5)
- net AIN6: now reaches J3.9 (Pin_9)
- net AIN6: now also U1.22 (PA6)
- net BUTTON LEFT: now reaches U1.24 (PC4)
- net BUTTON RIGHT: now reaches U1.25 (PC5)
- net BUTTON UP: now reaches U1.26 (PB0)
- net BUTTON DOWN: now reaches U1.27 (PB1)
- net BUTTON CENTER: now reaches U1.28 (PB2)
- net at U1.33 (PB12): now also R18.1
- net SPI MISO: now reaches U1.34 (PB13)
- net SPI MISO: now also R19.1
- net at U1.35 (PB14): now also R17.1
- net at U1.36 (PB15): now also R16.1
- net BUTTON 1: now reaches U1.41 (PA8)
- net BUTTON 1: now also SW1.2, R14.1
- net USB D-: now reaches U1.44 (PA11)
- net USB D-: now also L2.1
- net USB D+: now reaches U1.45 (PA12)
- net USB D+: now also L2.2
- net SWDIO: now reaches U1.46 (PA13)
- net SWDIO: now also R8.1
- net SWCLK: now reaches U1.49 (PA14)
- net SWCLK: now also R7.1
- net at U1.50 (PA15): now also R13.1
- net SWO: now reaches U1.55 (PB3)
- net SWO: now also R9.1
- net at U1.58 (PB6): now also R12.1
- net DEBUG RX: now reaches U1.59 (PB7)
- net DEBUG RX: now also J4.8 (Pin_8)
- net MCU PB8: now reaches U1.61 (PB8)
- net MCU PB8: now also R3.1
- net MCU PB9: now reaches U1.62 (PB9)
- net MCU PB9: now also R4.1
- net at J4.3 (Pin_3): now also R7.2
- net at J4.4 (Pin_4): now also R8.2
- net at J4.5 (Pin_5): now also R9.2
- net at J4.6 (Pin_6): now also R11.2
- net DEBUG TX: now reaches J4.7 (Pin_7)
- net DEBUG TX: now also R12.2
- net +5V: now reaches D1.1 (VDD)
- net +5V: now also C15.2
- net NEOPIXEL DOUT: now reaches D1.2 (DOUT)
- net NEOPIXEL DIN: now reaches D1.4 (DIN)
- net NEOPIXEL DIN: now also R13.2
- new net: L2.4, U5.4 (I/O2)
- new net: L2.3, U5.6 (I/O1)
Other:
- moved on the sheet: C10, C11, C9, J1, J2, J3, J4, J5, SW1, SW2, SW3, Y2

Commit message: Added libraries for custom components. Added OLED display. Started draft of routing.
Parts:
- added U6: OLED 128x64 1.3", STM32XP:OLED 128x64 1.3in, symbol STM32XP:OLED_128x64
- L2: footprint PhilsLab_Footprints_KiCad6:CMC-1206 -> Inductor_SMD:L_CommonModeChoke_TDK_ACM2520-2P
Connections:
- net +3.3V: now also U6.2 (VCC)
- net GND: now also C16.2, J3.2 (Pin_2), J5.2, U6.1 (GND); no longer C16.1
- net I2C SCL: now also J4.10 (Pin_10), U6.3 (SCL); no longer J4.9 (Pin_9)
- net I2C SDA: now also J4.9 (Pin_9), U6.4 (SDA); no longer J4.10 (Pin_10)
- net SWCLK: now also R8.1; no longer R7.1
- net SWDIO: now also R7.1; no longer R8.1
- net USB D+: now also L2.1; no longer L2.2
- net USB D-: now also L2.2; no longer L2.1
- net VBUS: now also C16.1; no longer C16.2
- net SD DAT2 SPI: now reaches J2.1 (DAT2), R20.1
- net SD DAT0 SPI: now reaches J2.7 (DAT0), R19.2
- net +VEXT: now reaches J5.1
- net SD DAT1 SPI: now reaches J2.8 (DAT1), R21.1
- net at J1.A6 (D+), J1.B6 (D+): now also U5.6 (I/O1); no longer U5.1 (I/O1)
- net at J1.A7 (D-), J1.B7 (D-): now also U5.4 (I/O2); no longer U5.3 (I/O2)
- net MCU PB15 SPI: now reaches R16.1, U1.36 (PB15)
- net at L2.4: now also U5.1 (I/O1); no longer U5.4 (I/O2)
- net at L2.3: now also U5.3 (I/O2); no longer U5.6 (I/O1)
- net MCU PA15: now reaches R13.1, U1.50 (PA15)
- net MCU PB12 SPI: now reaches R18.1, U1.33 (PB12)
- net MCU PB14 SPI: now reaches R17.1, U1.35 (PB14)
- net USB OTG ID: now reaches U1.43 (PA10)
Other:
- note added: "BUCK-BOOST TI TPS63070 https://www.ti.com/lit/ds/symlink/tps63070.pdf?ts=1715008161102 4-WAY SWITCH https://jlcpcb.com/partdetail/ShouHan-7_7_5_6P_LWX/C2858287"
- moved on the sheet: C11, C13, C14, C17, C18, L2, R1, R19, R2, R20, R21, SW3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
