File: HARDWARE/KICAD/STM32XP.kicad_pcb (KiCad board)
At the start: 2 copper layers, 99.1 x 53.3 mm, 64 parts, among them J1 USB_C_Receptacle_USB2.0_16P, J2 Micro_SD_Card, J3 Conn_01x20_Socket, J4 Conn_01x20_Socket, J5 Jack-DC, J9 Conn_02x05_Odd_Even, SW1 SW_Push, SW2 SW_Push, SW3 RST, U1 STM32F411RETx, U2 ADS1115IDGS, U3 LM324, U4 AMS1117-3.3, U5 USBLC6-2SC6, U6 OLED 128x64 1.3", Y1 32.768kHz, Y2 8MHz xpF

Commit message: Added logo and legend to board. Added OLED display libs to firmware.
Parts:
- added G***: LOGO, LOGO, F.Cu at (115.1, 84.1)
Other:
- board text added: "STM32 EXPLORER BOARD Mechatronix Lab Rev.00 2024.05.10"

Commit message: Added RGBfunctionality. Corrected SPI connections on schematic and layout.
Parts:
- moved R17 0.64 mm to (159.2, 103.8)
- moved R18 0.32 mm to (159.2, 105.4)
Connections:
- R16 pad 2: SPI NSS -> SPI MOSI
- R17 pad 1: /MCU PB14 SPI -> /MCU PB13 SPI
- R18 pad 2: SPI MOSI -> SPI NSS
- U1 pad 34: SPI MISO -> /MCU PB13 SPI
- U1 pad 35: /MCU PB14 SPI -> SPI MISO
Routing:
- net /MCU PB13 SPI: track 0.00 -> 2.81 mm
- net /MCU PB14 SPI: track 2.80 -> 0.00 mm
- net SPI MISO: track 29.7 -> 31.4 mm
- net SPI NSS: track 38.2 -> 36.7 mm, vias 0 -> 2
- net SPI MOSI: track 38.0 -> 38.7 mm, vias 2 -> 0
- net BUTTON 1: track 23.6 -> 24.2 mm
- net BUTTON 2: track 32.8 -> 32.3 mm

Commit message: Added AFE circuit.
Parts:
- added C19: 100nF 50V, Capacitor_SMD:C_0603_1608Metric_Pad1.08x0.95mm_HandSolder, F.Cu at (115.8, 94.3)
- added C20: 100nF 50V, Capacitor_SMD:C_0603_1608Metric_Pad1.08x0.95mm_HandSolder, F.Cu at (118.2, 95.0)
- added C21: 100nF 50V, Capacitor_SMD:C_0603_1608Metric_Pad1.08x0.95mm_HandSolder, F.Cu at (111.6, 94.9)
- added C22: 100nF 50V, Capacitor_SMD:C_0603_1608Metric_Pad1.08x0.95mm_HandSolder, F.Cu at (114.2, 94.3)
- added C23: 100nF 50V, Capacitor_SMD:C_0603_1608Metric_Pad1.08x0.95mm_HandSolder, F.Cu at (111.6, 104.8)
- added C24: 100nF 50V, Capacitor_SMD:C_0603_1608Metric_Pad1.08x0.95mm_HandSolder, F.Cu at (114.1, 105.7)
- added C25: 100nF 50V, Capacitor_SMD:C_0603_1608Metric_Pad1.08x0.95mm_HandSolder, F.Cu at (118.6, 104.8)
- added C26: 100nF 50V, Capacitor_SMD:C_0603_1608Metric_Pad1.08x0.95mm_HandSolder, F.Cu at (116.0, 105.7)
- added C27: 100nF 50V, Capacitor_SMD:C_0603_1608Metric_Pad1.08x0.95mm_HandSolder, F.Cu at (124.6, 104.8)
- added C28: 10uF 25V, Capacitor_SMD:C_0805_2012Metric_Pad1.18x1.45mm_HandSolder, F.Cu at (127.5, 100.0)
- added C29: 10uF 25V, Capacitor_SMD:C_0805_2012Metric_Pad1.18x1.45mm_HandSolder, F.Cu at (120.6, 99.7)
- added C30: 100nF 50V, Capacitor_SMD:C_0603_1608Metric_Pad1.08x0.95mm_HandSolder, F.Cu at (118.6, 99.7)
- added R22: 10K 1%, Resistor_SMD:R_0603_1608Metric_Pad0.98x0.95mm_HandSolder, F.Cu at (118.2, 93.4)
- added R23: 10K 1%, Resistor_SMD:R_0603_1608Metric_Pad0.98x0.95mm_HandSolder, F.Cu at (118.3, 91.7)
- added R24: 10K 1%, Resistor_SMD:R_0603_1608Metric_Pad0.98x0.95mm_HandSolder, F.Cu at (111.6, 91.7)
- added R25: 10K 1%, Resistor_SMD:R_0603_1608Metric_Pad0.98x0.95mm_HandSolder, F.Cu at (111.6, 93.3)
- added R26: 10K 1%, Resistor_SMD:R_0603_1608Metric_Pad0.98x0.95mm_HandSolder, F.Cu at (111.6, 107.9)
- added R27: 10K 1%, Resistor_SMD:R_0603_1608Metric_Pad0.98x0.95mm_HandSolder, F.Cu at (111.6, 106.3)
- added R28: 10K 1%, Resistor_SMD:R_0603_1608Metric_Pad0.98x0.95mm_HandSolder, F.Cu at (118.6, 107.9)
- added R29: 10K 1%, Resistor_SMD:R_0603_1608Metric_Pad0.98x0.95mm_HandSolder, F.Cu at (118.6, 106.3)
- added R30: 10K 1%, Resistor_SMD:R_0603_1608Metric_Pad0.98x0.95mm_HandSolder, F.Cu at (123.0, 105.1)
- added R31: 10K 1%, Resistor_SMD:R_0603_1608Metric_Pad0.98x0.95mm_HandSolder, F.Cu at (121.4, 105.1)
- added R32: 10K 1%, Resistor_SMD:R_0603_1608Metric_Pad0.98x0.95mm_HandSolder, F.Cu at (123.4, 94.3)
- added R33: 10K 1%, Resistor_SMD:R_0603_1608Metric_Pad0.98x0.95mm_HandSolder, F.Cu at (125.0, 94.3)
- moved G*** 1.62 mm to (115.1, 82.5)
- turned U3 to -90 degrees
Connections:
- net AIN4 renamed PA4
- net AIN5 renamed PA5
- net AIN6 renamed PA6
- net AIN7 renamed PA7
- J3 pad 3: AIN0 -> PA0
- J3 pad 4: AIN1 -> PA1
- J3 pad 5: AIN2 -> PA2
- J3 pad 6: AIN3 -> PA3
- J9 pad 1: unconnected-(J9-Pin_1-Pad1) -> A0
- J9 pad 10: unconnected-(J9-Pin_10-Pad10) -> GND
- J9 pad 2: unconnected-(J9-Pin_2-Pad2) -> GND
- J9 pad 3: unconnected-(J9-Pin_3-Pad3) -> A1
- J9 pad 4: unconnected-(J9-Pin_4-Pad4) -> GND
- J9 pad 6: unconnected-(J9-Pin_6-Pad6) -> GND
- J9 pad 7: unconnected-(J9-Pin_7-Pad7) -> A2
- J9 pad 8: unconnected-(J9-Pin_8-Pad8) -> GND
- J9 pad 9: unconnected-(J9-Pin_9-Pad9) -> A3
- U1 pad 14: AIN0 -> PA0
- U1 pad 15: AIN1 -> PA1
- U1 pad 16: AIN2 -> PA2
- U1 pad 17: AIN3 -> PA3
- U2 pad 1: unconnected-(U2-ADDR-Pad1) -> GND
- U2 pad 4: unconnected-(U2-AIN0-Pad4) -> AIN0
- U2 pad 5: unconnected-(U2-AIN1-Pad5) -> AIN1
- U2 pad 6: unconnected-(U2-AIN2-Pad6) -> AIN2
- U2 pad 7: unconnected-(U2-AIN3-Pad7) -> AIN3
- U2 pad 8: +3.3V -> +5VA
- U3 pad 1: unconnected-(U3-Pad1) -> AIN0
- U3 pad 10: unconnected-(U3C-+-Pad10) -> Net-(U3C-+)
- U3 pad 11: unconnected-(U3E-V--Pad11) -> GND
- U3 pad 12: unconnected-(U3D-+-Pad12) -> Net-(U3D-+)
- U3 pad 13: unconnected-(U3D---Pad13) -> AIN3
- U3 pad 14: unconnected-(U3-Pad14) -> AIN3
- U3 pad 2: unconnected-(U3A---Pad2) -> AIN0
- U3 pad 3: unconnected-(U3A-+-Pad3) -> Net-(U3A-+)
- U3 pad 4: unconnected-(U3E-V+-Pad4) -> +5VA
- U3 pad 5: unconnected-(U3B-+-Pad5) -> Net-(U3B-+)
- U3 pad 6: unconnected-(U3B---Pad6) -> AIN1
- U3 pad 7: unconnected-(U3-Pad7) -> AIN1
- U3 pad 8: unconnected-(U3-Pad8) -> AIN2
- U3 pad 9: unconnected-(U3C---Pad9) -> AIN2
Routing:
- net PA1: track 0.00 -> 0.93 mm
- net AIN1: track 0.93 -> 0.00 mm

Commit message: Added PWM outputs from MCU; added directional buttons; added part of buzzer circuit.
Parts:
- added C31: 10uF 25V, Capacitor_SMD:C_0805_2012Metric_Pad1.18x1.45mm_HandSolder, F.Cu at (127.1, 93.0)
- added D2: ESDA6V1-5SC6, Package_TO_SOT_SMD:SOT-23-6, F.Cu at (108.1, 100.0)
- added Q1: MMBT3904, Package_TO_SOT_SMD:SOT-23, F.Cu at (177.6, 119.0)
- added R34: 10K 1%, Resistor_SMD:R_0603_1608Metric_Pad0.98x0.95mm_HandSolder, F.Cu at (123.0, 110.2)
- added R35: 10K 1%, Resistor_SMD:R_0603_1608Metric_Pad0.98x0.95mm_HandSolder, F.Cu at (123.0, 119.7)
- added R36: 10K 1%, Resistor_SMD:R_0603_1608Metric_Pad0.98x0.95mm_HandSolder, F.Cu at (118.2, 114.9)
- added R37: 10K 1%, Resistor_SMD:R_0603_1608Metric_Pad0.98x0.95mm_HandSolder, F.Cu at (127.8, 114.9)
- added R38: 10K 1%, Resistor_SMD:R_0603_1608Metric_Pad0.98x0.95mm_HandSolder, F.Cu at (123.0, 114.9)
- added SW4: SW_Push, Button_Switch_SMD:SW_SPST_CK_KXT3, F.Cu at (123.0, 107.9)
- added SW5: SW_Push, Button_Switch_SMD:SW_SPST_CK_KXT3, F.Cu at (123.0, 117.5)
- added SW6: SW_Push, Button_Switch_SMD:SW_SPST_CK_KXT3, F.Cu at (118.2, 112.7)
- added SW7: SW_Push, Button_Switch_SMD:SW_SPST_CK_KXT3, F.Cu at (127.8, 112.7)
- added SW8: SW_Push, Button_Switch_SMD:SW_SPST_CK_KXT3, F.Cu at (123.0, 112.7)
- added U7: AMS1117-5.0, Package_TO_SOT_SMD:SOT-223-3_TabPin2, F.Cu at (128.4, 87.3)
- R30, R31, R32, R33: value 10K 1% -> 51R 1%
- moved BT1 54.3 mm to (108.1, 46.7)
- moved R31 39.4 mm to (160.8, 103.8), turned to 180 degrees
- moved R32 38.3 mm to (160.8, 102.2), turned to 180 degrees
- moved R30 37.8 mm to (160.8, 105.4), turned to 180 degrees
- moved R33 36.4 mm to (160.8, 100.6), turned to 180 degrees
- moved C29 9.30 mm to (111.3, 100.0)
- moved R16 5.63 mm to (160.8, 107.0)
- moved R17 5.03 mm to (160.8, 108.6)
- moved R18 5.03 mm to (160.8, 110.2)
- moved C27 4.86 mm to (125.6, 100.0), turned to -90 degrees
- moved J9 2.54 mm to (104.3, 94.9)
- moved U2 1.59 mm to (123.0, 100.0)
- moved C12 0.64 mm to (170.3, 93.0)
- moved U4 0.64 mm to (171.6, 87.3)
- moved C4 0.55 mm to (145.9, 108.6)
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Connections:
- J9 pad 5: unconnected-(J9-Pin_5-Pad5) -> GND
- R30 pad 1: GND -> TIM3 CH1
- R30 pad 2: AIN3 -> Net-(U1-PC6)
- R31 pad 1: GND -> TIM3 CH2
- R31 pad 2: AIN2 -> Net-(U1-PC7)
- R32 pad 1: GND -> TIM3 CH3
- R32 pad 2: AIN1 -> Net-(U1-PC8)
- R33 pad 1: GND -> TIM3 CH4
- R33 pad 2: AIN0 -> Net-(U1-PC9)
- U1 pad 37: unconnected-(U1-PC6-Pad37) -> Net-(U1-PC6)
- U1 pad 38: unconnected-(U1-PC7-Pad38) -> Net-(U1-PC7)
- U1 pad 39: unconnected-(U1-PC8-Pad39) -> Net-(U1-PC8)
- U1 pad 40: unconnected-(U1-PC9-Pad40) -> Net-(U1-PC9)
- U4 pad 3: unconnected-(U4-VI-Pad3) -> +9V
Routing:
- net BUTTON LEFT: track 0.00 -> 39.6 mm, vias 0 -> 2
- net BUTTON DOWN: track 0.00 -> 39.2 mm, vias 0 -> 2
- net SPI SCK: track 38.7 -> 0.00 mm
- net SPI MOSI: track 38.7 -> 0.00 mm
- net SPI NSS: track 36.7 -> 0.00 mm, vias 2 -> 0
- net BUTTON CENTER: track 0.00 -> 36.2 mm, vias 0 -> 2
- net BUTTON UP: track 0.00 -> 34.5 mm, vias 0 -> 2
- net I2C SDA: track 18.0 -> 51.7 mm, vias 0 -> 2
- net SPI MISO: track 31.4 -> 0.00 mm
- net BUTTON RIGHT: track 0.00 -> 31.3 mm, vias 0 -> 2
- net I2C SCL: track 17.0 -> 47.6 mm, vias 0 -> 2
- net PA0: track 0.00 -> 26.5 mm
- net PA1: track 0.93 -> 24.8 mm
- net PA2: track 0.00 -> 23.1 mm
- net PA3: track 0.00 -> 20.9 mm
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
Commit message: Refactoring.
Parts:
- moved C28 7.30 mm to (120.2, 100.0)
- moved C30 6.70 mm to (115.1, 94.3), turned to -90 degrees
- moved BT1 6.25 mm to (110.6, 52.4), turned to 180 degrees
- moved C27 5.40 mm to (123.0, 104.8), turned to 90 degrees
- moved C11 0.95 mm to (154.8, 111.4)
- moved C14 0.95 mm to (154.8, 109.5)
- moved R24 0.67 mm to (110.9, 92.1)
- moved C20 0.64 mm to (119.2, 95.2)
- moved C22 0.64 mm to (113.5, 94.3)
- moved C24 0.64 mm to (113.5, 105.7)
- moved C25 0.64 mm to (119.2, 104.8)
- moved R22 0.64 mm to (119.2, 93.7)
- moved R23 0.64 mm to (119.2, 92.1)
- moved R28 0.64 mm to (119.2, 107.9)
- moved R29 0.64 mm to (119.2, 106.3)
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Routing:
- net SPI NSS: track 0.00 -> 37.8 mm, vias 0 -> 2
- net SPI SCK: track 0.00 -> 35.3 mm
- net SPI MOSI: track 0.00 -> 34.8 mm
- net SPI MISO: track 0.00 -> 34.2 mm
- net /MCU PB12 SPI: track 0.00 -> 8.70 mm
- net /MCU PB13 SPI: track 0.00 -> 8.09 mm
- net /MCU PB15 SPI: track 0.00 -> 7.26 mm
- net Net-(U1-PC6): track 0.00 -> 6.25 mm
- net Net-(U1-PC7): track 0.00 -> 5.27 mm
- net Net-(U1-PC8): track 0.00 -> 4.82 mm
- net Net-(U1-PC9): track 0.00 -> 4.37 mm
- net VCORE: track 9.70 -> 6.31 mm
- net A3: track 7.07 -> 7.71 mm
- net A0: track 7.07 -> 7.71 mm
- net GND: track 40.2 -> 40.8 mm

Commit message: Added sheets and organized schematic; added DC-DC Boost Converter; added connections to headers; general improvements on schematic and layout.
Parts:
- added C32: 100nF 50V, Capacitor_SMD:C_0603_1608Metric_Pad1.08x0.95mm_HandSolder, F.Cu at (147.5, 85.3)
- added C33: 100nF 50V, Capacitor_SMD:C_0603_1608Metric_Pad1.08x0.95mm_HandSolder, F.Cu at (131.5, 82.0)
- added C34: 10uF 25V, Capacitor_SMD:C_0805_2012Metric_Pad1.18x1.45mm_HandSolder, F.Cu at (181.2, 87.3)
- added C35: 10uF 25V, Capacitor_SMD:C_0805_2012Metric_Pad1.18x1.45mm_HandSolder, F.Cu at (181.2, 80.7)
- added C36: 10uF 25V, Capacitor_SMD:C_0805_2012Metric_Pad1.18x1.45mm_HandSolder, F.Cu at (124.6, 94.9)
- added C37: 10uF 25V, Capacitor_SMD:C_0805_2012Metric_Pad1.18x1.45mm_HandSolder, F.Cu at (130.7, 86.0)
- added C38: 10uF 25V, Capacitor_SMD:C_0805_2012Metric_Pad1.18x1.45mm_HandSolder, F.Cu at (175.4, 93.1)
- added D3: 1N5819WS, Diode_SMD:D_SOD-323, F.Cu at (184.3, 81.7)
- added D4: BAT54C, Package_TO_SOT_SMD:SOT-23, F.Cu at (184.3, 92.9)
- added JP1: 9V, Jumper:SolderJumper-2_P1.3mm_Open_RoundedPad1.0x1.5mm, F.Cu at (185.1, 77.9)
- added JP2: VSEL, Jumper:SolderJumper-2_P1.3mm_Open_RoundedPad1.0x1.5mm, F.Cu at (185.1, 89.3)
- added L3: L_Small, Inductor_SMD:L_0603_1608Metric_Pad1.05x0.95mm_HandSolder, F.Cu at (184.3, 85.3)
- added L4: L_Small, Inductor_SMD:L_0603_1608Metric_Pad1.05x0.95mm_HandSolder, F.Cu at (125.6, 92.4)
- added LS1: Speaker_Crystal, Buzzer_Beeper:MagneticBuzzer_PUI_AT-0927-TT-6-R, B.Cu at (178.1, 100.0)
- added Q2: 2N7002, Package_TO_SOT_SMD:SOT-23, F.Cu at (142.4, 85.8)
- added Q3: 2N7002, Package_TO_SOT_SMD:SOT-23, F.Cu at (142.4, 89.3)
- added R39: 1K 1%, Resistor_SMD:R_0603_1608Metric_Pad0.98x0.95mm_HandSolder, F.Cu at (176.2, 101.8)
- added R40: 10K 1%, Resistor_SMD:R_0603_1608Metric_Pad0.98x0.95mm_HandSolder, F.Cu at (127.4, 90.3)
- added R41: 10K 1%, Resistor_SMD:R_0603_1608Metric_Pad0.98x0.95mm_HandSolder, F.Cu at (128.9, 90.3)
- added R42: 6K2 1%, Resistor_SMD:R_0603_1608Metric_Pad0.98x0.95mm_HandSolder, F.Cu at (181.2, 78.9)
- added R43: 10K 1%, Resistor_SMD:R_0603_1608Metric_Pad0.98x0.95mm_HandSolder, F.Cu at (181.2, 77.4)
- added R44: 10K 1%, Resistor_SMD:R_0603_1608Metric_Pad0.98x0.95mm_HandSolder, F.Cu at (180.2, 89.1)
- added U8: AP3012, Package_TO_SOT_SMD:SOT-23-5, F.Cu at (180.2, 84.0)
- BT1: value Battery_Cell -> CR2032
- C15: value 100nF 50V -> 10uF 25V; footprint Capacitor_SMD:C_0603_1608Metric_Pad1.08x0.95mm_HandSolder -> Capacitor_SMD:C_0805_2012Metric_Pad1.18x1.45mm_HandSolder
- R30, R31, R32, R33: value 51R 1% -> 1K 1%
- moved D1 44.9 mm to (136.0, 81.7), turned to 0 degrees
- moved C15 35.7 mm to (147.5, 83.5)
- moved BT1 21.5 mm to (91.8, 62.9)
- moved Q1 20.1 mm to (171.1, 100.0)
- moved C31 4.17 mm to (124.6, 89.7)
- moved U7 4.17 mm to (125.9, 84.0)
- moved G*** 4.07 mm to (111.1, 81.5)
- moved C12 3.25 mm to (172.9, 91.0)
- moved U4 3.25 mm to (174.1, 85.3)
- moved L2 1.91 mm to (182.0, 96.8)
- moved R10 1.65 mm to (139.8, 102.3)
- moved C13 1.46 mm to (139.8, 100.8)
- moved C11 1.08 mm to (153.8, 110.9)
- moved C14 1.03 mm to (153.8, 109.1)
- moved J5 1.02 mm to (187.9, 86.0)
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Connections:
- net /MCU PA15 renamed /MCU/MCU PA15
- net /MCU PB12 SPI renamed /MCU/MCU PB12 SPI
- net /MCU PB13 SPI renamed /MCU/MCU PB13 SPI
- net /MCU PB15 SPI renamed /MCU/MCU PB15 SPI
- net /MCU PB8 renamed /MCU/MCU PB8
- net /MCU PB9 renamed /MCU/MCU PB9
- net /SD DAT0 SPI renamed /IO/SD DAT0 SPI
- net /SD DAT1 SPI renamed /IO/SD DAT1 SPI
- net /SD DAT2 SPI renamed /IO/SD DAT2 SPI
- net Net-(J1-D+-PadA6) renamed /IO/USB DATA+
- net Net-(J1-D--PadA7) renamed /IO/USB DATA-
- net Net-(L2-Pad3) renamed /IO/USB FILTERED D-
- net Net-(L2-Pad4) renamed /IO/USB FILTERED D+
- net Net-(U1-PC6) renamed /MCU/TIM3 CH1
- net Net-(U1-PC7) renamed /MCU/TIM3 CH2
- net Net-(U1-PC8) renamed /MCU/TIM3 CH3
- net Net-(U1-PC9) renamed /MCU/TIM3 CH4
- net VBUS renamed +VBUS
- C15 pad 2: +5V -> +3.3V
- C31 pad 2: +5VA -> +5V
- C6 pad 2: +3.3VA -> +3.3V
- C7 pad 2: +3.3V -> +3.3VA
- D2 pad 2: unconnected-(D2-GND-Pad2) -> GND
- D2 pad 4: unconnected-(D2-IO3-Pad4) -> A2
- D2 pad 5: unconnected-(D2-IO4-Pad5) -> GND
- D2 pad 6: unconnected-(D2-IO5-Pad6) -> A3
- J3 pad 1: unconnected-(J3-Pin_1-Pad1) -> PA0
- J3 pad 10: PA7 -> SPI MISO
- J3 pad 11: unconnected-(J3-Pin_11-Pad11) -> SPI MOSI
- J3 pad 12: unconnected-(J3-Pin_12-Pad12) -> SPI SCK
- J3 pad 13: unconnected-(J3-Pin_13-Pad13) -> SPI NSS
- J3 pad 14: unconnected-(J3-Pin_14-Pad14) -> PWM RED
- J3 pad 15: unconnected-(J3-Pin_15-Pad15) -> PWM GREEN
- J3 pad 16: unconnected-(J3-Pin_16-Pad16) -> PWM BLUE
- J3 pad 17: unconnected-(J3-Pin_17-Pad17) -> PWM BUZZER
- J3 pad 19: unconnected-(J3-Pin_19-Pad19) -> GND
- J3 pad 2: GND -> PA1
- J3 pad 20: unconnected-(J3-Pin_20-Pad20) -> +3.3V
- J3 pad 3: PA0 -> PA2
- J3 pad 4: PA1 -> PA3
- J3 pad 5: PA2 -> PA4
- J3 pad 6: PA3 -> PA5
- J3 pad 7: PA4 -> PA6
- J3 pad 8: PA5 -> PA7
- J3 pad 9: PA6 -> GND
- J4 pad 10: I2C SCL -> I2C SCL 3.3V
- J4 pad 11: unconnected-(J4-Pin_11-Pad11) -> PC3
- J4 pad 12: unconnected-(J4-Pin_12-Pad12) -> PC2
- J4 pad 13: unconnected-(J4-Pin_13-Pad13) -> PC1
- J4 pad 14: unconnected-(J4-Pin_14-Pad14) -> PC0
- J4 pad 15: unconnected-(J4-Pin_15-Pad15) -> GND
- J4 pad 16: unconnected-(J4-Pin_16-Pad16) -> I2C SDA 5V
- J4 pad 17: unconnected-(J4-Pin_17-Pad17) -> I2C SCL 5V
- J4 pad 18: unconnected-(J4-Pin_18-Pad18) -> NEOPIXEL DIN
- J4 pad 19: unconnected-(J4-Pin_19-Pad19) -> NEOPIXEL DOUT
- J4 pad 20: unconnected-(J4-Pin_20-Pad20) -> +5V
- J4 pad 9: I2C SDA -> I2C SDA 3.3V
- Q1 pad 1: unconnected-(Q1-B-Pad1) -> PWM BUZZER
- Q1 pad 2: unconnected-(Q1-E-Pad2) -> GND
- Q1 pad 3: unconnected-(Q1-C-Pad3) -> Net-(Q1-C)
- R3 pad 2: I2C SCL -> I2C SCL 3.3V
- R30 pad 1: TIM3 CH1 -> PWM RED
- R31 pad 1: TIM3 CH2 -> PWM GREEN
- R32 pad 1: TIM3 CH3 -> PWM BLUE
- R33 pad 1: TIM3 CH4 -> PWM BUZZER
- R4 pad 2: I2C SDA -> I2C SDA 3.3V
- R5 pad 1: I2C SCL -> I2C SCL 3.3V
- R6 pad 1: I2C SDA -> I2C SDA 3.3V
- U1 pad 10: unconnected-(U1-PC2-Pad10) -> PC2
- U1 pad 11: unconnected-(U1-PC3-Pad11) -> PC3
- U1 pad 8: unconnected-(U1-PC0-Pad8) -> PC0
- U1 pad 9: unconnected-(U1-PC1-Pad9) -> PC1
- U2 pad 10: I2C SCL -> I2C SCL 5V
- U2 pad 9: I2C SDA -> I2C SDA 5V
- U4 pad 3: +9V -> +VSEL
- U6 pad 3: I2C SCL -> I2C SCL 3.3V
- U6 pad 4: I2C SDA -> I2C SDA 3.3V
- U7 pad 2: +5VA -> +5V
Routing:
- net I2C SDA: track 51.7 -> 0.00 mm, vias 2 -> 0
- net I2C SCL: track 47.6 -> 0.00 mm, vias 2 -> 0
- net I2C SDA 5V: track 0.00 -> 34.3 mm, vias 0 -> 3
- net I2C SCL 5V: track 0.00 -> 34.3 mm, vias 0 -> 3
- net PC2: track 0.00 -> 30.9 mm, vias 0 -> 1
- net PC3: track 0.00 -> 29.6 mm, vias 0 -> 1
- net PWM BUZZER: track 0.00 -> 27.0 mm, vias 0 -> 2
- net PC1: track 0.00 -> 26.0 mm, vias 0 -> 1
- net NEOPIXEL DIN: track 25.5 -> 0.00 mm, vias 2 -> 0
- net PC0: track 0.00 -> 25.1 mm, vias 0 -> 1
- net PWM BLUE: track 0.00 -> 24.6 mm, vias 0 -> 1
- net I2C SDA 3.3V: track 0.00 -> 23.2 mm
- net I2C SCL 3.3V: track 0.00 -> 22.9 mm
- net PWM GREEN: track 0.00 -> 22.2 mm, vias 0 -> 1
- net PWM RED: track 0.00 -> 21.3 mm, vias 0 -> 1
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
Commit message: Continuing layout and routing.
Parts:
- added C39: 10uF 25V, Capacitor_SMD:C_0805_2012Metric_Pad1.18x1.45mm_HandSolder, F.Cu at (180.7, 93.1)
- added D5: LED, LED_SMD:LED_0603_1608Metric_Pad1.05x0.95mm_HandSolder, F.Cu at (186.8, 100.9)
- added D6: LED, LED_SMD:LED_0603_1608Metric_Pad1.05x0.95mm_HandSolder, F.Cu at (184.3, 75.2)
- added D7: LED, LED_SMD:LED_0603_1608Metric_Pad1.05x0.95mm_HandSolder, F.Cu at (169.7, 81.2)
- added D8: LED, LED_SMD:LED_0603_1608Metric_Pad1.05x0.95mm_HandSolder, F.Cu at (121.4, 82.2)
- added D9: LED, LED_SMD:LED_0603_1608Metric_Pad1.05x0.95mm_HandSolder, F.Cu at (186.8, 94.3)
- added R45: 10K 1%, Resistor_SMD:R_0603_1608Metric_Pad0.98x0.95mm_HandSolder, F.Cu at (183.5, 100.9)
- added R46: 10K 1%, Resistor_SMD:R_0603_1608Metric_Pad0.98x0.95mm_HandSolder, F.Cu at (181.1, 75.2)
- added R47: 1K 1%, Resistor_SMD:R_0603_1608Metric_Pad0.98x0.95mm_HandSolder, F.Cu at (169.7, 84.8)
- added R48: 1K 1%, Resistor_SMD:R_0603_1608Metric_Pad0.98x0.95mm_HandSolder, F.Cu at (121.4, 86.0)
- added R49: 1K 1%, Resistor_SMD:R_0603_1608Metric_Pad0.98x0.95mm_HandSolder, F.Cu at (183.5, 94.3)
- added TP1: +3.3V, TestPoint:TestPoint_Keystone_5000-5004_Miniature, F.Cu at (177.9, 77.1)
- added TP10: GND, TestPoint:TestPoint_Keystone_5000-5004_Miniature, F.Cu at (104.3, 84.5)
- added TP11: GND, TestPoint:TestPoint_Keystone_5000-5004_Miniature, F.Cu at (104.3, 115.2)
- added TP2: +5VA, TestPoint:TestPoint_Keystone_5000-5004_Miniature, F.Cu at (104.3, 110.2)
- added TP3: +9V, TestPoint:TestPoint_Keystone_5000-5004_Miniature, F.Cu at (187.3, 77.9)
- added TP4: +VSEL, TestPoint:TestPoint_Keystone_5000-5004_Miniature, F.Cu at (177.9, 93.1)
- added TP5: +VEXT, TestPoint:TestPoint_Keystone_5000-5004_Miniature, F.Cu at (190.1, 93.1)
- added TP6: +3VBAT, TestPoint:TestPoint_Keystone_5000-5004_Miniature, F.Cu at (117.6, 77.1)
- added TP7: +5V, TestPoint:TestPoint_Keystone_5000-5004_Miniature, F.Cu at (122.1, 77.1)
- added TP8: +VBUS, TestPoint:TestPoint_Keystone_5000-5004_Miniature, F.Cu at (190.1, 100.5)
- added TP9: GND, TestPoint:TestPoint_Keystone_5000-5004_Miniature, F.Cu at (190.1, 75.4)
- moved BT1 19.0 mm to (96.2, 44.4)
- moved C30 6.42 mm to (118.0, 100.0), turned to 90 degrees
- moved R21 6.13 mm to (183.0, 110.4)
- moved C27 5.48 mm to (125.6, 100.0), turned to -90 degrees
- moved C16 5.24 mm to (186.8, 99.4)
- moved Q1 4.87 mm to (174.2, 103.7), turned to 90 degrees
- moved C37 4.13 mm to (127.9, 89.1), turned to 0 degrees
- moved C38 4.13 mm to (176.2, 89.1)
- moved C6 3.24 mm to (138.1, 109.9)
- moved C7 3.24 mm to (138.1, 106.6)
- moved R41 2.34 mm to (127.1, 91.9)
- moved C12 2.05 mm to (172.1, 89.1)
- moved R40 1.98 mm to (128.7, 91.9)
- moved R39 1.78 mm to (176.2, 100.0), turned to 90 degrees
- moved U4 1.78 mm to (174.1, 83.5)
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Connections:
- J1 pad S1: unconnected-(J1-SHIELD-PadS1) -> GND
- J2 pad 9: unconnected-(J2-SHIELD-Pad9) -> GND
- J3 pad 18: unconnected-(J3-Pin_18-Pad18) -> USB OTG ID
- U6 pad 1: GND -> +3.3V
- U6 pad 2: +3.3V -> GND
Routing:
- net USB OTG ID: track 0.00 -> 36.4 mm, vias 0 -> 1
- net NEOPIXEL DIN: track 0.00 -> 34.5 mm, vias 0 -> 2
- net +3.3V: track 31.7 -> 48.3 mm
- net +5V: track 0.00 -> 16.6 mm
- net PWM BUZZER: track 27.0 -> 38.7 mm, vias 2 -> 1
- net NEOPIXEL DOUT: track 0.00 -> 10.7 mm
- net I2C SDA 5V: track 34.3 -> 43.7 mm
- net GND: track 48.2 -> 39.1 mm
- net I2C SCL 5V: track 34.3 -> 40.7 mm
- net Net-(Q1-C): track 0.00 -> 5.19 mm
- net +VSEL: track 0.00 -> 5.17 mm
- net +5VA: track 13.6 -> 18.2 mm
- net +9V: track 0.00 -> 2.76 mm
- net /IO/SD DAT1 SPI: track 11.6 -> 13.5 mm
- net A0: track 23.1 -> 21.3 mm
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- added copper zone on In2.Cu, net +3.3V
- added copper zone on In2.Cu, net +5V
- added copper zone on In2.Cu, net +5VA
- added copper zone on In2.Cu, net +9V
- added copper zone on In2.Cu, net +VBUS
- added copper zone on In2.Cu, net +VSEL
- added copper zone on B.Cu, net GND
- added copper zone on F.Cu, net GND
- added copper zone on In1.Cu, net GND
- added copper zone on In2.Cu, net GND
Other:
- copper layers 2 -> 4
- board text added: "STM32 EXPLORER Mechatronix Lab Rev.00 2024.05.10"
- board text removed: "STM32 EXPLORER BOARD Mechatronix Lab Rev.00 2024.05.10"

Commit message: Added new PNs for some components. Overall improvements in schematic and layout.
Parts:
- D3: value 1N5819WS -> STPS1L40-Y; footprint Diode_SMD:D_SOD-323 -> Diode_SMD:D_SOD-123
- L3: value L_Small -> 10uH; footprint Inductor_SMD:L_0603_1608Metric_Pad1.05x0.95mm_HandSolder -> STM32XP:WE 74404024100
- moved D6 2.54 mm to (186.8, 75.1)
- moved R46 2.42 mm to (183.5, 75.1)
- moved R43 1.27 mm to (180.5, 78.4), turned to 90 degrees
- moved R42 0.92 mm to (182.0, 78.4), turned to -90 degrees
- moved D3 0.82 mm to (184.0, 81.0)
- moved JP1 0.80 mm to (184.5, 77.1), turned to 0 degrees
- moved C35 0.72 mm to (180.7, 81.2)
- moved JP2 0.65 mm to (184.5, 88.1)
- moved U8 0.57 mm to (180.7, 84.3)
- moved D4 0.55 mm to (184.5, 91.5)
- moved C34 0.51 mm to (180.7, 87.3)
- moved R44 0.51 mm to (180.7, 89.1)
- moved TP3 0.51 mm to (187.8, 77.9)
- moved L3 0.36 mm to (184.0, 85.0)
Routing:
- net +5VA: track 18.2 -> 34.8 mm, vias 0 -> 9
- net GND: track 39.1 -> 33.7 mm, vias 3 -> 16
- net PC2: track 30.9 -> 31.9 mm
- net SWDIO: track 22.2 -> 21.4 mm
- net AIN2: track 16.8 -> 17.6 mm
- net PA2: track 26.2 -> 27.0 mm
- net PA3: track 26.5 -> 27.3 mm
- net PA1: track 29.0 -> 29.7 mm
- net PA0: track 31.7 -> 32.4 mm
- net AIN1: track 16.0 -> 16.5 mm
