File: HARDWARE/KICAD/STM32XP.kicad_pcb (KiCad board)
At the start: 4 copper layers, 99.1 x 53.3 mm, 148 parts, among them J1 USB_C_Receptacle_USB2.0_16P, J2 Micro_SD_Card, J3 Conn_01x20_Socket, J4 Conn_01x20_Socket, J5 Jack-DC, J9 Conn_02x05_Odd_Even, Q1 MMBT3904, Q2 2N7002, Q3 2N7002, SW1 SW_Push, SW2 SW_Push, SW3 RST, SW4 SW_Push, SW5 SW_Push, SW6 SW_Push, SW7 SW_Push, SW8 SW_Push, U1 STM32F411RETx, U2 ADS1115IDGS, U3 LM324, U4 AMS1117-3.3, U5 USBLC6-2SC6, U6 OLED 128x64 1.3", U7 AMS1117-5.0, U8 AP3012, Y1 32.768kHz, Y2 8MHz xpF

Commit message: Continuing layout and routing.
Parts:
- moved R48 1.40 mm to (121.4, 84.6)
- moved C33 1.40 mm to (130.3, 81.7)
- moved D1 1.27 mm to (134.8, 81.7)
- moved R7 1.14 mm to (166.0, 81.2)
- moved D8 1.02 mm to (121.4, 81.2)
- moved R8 0.76 mm to (164.5, 81.2)
- moved R44 0.51 mm to (180.7, 88.6)
- moved C34 0.51 mm to (180.7, 86.8)
- moved C35 0.51 mm to (180.7, 80.7)
- moved R42 0.51 mm to (182.0, 77.9)
- moved R43 0.51 mm to (180.5, 77.9)
- moved U8 0.51 mm to (180.7, 83.7)
- moved R9 0.38 mm to (163.0, 81.2)
- moved C3 0.13 mm to (154.6, 107.6)
Routing:
- net +9V: track 2.76 -> 81.3 mm, vias 0 -> 1
- net +VSEL: track 5.17 -> 21.8 mm, vias 0 -> 3
- net /POWER/BOOST FB: track 0.00 -> 8.58 mm, vias 0 -> 2
- net GND: track 33.7 -> 25.4 mm, vias 16 -> 26
- net +5V: track 16.6 -> 22.5 mm, vias 0 -> 2
- net /POWER/BOOST ~{SHDN}: track 0.00 -> 4.86 mm
- net VCORE: track 5.41 -> 9.42 mm
- net /POWER/BOOST SW: track 0.00 -> 3.82 mm
- net Net-(D7-K): track 0.00 -> 1.78 mm
- net Net-(D8-K): track 0.00 -> 1.64 mm
- net Net-(D9-K): track 0.00 -> 1.52 mm
- net Net-(D6-K): track 0.00 -> 1.51 mm
- net NRST: track 34.9 -> 33.6 mm
- net I2C SCL 5V: track 40.7 -> 41.2 mm
- net +VBUS: track 14.2 -> 14.1 mm, vias 3 -> 6
- added copper zone on F.Cu, net +VBUS
- added copper zone on F.Cu, net +VEXT
- added copper zone on F.Cu, net /POWER/BOOST IN
- added copper zone on F.Cu, net /POWER/BOOST OUT

Commit message: Continuing PCB layout and routing.
Parts:
- moved C6 5.93 mm to (133.7, 105.8), turned to 90 degrees
- moved L1 5.46 mm to (136.5, 104.8), turned to 0 degrees
- moved R10 3.34 mm to (136.5, 102.8)
- moved C7 1.48 mm to (139.3, 105.8), turned to 90 degrees
- moved C5 0.88 mm to (141.1, 105.6), turned to 90 degrees
Routing:
- net +3.3V: track 48.5 -> 60.9 mm, vias 3 -> 15
- net GND: track 25.4 -> 22.1 mm, vias 26 -> 73
- net NRST: track 33.6 -> 36.1 mm
- net +5V: track 22.5 -> 24.4 mm, vias 2 -> 5
- net +3.3VA: track 9.54 -> 8.38 mm
- net +VBUS: track 14.1 -> 14.9 mm

Commit message: Trying to solve all errors on DRC, but some depend on finishing other tasks.
Parts:
- added TP12: +VCORE, TestPoint:TestPoint_Keystone_5000-5004_Miniature, F.Cu at (153.7, 114.0)
- Q3: renamed from Q1; value MMBT3904 -> 2N7002
- moved G*** 18.4 mm to (109.4, 63.2)
- moved TP2 15.4 mm to (104.3, 84.8)
- moved BT1 5.91 mm to (91.7, 48.3), turned to -90 degrees
- moved TP6 5.33 mm to (104.3, 89.8)
- moved TP7 3.81 mm to (174.1, 93.1)
- renumbered C35 to C1, C8 to C10, C1 to C11, C39 to C12, C22 to C13, C19 to C14, C36 to C15, C21 to C16, C20 to C17, C2 to C18, C10 to C19, C33 to C2, C16 to C20, C29 to C21, C30 to C22, C28 to C23, C27 to C24, C9 to C25, C13 to C26, C23 to C27, C25 to C28, C5 to C29, C15 to C3, C24 to C30, C26 to C31, C6 to C32, C7 to C33, C4 to C34, C3 to C35, C14 to C36, C11 to C37, C18 to C38, C17 to C39, C32 to C4, C34 to C5, C31 to C6, C37 to C7, C12 to C8, C38 to C9, D6 to D1, D3 to D2, D8 to D3, D7 to D4, D1 to D5, D4 to D6, D9 to D7, D2 to D8, D5 to D9, J4 to J1, J5 to J2, J9 to J3, J1 to J4, J2 to J5, J3 to J6, L3 to L1, L4 to L2, L2 to L3, L1 to L4, Q2 to Q1, Q3 to Q2, R46 to R1, R44 to R10, R5 to R11, R4 to R12, R3 to R13, R6 to R14, R1 to R15, R12 to R16, R13 to R17, R41 to R18, R40 to R19, R43 to R2, R24 to R20, R23 to R21, R25 to R22, R22 to R23, R49 to R24, R2 to R25, R39 to R26, R33 to R27, R45 to R28, R32 to R29, R42 to R3, R10 to R30, R30 to R32, R20 to R33, R27 to R34, R29 to R35, R16 to R36, R26 to R37, R28 to R38, R17 to R39, R11 to R4, R19 to R40, R34 to R41, R18 to R42, R21 to R43, R36 to R44, R38 to R45, R37 to R46, R14 to R47, R15 to R48, R35 to R49, R9 to R5, R8 to R6, R48 to R8, R47 to R9, SW3 to SW1, SW4 to SW2, SW6 to SW3, SW8 to SW4, SW7 to SW5, SW1 to SW6, SW2 to SW7, SW5 to SW8, TP9 to TP1, TP2 to TP10, TP6 to TP2, TP7 to TP3, TP1 to TP4, TP3 to TP5, TP10 to TP6, TP4 to TP7, TP5 to TP8, TP8 to TP9, U7 to U1, U4 to U2, U8 to U3, U6 to U4, U3 to U6, U2 to U7, U1 to U8
Connections:
- net VCORE renamed +VCORE
Routing:
- net +VSEL: track 21.8 -> 32.0 mm
- net +VCORE: track 9.41 -> 18.2 mm
- net GND: track 22.1 -> 19.9 mm, vias 73 -> 98
- net Net-(D9-K): track 0.00 -> 1.51 mm
- net +5V: track 24.4 -> 25.7 mm, vias 5 -> 6
- net +3.3V: track 60.9 -> 62.1 mm

Commit message: Changed tactile switch model; had to enlarge board and adjust positioning of components; added some 3D models and comments with PNs for further reference; general layout and routing improvements.
Parts:
- added C40: 100nF 50V, Capacitor_SMD:C_0603_1608Metric_Pad1.08x0.95mm_HandSolder, F.Cu at (139.8, 84.1)
- added C41: 100nF 50V, Capacitor_SMD:C_0603_1608Metric_Pad1.08x0.95mm_HandSolder, F.Cu at (136.0, 83.2)
- added C42: 10pF 50V, Capacitor_SMD:C_0603_1608Metric_Pad1.08x0.95mm_HandSolder, F.Cu at (139.8, 90.8)
- added C43: 10pF 50V, Capacitor_SMD:C_0603_1608Metric_Pad1.08x0.95mm_HandSolder, F.Cu at (137.9, 90.8)
- added R50: 10K 1%, Resistor_SMD:R_0603_1608Metric_Pad0.98x0.95mm_HandSolder, F.Cu at (183.0, 112.4)
- added TP13: GND, TestPoint:TestPoint_Keystone_5000-5004_Miniature, F.Cu at (197.0, 125.4)
- SW1: footprint Button_Switch_SMD:SW_SPST_CK_KXT3 -> Button_Switch_SMD:SW_Push_1P1T_NO_CK_KSC6xxJ
- SW2: value SW_Push -> UP; footprint Button_Switch_SMD:SW_SPST_CK_KXT3 -> Button_Switch_SMD:SW_Push_1P1T_NO_CK_KSC6xxJ
- SW3: value SW_Push -> LEFT; footprint Button_Switch_SMD:SW_SPST_CK_KXT3 -> Button_Switch_SMD:SW_Push_1P1T_NO_CK_KSC6xxJ
- SW4: value SW_Push -> CENTER; footprint Button_Switch_SMD:SW_SPST_CK_KXT3 -> Button_Switch_SMD:SW_Push_1P1T_NO_CK_KSC6xxJ
- SW5: value SW_Push -> RIGHT; footprint Button_Switch_SMD:SW_SPST_CK_KXT3 -> Button_Switch_SMD:SW_Push_1P1T_NO_CK_KSC6xxJ
- SW6: value SW_Push -> BUTTON 1; footprint Button_Switch_SMD:SW_SPST_CK_KXT3 -> Button_Switch_SMD:SW_Push_1P1T_NO_CK_KSC6xxJ
- SW7: value SW_Push -> BUTTON 2; footprint Button_Switch_SMD:SW_SPST_CK_KXT3 -> Button_Switch_SMD:SW_Push_1P1T_NO_CK_KSC6xxJ
- SW8: value SW_Push -> DOWN; footprint Button_Switch_SMD:SW_SPST_CK_KXT3 -> Button_Switch_SMD:SW_Push_1P1T_NO_CK_KSC6xxJ
- moved TP6 22.2 mm to (109.4, 68.2)
- moved G*** 14.2 mm to (111.9, 77.1)
- moved SW8 13.9 mm to (118.2, 130.5), turned to 180 degrees
- moved R18 13.6 mm to (136.1, 81.6), turned to 180 degrees
- moved SW3 12.6 mm to (109.4, 121.6), turned to 90 degrees
- moved R41 12.0 mm to (113.8, 117.8), turned to -90 degrees
- moved R44 11.4 mm to (113.8, 125.4), turned to -90 degrees
- moved TP11 10.2 mm to (103.0, 125.4)
- moved R19 10.2 mm to (136.0, 84.8), turned to 180 degrees
- moved SW4 10.1 mm to (118.2, 121.6), turned to 90 degrees
- moved TP5 9.72 mm to (197.0, 74.6)
- moved C12 8.96 mm to (189.7, 93.3), turned to 180 degrees
- moved R14 8.95 mm to (142.7, 86.0), turned to 90 degrees
- moved SW6 8.91 mm to (172.9, 121.6), turned to 90 degrees
- moved SW5 8.91 mm to (127.1, 121.6), turned to -90 degrees
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Connections:
- J3 pad 5: GND -> +5VA
- J5 pad 8: /IO/SD DAT1 SPI -> SPI SCK
- R43 pad 1: /IO/SD DAT1 SPI -> SPI SCK
- U8 pad 51: unconnected-(U8-PC10-Pad51) -> SD CARD ~{IN}
Routing:
- net SPI SCK: track 53.6 -> 73.5 mm
- net BUTTON UP: track 34.5 -> 53.2 mm
- net BUTTON RIGHT: track 31.3 -> 48.8 mm
- net BUTTON LEFT: track 39.6 -> 56.4 mm
- net BUTTON DOWN: track 39.3 -> 52.9 mm
- net /IO/SD DAT1 SPI: track 13.5 -> 0.00 mm
- net I2C SCL 3.3V: track 23.0 -> 34.8 mm
- net BUTTON CENTER: track 36.2 -> 47.0 mm
- net NRST: track 36.1 -> 46.4 mm
- net +VBUS: track 14.9 -> 5.66 mm, vias 6 -> 4
- net I2C SDA 3.3V: track 23.3 -> 32.5 mm
- net DEBUG TX: track 13.9 -> 21.2 mm
- net SWO: track 21.0 -> 28.2 mm
- net SWCLK: track 18.0 -> 25.2 mm
- net SWDIO: track 20.9 -> 28.1 mm
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Other:
- board size 99.1 x 53.3 mm -> 99.1 x 68.6 mm
- board text added: "STM32 EXPLORER BOARD Rev.00 2024.05.10 Mechatronix Lab Eng. André A. M. Araújo"
- board text removed: "STM32 EXPLORER Mechatronix Lab Rev.00 2024.05.10"

Commit message: More improvements. Added 3D models. Added legends.
Parts:
- BT1: footprint Battery:BatteryHolder_Multicomp_BC-2001_1x2032 -> Battery:BatteryHolder_Keystone_1060_1x2032
- LS1: moved to F.Cu
- moved BT1 81.8 mm to (150.0, 100.0), turned to 0 degrees
- moved TP2 33.3 mm to (130.9, 102.9)
- moved R26 14.4 mm to (174.1, 85.7), turned to 0 degrees
- moved Q3 13.8 mm to (167.5, 91.7)
- moved LS1 8.81 mm to (176.1, 91.4)
- moved TP7 8.74 mm to (179.2, 86.0)
- moved R1 7.98 mm to (190.3, 74.0), turned to 180 degrees
- moved R28 6.81 mm to (190.3, 100.6), turned to 180 degrees
- moved R24 6.80 mm to (190.3, 89.2), turned to 180 degrees
- moved C39 5.02 mm to (195.3, 121.6)
- moved C38 4.95 mm to (195.3, 119.8)
- moved D1 4.19 mm to (186.8, 74.0), turned to 180 degrees
- moved J1 2.54 mm to (174.1, 68.2)
- moved J6 2.54 mm to (125.9, 131.8)
- moved R8 1.40 mm to (121.4, 79.7)
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Connections:
- J5 pad 8: SPI SCK -> /IO/SD DAT1 SPI
- R43 pad 1: SPI SCK -> /IO/SD DAT1 SPI
Routing:
- net SD CARD ~{IN}: track 0.00 -> 49.4 mm, vias 0 -> 2
- net BUTTON 2: track 25.5 -> 41.7 mm
- net +3VBAT: track 3.91 -> 18.6 mm, vias 0 -> 1
- net /IO/SD DAT1 SPI: track 0.00 -> 14.6 mm
- net BUTTON 1: track 22.9 -> 37.5 mm
- net +5VA: track 33.5 -> 46.8 mm
- net SPI SCK: track 73.5 -> 62.5 mm
- net Net-(Q3-D): track 5.19 -> 11.4 mm
- net +VSEL: track 32.1 -> 26.0 mm
- net +3.3V: track 62.0 -> 67.8 mm, vias 15 -> 25
- net +5V: track 26.4 -> 20.8 mm, vias 8 -> 7
- net /POWER/BOOST FB: track 3.17 -> 8.61 mm
- net Net-(J1-Pin_6): track 3.99 -> 7.87 mm
- net Net-(J1-Pin_5): track 3.57 -> 7.45 mm
- net Net-(J1-Pin_4): track 3.15 -> 7.03 mm
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Other:
- board text added: "+3.3V"
- board text added: "+5V"
- board text added: "A0"
- board text added: "A1"
- board text added: "A2"
- board text added: "A3"
- board text added: "A4"
- board text added: "A5"
- board text added: "A6"
- board text added: "A7"
- board text added: "BLUE"
- board text added: "BUZZER"
- board text added: "C0"
- board text added: "C1"
- board text added: "C2"
- board text added: "C3"
- board text added: "DIN"
- board text added: "DOUT"
- board text added: "GND"
- board text added: "GREEN"
- board text added: "MISO"
- board text added: "MOSI"
- board text added: "NSS"
- board text added: "OTG"
- board text added: "RED"
- board text added: "RST"
- board text added: "RX"
- board text added: "SCK"
- board text added: "SCL3"
- board text added: "SCL5"
- board text added: "SDA3"
- board text added: "SDA5"
- board text added: "SWCLK"
- board text added: "SWDIO"
- board text added: "SWO"
- board text added: "TX"
