File: HARDWARE/KICAD/STM32XP.kicad_pcb (KiCad board)
At the start: 4 copper layers, 99.1 x 68.6 mm, 155 parts, among them J1 Conn_01x20_Socket, J2 Jack-DC, J3 Conn_02x05_Odd_Even, J4 USB_C_Receptacle_USB2.0_16P, J5 Micro_SD_Card, J6 Conn_01x20_Socket, Q1 2N7002, Q2 2N7002, Q3 2N7002, SW1 RST, SW2 UP, SW3 LEFT, SW4 CENTER, SW5 RIGHT, SW6 BUTTON 1, SW7 BUTTON 2, SW8 DOWN, U1 AMS1117-5.0, U2 AMS1117-3.3, U3 AP3012, U4 OLED 128x64 1.3", U5 USBLC6-2SC6, U6 LM324, U7 ADS1115IDGS, U8 STM32F411RETx, Y1 32.768kHz, Y2 8MHz xpF

Commit message: Added stiching vias.
Routing:
- net GND: track 21.9 -> 17.3 mm, vias 78 -> 197
- net Net-(D4-K): track 0.00 -> 1.70 mm
- net +5V: track 20.8 -> 19.8 mm
- net +3.3V: track 67.8 -> 68.7 mm, vias 25 -> 26

Commit message: Added fiducial marks.
Parts:
- added FID1: Fiducial, Fiducial:Fiducial_0.75mm_Mask1.5mm, F.Cu at (104.3, 74.6)
- added FID2: Fiducial, Fiducial:Fiducial_0.75mm_Mask1.5mm, F.Cu at (190.6, 125.4)
- added FID3: Fiducial, Fiducial:Fiducial_0.75mm_Mask1.5mm, F.Cu at (109.4, 130.5)

Commit message: Improvements to layout. Fixed most of errors and warnings. Added correct footprint for Micro SD socket. Added markings and symbols to legend.
Parts:
- added G***: LOGO, LOGO, B.Cu at (119.8, 87.3)
- added REF**: OSHW-Symbol_6.7x6mm_SilkScreen, Symbol:OSHW-Symbol_6.7x6mm_SilkScreen, F.Cu at (150.0, 122.6)
- added REF**: OSHW-Logo_19x20mm_SilkScreen, Symbol:OSHW-Logo_19x20mm_SilkScreen, B.Cu at (119.8, 112.7)
- J5: value Micro_SD_Card -> MICRO SD; footprint Connector_Card:microSD_HC_Wuerth_693072010801 -> STM32XP:WE 693071020811
- moved FID2 51.1 mm to (195.7, 74.6)
- moved C39 19.6 mm to (183.3, 106.1)
- moved C38 14.8 mm to (183.3, 111.2)
- moved R28 13.6 mm to (181.1, 90.6)
- moved D9 13.0 mm to (181.2, 89.0), turned to 0 degrees
- moved R1 9.72 mm to (181.5, 69.9), turned to 0 degrees
- moved TP9 7.55 mm to (183.0, 100.0)
- moved R47 6.99 mm to (168.4, 121.6), turned to -90 degrees
- moved R48 6.99 mm to (177.3, 121.6), turned to 90 degrees
- moved R50 6.99 mm to (177.3, 117.8), turned to -90 degrees
- moved TP5 6.48 mm to (190.6, 73.3)
- moved TP8 6.35 mm to (190.6, 88.7)
- moved R24 5.58 mm to (184.9, 90.6), turned to 0 degrees
- moved R40 5.55 mm to (183.3, 114.2)
- moved R43 5.18 mm to (183.3, 115.7)
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Connections:
- J5 pad 9: GND -> SD CARD ~{IN}
Routing:
- net SPI NSS: track 63.1 -> 49.8 mm
- net /IO/SD DAT0 SPI: track 14.9 -> 2.67 mm
- net /IO/SD DAT1 SPI: track 14.6 -> 2.61 mm
- net +VBUS: track 5.64 -> 16.9 mm, vias 4 -> 8
- net +VSEL: track 26.0 -> 37.1 mm
- net /IO/SD DAT2 SPI: track 13.5 -> 2.57 mm
- net GND: track 17.3 -> 6.88 mm, vias 197 -> 258
- net SPI SCK: track 62.5 -> 52.5 mm
- net SPI MOSI: track 64.1 -> 55.0 mm
- net +3.3V: track 68.7 -> 62.5 mm, vias 26 -> 27
- net SD CARD ~{IN}: track 49.4 -> 54.8 mm
- net BUTTON 2: track 41.7 -> 46.9 mm
- net BUTTON 1: track 37.5 -> 41.2 mm
- net SPI MISO: track 58.9 -> 61.5 mm
- net USB OTG ID: track 46.0 -> 44.1 mm
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- removed copper zone on F.Cu, net +VBUS
Other:
- board text added: "FW"
- board text added: "SCL3V"
- board text added: "SCL5V"
- board text added: "SDA3V"
- board text added: "SDA5V"
- board text added: "github.com/mechatronixlab instagram.com/mechatronixlab"
- board text removed: "SCL3"
- board text removed: "SCL5"
- board text removed: "SDA3"
- board text removed: "SDA5"

Commit message: Finished PCB design, but needs to be reviewed. Added all components and PNs that were missing or incorrect. Added draft of STM32 EXPLORER logo.
Parts:
- removed the G*** at (109.4, 78.4)
- removed the L3 at (180.5, 96.2)
- removed REF**: OSHW-Symbol_6.7x6mm_SilkScreen, Symbol:OSHW-Symbol_6.7x6mm_SilkScreen
- removed REF**: OSHW-Logo_19x20mm_SilkScreen, Symbol:OSHW-Logo_19x20mm_SilkScreen
- added C1: 10uF 25V, Capacitor_SMD:C_0805_2012Metric_Pad1.18x1.45mm_HandSolder, F.Cu at (115.5, 74.3)
- added C16: 680nF 16V, Capacitor_SMD:C_0603_1608Metric_Pad1.08x0.95mm_HandSolder, F.Cu at (186.8, 92.1)
- added D10: 150505M173300, STM32XP:WE 150505M173300, F.Cu at (174.1, 100.0)
- added FB1: 600R, Inductor_SMD:L_0603_1608Metric_Pad1.05x0.95mm_HandSolder, F.Cu at (124.9, 86.8)
- added FB2: 600R, Inductor_SMD:L_0603_1608Metric_Pad1.05x0.95mm_HandSolder, F.Cu at (181.1, 93.7)
- added FB3: 600R, Inductor_SMD:L_0603_1608Metric_Pad1.05x0.95mm_HandSolder, F.Cu at (186.8, 93.7)
- added G***: LOGO, LOGO, F.Cu at (135.6, 123.3)
- added G***: LOGO, LOGO, F.Cu at (188.5, 124.3)
- J4: value USB_C_Receptacle_USB2.0_16P -> USB TYPE C
- L2: value L_Small -> 744232090; footprint Inductor_SMD:L_0603_1608Metric_Pad1.05x0.95mm_HandSolder -> STM32XP:WE 744232090
- LS1: value Speaker_Crystal -> 78dB 4kHz; footprint Buzzer_Beeper:MagneticBuzzer_PUI_AT-0927-TT-6-R -> STM32XP:PKM13EPYH4000-A0; moved to B.Cu
- moved LS1 65.8 mm to (111.9, 77.1), turned to -90 degrees
- moved R8 60.8 mm to (111.9, 77.1), turned to 180 degrees
- moved L2 57.0 mm to (181.1, 96.2), turned to 0 degrees
- moved Q1 53.9 mm to (115.6, 77.1), turned to 180 degrees
- moved G*** 12.9 mm to (118.2, 100.1)
- moved SW1 0.32 mm to (158.9, 77.1)
- moved R18 0.32 mm to (153.0, 90.3)
- moved R19 0.32 mm to (154.6, 90.3)
- moved R20 0.32 mm to (156.1, 90.3)
- moved R16 0.19 mm to (146.7, 90.3)
- moved R17 0.19 mm to (148.2, 90.3)
- renumbered C9 to C10, C40 to C11, C4 to C12, C15 to C13, C43 to C14, C42 to C15, C10 to C17, C11 to C18, C12 to C19, C1 to C2, C13 to C20, C14 to C21, C16 to C22, C17 to C23, C18 to C24, C19 to C25, C20 to C26, C21 to C27, C22 to C28, C23 to C29, C2 to C3, C24 to C30, C25 to C31, C26 to C32, C27 to C33, C28 to C34, C29 to C35, C32 to C36, C33 to C37, C30 to C38, C31 to C39, C5 to C4, C39 to C40, C34 to C41, C35 to C42, C36 to C43, C37 to C44, C38 to C45, C41 to C5, C3 to C6, C6 to C7, C7 to C8, C8 to C9, D9 to D7, D7 to D8, D8 to D9, L4 to L3, Q3 to Q1, Q1 to Q2, Q2 to Q3, R9 to R10, R18 to R11, R11 to R12, R10 to R13, R19 to R14, R14 to R15, R12 to R16, R13 to R17, R15 to R18, R16 to R19, R17 to R20, R28 to R21, R24 to R22, R20 to R23, R21 to R24, R22 to R25, R23 to R26, R25 to R27, R27 to R28, R34 to R33, R35 to R34, R36 to R35, R37 to R36, R38 to R37, R33 to R38, R42 to R40, R40 to R41, R43 to R42, R41 to R43, R45 to R44, R50 to R45, R44 to R49, R49 to R50, R26 to R8, R8 to R9, TP6 to TP1, TP12 to TP11, TP11 to TP12, TP3 to TP2, TP4 to TP3, TP1 to TP4, TP7 to TP6, TP8 to TP7, TP9 to TP8, TP2 to TP9
Connections:
- D6 pad 1: +VBUS -> +VBUSF
- D7 pad 2: +VBUS -> +VBUSF
- L2 pad 1: +5V -> USB D-
- L2 pad 2: +5VA -> /IO/USB FILTERED D-
- LS1 pad 1: +VSEL -> +9V
- R8 pad 2: +VSEL -> +9V
Routing:
- net PWM BUZZER: track 47.7 -> 109.4 mm, vias 2 -> 4
- net +9V: track 83.4 -> 108.5 mm
- net PWM GREEN: track 30.9 -> 50.5 mm, vias 1 -> 3
- net PWM RED: track 29.8 -> 49.2 mm
- net +VSEL: track 37.1 -> 21.0 mm, vias 3 -> 5
- net PWM BLUE: track 33.7 -> 46.8 mm
- net +VBUSF: track 0.00 -> 8.22 mm
- net Net-(Q1-D): track 11.0 -> 4.71 mm
- net /IO/USB FILTERED POWER: track 0.00 -> 5.56 mm
- net NRST: track 47.9 -> 45.4 mm
- net +VBUS: track 16.9 -> 14.5 mm, vias 8 -> 6
- net GND: track 6.88 -> 4.74 mm, vias 258 -> 439
- net BUTTON 2: track 46.9 -> 48.0 mm
- net USB OTG ID: track 44.1 -> 45.0 mm
- net /IO/USB FILTERED D-: track 4.54 -> 3.72 mm
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Other:
- board text added: "STM32 EXPLORER"
- board text added: "STM32XP Rev.00 2024.05.10 Mechatronix Lab Eng. André A. M. Araújo"
- board text removed: "STM32 EXPLORER BOARD Rev.00 2024.05.10 Mechatronix Lab Eng. André A. M. Araújo"
