File: HARDWARE/KICAD/ANALOG.kicad_sch (KiCad schematic)
At the start: 24 parts, among them J9 Conn_02x05_Odd_Even, U2 ADS1115IDGS, U3 LM324

Commit message: Continuing layout and routing.
Other:
- company: (none) -> Mechatronix Lab
- title: (none) -> STM32 EXPLORER BOARD
- moved on the sheet: C24
Changed lines of the file:
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@@
 	(generator_version "8.0")
 	(paper "A4")
+	(title_block
+		(title "STM32 EXPLORER BOARD")
+		(date "2024-04-26")
+		(rev "00")
+		(company "Mechatronix Lab")
+		(comment 1 "Eng. André A. M. Araújo")
+	)
 	(junction
 		(at 68.58 105.41)
@@
 	(symbol
 		(lib_id "Device:C_Small")
-		(at 139.7 127 180)
+		(at 139.7 127 0)
+		(mirror x)
 		(unit 1)
 		(exclude_from_sim no)
@@
 		(dnp no)
 		(property "Reference" "C24"
-			(at 137.16 128.27 90)
+			(at 142.24 128.27 90)
 			(effects
 				(font
@@
 		)
 		(property "Value" "100nF 50V"
-			(at 142.24 132.08 90)
-			(effects
-				(font
+			(at 137.16 132.08 90)
+			(effects
+				(font

Commit message: Trying to solve all errors on DRC, but some depend on finishing other tasks.
Parts:
- renumbered C22 to C13, C19 to C14, C21 to C16, C20 to C17, C29 to C21, C30 to C22, C28 to C23, C27 to C24, C23 to C27, C25 to C28, C24 to C30, C26 to C31, D2 to D8, J9 to J3, R24 to R20, R23 to R21, R25 to R22, R22 to R23, R27 to R34, R29 to R35, R26 to R37, R28 to R38, U3 to U6, U2 to U7
Changed lines of the file:
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@@
 		(on_board yes)
 		(dnp no)
-		(property "Reference" "J9"
+		(property "Reference" "J3"
 			(at 46.99 91.44 0)
 			(effects
@@
 			(project "STM32XP"
 				(path "/1f1b32b0-2877-4942-afdb-ad5dc4634e8b/f17fb096-3b39-4a0e-96ae-7df73a2ffb98"
-					(reference "J9")
+					(reference "J3")
 					(unit 1)
 				)
@@
 		(on_board yes)
 		(dnp no)
-		(property "Reference" "R25"
+		(property "Reference" "R22"
 			(at 133.35 78.74 90)
 			(effects
@@
 			(project "STM32XP"
 				(path "/1f1b32b0-2877-4942-afdb-ad5dc4634e8b/f17fb096-3b39-4a0e-96ae-7df73a2ffb98"
-					(reference "R25")
+					(reference "R22")
 					(unit 1)
 				)
@@
 		(on_board yes)
 		(dnp no)
-		(property "Reference" "C25"
+		(property "Reference" "C28"
 			(at 132.08 144.78 90)
 			(effects
@@
 			(project "STM32XP"
 				(path "/1f1b32b0-2877-4942-afdb-ad5dc4634e8b/f17fb096-3b39-4a0e-96ae-7df73a2ffb98"
-					(reference "C25")
+					(reference "C28")
 					(unit 1)
 				)
@@
 		(on_board yes)
 		(dnp no)
-		(property "Reference" "R28"
+		(property "Reference" "R38"
 			(at 120.65 154.94 90)
 			(effects
@@
 			(project "STM32XP"
 				(path "/1f1b32b0-2877-4942-afdb-ad5dc4634e8b/f17fb096-3b39-4a0e-96ae-7df73a2ffb98"
-					(reference "R28")
+					(reference "R38")
 					(unit 1)
 				)
@@
 		(on_board yes)
 		(dnp no)
-		(property "Reference" "C24"
+		(property "Reference" "C30"
 			(at 142.24 128.27 90)
 			(effects
@@
 			(project "STM32XP"
 				(path "/1f1b32b0-2877-4942-afdb-ad5dc4634e8b/f17fb096-3b39-4a0e-96ae-7df73a2ffb98"
-					(reference "C24")
+					(reference "C30")
 					(unit 1)
 				)
@@
 		(on_board yes)
 		(dnp no)
-		(property "Reference" "R26"
+		(property "Reference" "R37"
 			(at 120.65 116.84 90)
 			(effects
@@
 			(project "STM32XP"
 				(path "/1f1b32b0-2877-4942-afdb-ad5dc4634e8b/f17fb096-3b39-4a0e-96ae-7df73a2ffb98"
-					(reference "R26")
+					(reference "R37")
 					(unit 1)
 				)
@@
 		(on_board yes)
 		(dnp no)
-		(property "Reference" "U3"
+		(property "Reference" "U6"
 			(at 149.86 45.72 0)
 			(effects
@@
 			(project "STM32XP"
 				(path "/1f1b32b0-2877-4942-afdb-ad5dc4634e8b/f17fb096-3b39-4a0e-96ae-7df73a2ffb98"
-					(reference "U3")
+					(reference "U6")
 					(unit 1)
 				)
@@
 		(on_board yes)
 		(dnp no)
-		(property "Reference" "C30"
+		(property "Reference" "C22"
 			(at 67.31 44.45 90)
 			(effects
@@
 			(project "STM32XP"
 				(path "/1f1b32b0-2877-4942-afdb-ad5dc4634e8b/f17fb096-3b39-4a0e-96ae-7df73a2ffb98"
-					(reference "C30")
+					(reference "C22")
 					(unit 1)
 				)
@@
 		(on_board yes)
 		(dnp no)
-		(property "Reference" "R27"
+		(property "Reference" "R34"
 			(at 133.35 116.84 90)
 			(effects
@@
 			(project "STM32XP"
 				(path "/1f1b32b0-2877-4942-afdb-ad5dc4634e8b/f17fb096-3b39-4a0e-96ae-7df73a2ffb98"
-					(reference "R27")
+					(reference "R34")
 					(unit 1)
 				)
@@
 		(dnp no)
 		(fields_autoplaced yes)
-		(property "Reference" "U3"
+		(property "Reference" "U6"
 			(at 77.47 41.9099 0)
 			(effects
@@
 			(project "STM32XP"
 				(path "/1f1b32b0-2877-4942-afdb-ad5dc4634e8b/f17fb096-3b39-4a0e-96ae-7df73a2ffb98"
-					(reference "U3")
+					(reference "U6")
 					(unit 5)
 				)
@@
 		(on_board yes)
 		(dnp no)
-		(property "Reference" "C27"
+		(property "Reference" "C24"
 			(at 219.71 83.82 90)
 			(effects
@@
 			(project "STM32XP"
 				(path "/1f1b32b0-2877-4942-afdb-ad5dc4634e8b/f17fb096-3b39-4a0e-96ae-7df73a2ffb98"
-					(reference "C27")
+					(reference "C24")
 					(unit 1)
 				)
@@
 		(on_board yes)
 		(dnp no)
-		(property "Reference" "C29"
+		(property "Reference" "C21"
 			(at 58.42 44.45 90)
 			(effects
@@
 			(project "STM32XP"
 				(path "/1f1b32b0-2877-4942-afdb-ad5dc4634e8b/f17fb096-3b39-4a0e-96ae-7df73a2ffb98"
-					(reference "C29")
+					(reference "C21")
 					(unit 1)
 				)
@@
 		(on_board yes)
 		(dnp no)
-		(property "Reference" "R24"
+		(property "Reference" "R20"
 			(at 120.65 78.74 90)
 			(effects
@@
 			(project "STM32XP"
 				(path "/1f1b32b0-2877-4942-afdb-ad5dc4634e8b/f17fb096-3b39-4a0e-96ae-7df73a2ffb98"
-					(reference "R24")
+					(reference "R20")
 					(unit 1)
 				)
@@
 		(on_board yes)
 		(dnp no)
-		(property "Reference" "C20"
+		(property "Reference" "C17"
 			(at 132.08 30.48 90)
 			(effects
@@
 			(project "STM32XP"
 				(path "/1f1b32b0-2877-4942-afdb-ad5dc4634e8b/f17fb096-3b39-4a0e-96ae-7df73a2ffb98"
-					(reference "C20")
+					(reference "C17")
 					(unit 1)
 				)
@@
 		(on_board yes)
 		(dnp no)
-		(property "Reference" "U3"
+		(property "Reference" "U6"
 			(at 149.86 121.92 0)
 			(effects
@@
 			(project "STM32XP"
 				(path "/1f1b32b0-2877-4942-afdb-ad5dc4634e8b/f17fb096-3b39-4a0e-96ae-7df73a2ffb98"
-					(reference "U3")
+					(reference "U6")
 					(unit 3)
 				)
@@
 		(on_board yes)
 		(dnp no)
-		(property "Reference" "C28"
+		(property "Reference" "C23"
 			(at 219.71 76.2 90)
 			(effects
@@
 			(project "STM32XP"
 				(path "/1f1b32b0-2877-4942-afdb-ad5dc4634e8b/f17fb096-3b39-4a0e-96ae-7df73a2ffb98"
-					(reference "C28")
+					(reference "C23")
 					(unit 1)
 				)
@@
 		(on_board yes)
 		(dnp no)
-		(property "Reference" "C19"
+		(property "Reference" "C14"
 			(at 137.16 52.07 90)
 			(effects
@@
 			(project "STM32XP"
 				(path "/1f1b32b0-2877-4942-afdb-ad5dc4634e8b/f17fb096-3b39-4a0e-96ae-7df73a2ffb98"
-					(reference "C19")
+					(reference "C14")
 					(unit 1)
 				)
@@
 		(dnp no)
 		(fields_autoplaced yes)
-		(property "Reference" "D2"
+		(property "Reference" "D8"
 			(at 78.74 114.2999 0)
 			(effects
@@
 			(project "STM32XP"
 				(path "/1f1b32b0-2877-4942-afdb-ad5dc4634e8b/f17fb096-3b39-4a0e-96ae-7df73a2ffb98"
-					(reference "D2")
+					(reference "D8")
 					(unit 1)
 				)
@@
 		(on_board yes)
 		(dnp no)
-		(property "Reference" "R22"
+		(property "Reference" "R23"
 			(at 133.35 40.64 90)
 			(effects
@@
 			(project "STM32XP"
 				(path "/1f1b32b0-2877-4942-afdb-ad5dc4634e8b/f17fb096-3b39-4a0e-96ae-7df73a2ffb98"
-					(reference "R22")
+					(reference "R23")
 					(unit 1)
 				)
@@
 		(on_board yes)
 		(dnp no)
-		(property "Reference" "C22"
+		(property "Reference" "C13"
 			(at 137.16 90.17 90)
 			(effects
@@
 			(project "STM32XP"
 				(path "/1f1b32b0-2877-4942-afdb-ad5dc4634e8b/f17fb096-3b39-4a0e-96ae-7df73a2ffb98"
-					(reference "C22")
+					(reference "C13")
 					(unit 1)
 				)
@@
 		(on_board yes)
 		(dnp no)
-		(property "Reference" "R29"
+		(property "Reference" "R35"
 			(at 133.35 154.94 90)
 			(effects
@@
 			(project "STM32XP"
 				(path "/1f1b32b0-2877-4942-afdb-ad5dc4634e8b/f17fb096-3b39-4a0e-96ae-7df73a2ffb98"
-					(reference "R29")
+					(reference "R35")
 					(unit 1)
 				)
@@
 		(on_board yes)
 		(dnp no)
-		(property "Reference" "U3"
+		(property "Reference" "U6"
 			(at 149.86 83.82 0)
 			(effects
@@
 			(project "STM32XP"
 				(path "/1f1b32b0-2877-4942-afdb-ad5dc4634e8b/f17fb096-3b39-4a0e-96ae-7df73a2ffb98"
-					(reference "U3")
+					(reference "U6")
 					(unit 2)
 				)
@@
 		(on_board yes)
 		(dnp no)
-		(property "Reference" "R23"
+		(property "Reference" "R21"
 			(at 120.65 40.64 90)
 			(effects
@@
 			(project "STM32XP"
 				(path "/1f1b32b0-2877-4942-afdb-ad5dc4634e8b/f17fb096-3b39-4a0e-96ae-7df73a2ffb98"
-					(reference "R23")
+					(reference "R21")
 					(unit 1)
 				)
@@
 		(on_board yes)
 		(dnp no)
-		(property "Reference" "C26"
+		(property "Reference" "C31"
 			(at 137.16 166.37 90)
 			(effects
@@
 			(project "STM32XP"
 				(path "/1f1b32b0-2877-4942-afdb-ad5dc4634e8b/f17fb096-3b39-4a0e-96ae-7df73a2ffb98"
-					(reference "C26")
+					(reference "C31")
 					(unit 1)
 				)
@@
 		(dnp no)
 		(fields_autoplaced yes)
-		(property "Reference" "U2"
+		(property "Reference" "U7"
 			(at 230.7941 86.36 0)
 			(effects
@@
 			(project "STM32XP"
 				(path "/1f1b32b0-2877-4942-afdb-ad5dc4634e8b/f17fb096-3b39-4a0e-96ae-7df73a2ffb98"
-					(reference "U2")
+					(reference "U7")
 					(unit 1)
 				)
@@
 		(on_board yes)
 		(dnp no)
-		(property "Reference" "U3"
+		(property "Reference" "U6"
 			(at 149.86 160.02 0)
 			(effects
@@
 			(project "STM32XP"
 				(path "/1f1b32b0-2877-4942-afdb-ad5dc4634e8b/f17fb096-3b39-4a0e-96ae-7df73a2ffb98"
-					(reference "U3")
+					(reference "U6")
 					(unit 4)
 				)
@@
 		(on_board yes)
 		(dnp no)
-		(property "Reference" "C21"
+		(property "Reference" "C16"
 			(at 132.08 68.58 90)
 			(effects
@@
 			(project "STM32XP"
 				(path "/1f1b32b0-2877-4942-afdb-ad5dc4634e8b/f17fb096-3b39-4a0e-96ae-7df73a2ffb98"
-					(reference "C21")
+					(reference "C16")
 					(unit 1)
 				)
@@
 		(on_board yes)
 		(dnp no)
-		(property "Reference" "C23"
+		(property "Reference" "C27"
 			(at 132.08 106.68 90)
 			(effects
@@
 			(project "STM32XP"
 				(path "/1f1b32b0-2877-4942-afdb-ad5dc4634e8b/f17fb096-3b39-4a0e-96ae-7df73a2ffb98"
-					(reference "C23")
-					(unit 1)
-				)
+					(reference "C27")
+					(unit 1)
+				)

Commit message: Changed tactile switch model; had to enlarge board and adjust positioning of components; added some 3D models and comments with PNs for further reference; general layout and routing improvements.
Connections:
- net +5VA: now also J3.5 (Pin_5)
- net GND: no longer J3.5 (Pin_5)
Other:
- moved on the sheet: D8

Commit message: Finished PCB design, but needs to be reviewed. Added all components and PNs that were missing or incorrect. Added draft of STM32 EXPLORER logo.
Parts:
- renumbered C13 to C20, C14 to C21, C16 to C22, C17 to C23, C21 to C27, C22 to C28, C23 to C29, C24 to C30, C27 to C33, C28 to C34, C30 to C38, C31 to C39, D8 to D9, R20 to R23, R21 to R24, R22 to R25, R23 to R26, R34 to R33, R35 to R34, R37 to R36, R38 to R37
Changed lines of the file:
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@@
 		(on_board yes)
 		(dnp no)
-		(property "Reference" "R22"
+		(property "Reference" "R25"
 			(at 133.35 78.74 90)
 			(effects
@@
 			(project "STM32XP"
 				(path "/1f1b32b0-2877-4942-afdb-ad5dc4634e8b/f17fb096-3b39-4a0e-96ae-7df73a2ffb98"
-					(reference "R22")
+					(reference "R25")
 					(unit 1)
 				)
@@
 		(on_board yes)
 		(dnp no)
-		(property "Reference" "C28"
+		(property "Reference" "C34"
 			(at 132.08 144.78 90)
 			(effects
@@
 			(project "STM32XP"
 				(path "/1f1b32b0-2877-4942-afdb-ad5dc4634e8b/f17fb096-3b39-4a0e-96ae-7df73a2ffb98"
-					(reference "C28")
+					(reference "C34")
 					(unit 1)
 				)
@@
 		(on_board yes)
 		(dnp no)
-		(property "Reference" "R38"
+		(property "Reference" "R37"
 			(at 120.65 154.94 90)
 			(effects
@@
 			(project "STM32XP"
 				(path "/1f1b32b0-2877-4942-afdb-ad5dc4634e8b/f17fb096-3b39-4a0e-96ae-7df73a2ffb98"
-					(reference "R38")
+					(reference "R37")
 					(unit 1)
 				)
@@
 		(on_board yes)
 		(dnp no)
-		(property "Reference" "C30"
+		(property "Reference" "C38"
 			(at 142.24 128.27 90)
 			(effects
@@
 			(project "STM32XP"
 				(path "/1f1b32b0-2877-4942-afdb-ad5dc4634e8b/f17fb096-3b39-4a0e-96ae-7df73a2ffb98"
-					(reference "C30")
+					(reference "C38")
 					(unit 1)
 				)
@@
 		(on_board yes)
 		(dnp no)
-		(property "Reference" "R37"
+		(property "Reference" "R36"
 			(at 120.65 116.84 90)
 			(effects
@@
 			(project "STM32XP"
 				(path "/1f1b32b0-2877-4942-afdb-ad5dc4634e8b/f17fb096-3b39-4a0e-96ae-7df73a2ffb98"
-					(reference "R37")
+					(reference "R36")
 					(unit 1)
 				)
@@
 		(on_board yes)
 		(dnp no)
-		(property "Reference" "C22"
+		(property "Reference" "C28"
 			(at 67.31 44.45 90)
 			(effects
@@
 			(project "STM32XP"
 				(path "/1f1b32b0-2877-4942-afdb-ad5dc4634e8b/f17fb096-3b39-4a0e-96ae-7df73a2ffb98"
-					(reference "C22")
+					(reference "C28")
 					(unit 1)
 				)
@@
 		(on_board yes)
 		(dnp no)
-		(property "Reference" "R34"
+		(property "Reference" "R33"
 			(at 133.35 116.84 90)
 			(effects
@@
 			(project "STM32XP"
 				(path "/1f1b32b0-2877-4942-afdb-ad5dc4634e8b/f17fb096-3b39-4a0e-96ae-7df73a2ffb98"
-					(reference "R34")
+					(reference "R33")
 					(unit 1)
 				)
@@
 		(on_board yes)
 		(dnp no)
-		(property "Reference" "C24"
+		(property "Reference" "C30"
 			(at 219.71 83.82 90)
 			(effects
@@
 			(project "STM32XP"
 				(path "/1f1b32b0-2877-4942-afdb-ad5dc4634e8b/f17fb096-3b39-4a0e-96ae-7df73a2ffb98"
-					(reference "C24")
+					(reference "C30")
 					(unit 1)
 				)
@@
 		(on_board yes)
 		(dnp no)
-		(property "Reference" "C21"
+		(property "Reference" "C27"
 			(at 58.42 44.45 90)
 			(effects
@@
 			(project "STM32XP"
 				(path "/1f1b32b0-2877-4942-afdb-ad5dc4634e8b/f17fb096-3b39-4a0e-96ae-7df73a2ffb98"
-					(reference "C21")
+					(reference "C27")
 					(unit 1)
 				)
@@
 		(on_board yes)
 		(dnp no)
-		(property "Reference" "R20"
+		(property "Reference" "R23"
 			(at 120.65 78.74 90)
 			(effects
@@
 			(project "STM32XP"
 				(path "/1f1b32b0-2877-4942-afdb-ad5dc4634e8b/f17fb096-3b39-4a0e-96ae-7df73a2ffb98"
-					(reference "R20")
+					(reference "R23")
 					(unit 1)
 				)
@@
 		(on_board yes)
 		(dnp no)
-		(property "Reference" "C17"
+		(property "Reference" "C23"
 			(at 132.08 30.48 90)
 			(effects
@@
 			(project "STM32XP"
 				(path "/1f1b32b0-2877-4942-afdb-ad5dc4634e8b/f17fb096-3b39-4a0e-96ae-7df73a2ffb98"
-					(reference "C17")
+					(reference "C23")
 					(unit 1)
 				)
@@
 		(on_board yes)
 		(dnp no)
-		(property "Reference" "C23"
+		(property "Reference" "C29"
 			(at 219.71 76.2 90)
 			(effects
@@
 			(project "STM32XP"
 				(path "/1f1b32b0-2877-4942-afdb-ad5dc4634e8b/f17fb096-3b39-4a0e-96ae-7df73a2ffb98"
-					(reference "C23")
+					(reference "C29")
 					(unit 1)
 				)
@@
 		(on_board yes)
 		(dnp no)
-		(property "Reference" "C14"
+		(property "Reference" "C21"
 			(at 137.16 52.07 90)
 			(effects
@@
 			(project "STM32XP"
 				(path "/1f1b32b0-2877-4942-afdb-ad5dc4634e8b/f17fb096-3b39-4a0e-96ae-7df73a2ffb98"
-					(reference "C14")
+					(reference "C21")
 					(unit 1)
 				)
@@
 		(on_board yes)
 		(dnp no)
-		(property "Reference" "D8"
+		(property "Reference" "D9"
 			(at 74.93 116.84 0)
 			(effects
@@
 			(project "STM32XP"
 				(path "/1f1b32b0-2877-4942-afdb-ad5dc4634e8b/f17fb096-3b39-4a0e-96ae-7df73a2ffb98"
-					(reference "D8")
+					(reference "D9")
 					(unit 1)
 				)
@@
 		(on_board yes)
 		(dnp no)
-		(property "Reference" "R23"
+		(property "Reference" "R26"
 			(at 133.35 40.64 90)
 			(effects
@@
 			(project "STM32XP"
 				(path "/1f1b32b0-2877-4942-afdb-ad5dc4634e8b/f17fb096-3b39-4a0e-96ae-7df73a2ffb98"
-					(reference "R23")
+					(reference "R26")
 					(unit 1)
 				)
@@
 		(on_board yes)
 		(dnp no)
-		(property "Reference" "C13"
+		(property "Reference" "C20"
 			(at 137.16 90.17 90)
 			(effects
@@
 			(project "STM32XP"
 				(path "/1f1b32b0-2877-4942-afdb-ad5dc4634e8b/f17fb096-3b39-4a0e-96ae-7df73a2ffb98"
-					(reference "C13")
+					(reference "C20")
 					(unit 1)
 				)
@@
 		(on_board yes)
 		(dnp no)
-		(property "Reference" "R35"
+		(property "Reference" "R34"
 			(at 133.35 154.94 90)
 			(effects
@@
 			(project "STM32XP"
 				(path "/1f1b32b0-2877-4942-afdb-ad5dc4634e8b/f17fb096-3b39-4a0e-96ae-7df73a2ffb98"
-					(reference "R35")
+					(reference "R34")
 					(unit 1)
 				)
@@
 		(on_board yes)
 		(dnp no)
-		(property "Reference" "R21"
+		(property "Reference" "R24"
 			(at 120.65 40.64 90)
 			(effects
@@
 			(project "STM32XP"
 				(path "/1f1b32b0-2877-4942-afdb-ad5dc4634e8b/f17fb096-3b39-4a0e-96ae-7df73a2ffb98"
-					(reference "R21")
+					(reference "R24")
 					(unit 1)
 				)
@@
 		(on_board yes)
 		(dnp no)
-		(property "Reference" "C31"
+		(property "Reference" "C39"
 			(at 137.16 166.37 90)
 			(effects
@@
 			(project "STM32XP"
 				(path "/1f1b32b0-2877-4942-afdb-ad5dc4634e8b/f17fb096-3b39-4a0e-96ae-7df73a2ffb98"
-					(reference "C31")
+					(reference "C39")
 					(unit 1)
 				)
@@
 		(on_board yes)
 		(dnp no)
-		(property "Reference" "C16"
+		(property "Reference" "C22"
 			(at 132.08 68.58 90)
 			(effects
@@
 			(project "STM32XP"
 				(path "/1f1b32b0-2877-4942-afdb-ad5dc4634e8b/f17fb096-3b39-4a0e-96ae-7df73a2ffb98"
-					(reference "C16")
+					(reference "C22")
 					(unit 1)
 				)
@@
 		(on_board yes)
 		(dnp no)
-		(property "Reference" "C27"
+		(property "Reference" "C33"
 			(at 132.08 106.68 90)
 			(effects
@@
 			(project "STM32XP"
 				(path "/1f1b32b0-2877-4942-afdb-ad5dc4634e8b/f17fb096-3b39-4a0e-96ae-7df73a2ffb98"
-					(reference "C27")
-					(unit 1)
-				)
+					(reference "C33")
+					(unit 1)
+				)

Commit message: Finished Revision 0 design. Used plugin to make manufacturing files. Purchased 5 units in JLCPCB. Let's wait to check the results! :D
Parts:
- renumbered R23 to R24, R24 to R25, R25 to R26, R26 to R27, R33 to R35, R34 to R36, R36 to R39, R37 to R40
Connections:
- net AA2FB: now reaches C22.1, R24.2, R26.1
- net AA2+: now reaches C20.2, R26.2, U6.5 (+)
- net AA4FB: now reaches C34.1, R36.1, R40.2
- net AA3+: now reaches C38.2, R35.2, U6.10 (+)
- net AA3FB: now reaches C33.1, R35.1, R39.2
- net AA1+: now reaches C21.2, R27.2, U6.3 (+)
- net AA1FB: now reaches C23.1, R25.2, R27.1
- net AA4+: now reaches C39.2, R36.2, U6.12 (+)
Other:
- title: STM32 EXPLORER BOARD -> STM32 EXPLORER BOARD PROTOTYPE
Changed lines of the file:
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@@
 	(paper "A4")
 	(title_block
-		(title "STM32 EXPLORER BOARD")
-		(date "2024-04-26")
+		(title "STM32 EXPLORER BOARD PROTOTYPE")
+		(date "2024-07-21")
 		(rev "00")
 		(company "Mechatronix Lab")
@@
 	(wire
 		(pts
-			(xy 137.16 81.28) (xy 139.7 81.28)
-		)
-		(stroke
-			(width 0)
-			(type default)
-		)
-	)
-	(wire
-		(pts
 			(xy 66.04 128.27) (xy 66.04 125.73)
 		)
@@
 	(wire
 		(pts
+			(xy 139.7 81.28) (xy 137.16 81.28)
+		)
+		(stroke
+			(width 0)
+			(type default)
+		)
+	)
+	(wire
+		(pts
 			(xy 228.6 111.76) (xy 228.6 114.3)
 		)
@@
 		)
 	)
+	(label "AA2FB"
+		(at 127 71.12 0)
+		(fields_autoplaced yes)
+		(effects
+			(font
+				(size 0.635 0.635)
+			)
+			(justify left bottom)
+		)
+	)
+	(label "AA2+"
+		(at 139.7 81.28 0)
+		(fields_autoplaced yes)
+		(effects
+			(font
+				(size 0.635 0.635)
+			)
+			(justify left bottom)
+		)
+	)
+	(label "AA3+"
+		(at 139.7 119.38 0)
+		(fields_autoplaced yes)
+		(effects
+			(font
+				(size 0.635 0.635)
+			)
+			(justify left bottom)
+		)
+	)
+	(label "AA4+"
+		(at 139.7 157.48 0)
+		(fields_autoplaced yes)
+		(effects
+			(font
+				(size 0.635 0.635)
+			)
+			(justify left bottom)
+		)
+	)
+	(label "AA3FB"
+		(at 127 109.22 0)
+		(fields_autoplaced yes)
+		(effects
+			(font
+				(size 0.635 0.635)
+			)
+			(justify left bottom)
+		)
+	)
+	(label "AA1+"
+		(at 139.7 43.18 0)
+		(fields_autoplaced yes)
+		(effects
+			(font
+				(size 0.635 0.635)
+			)
+			(justify left bottom)
+		)
+	)
+	(label "AA4FB"
+		(at 127 147.32 0)
+		(fields_autoplaced yes)
+		(effects
+			(font
+				(size 0.635 0.635)
+			)
+			(justify left bottom)
+		)
+	)
+	(label "AA1FB"
+		(at 127 33.02 0)
+		(fields_autoplaced yes)
+		(effects
+			(font
+				(size 0.635 0.635)
+			)
+			(justify left bottom)
+		)
+	)
 	(global_label "I2C SDA 5V"
 		(shape bidirectional)
@@
 		(on_board yes)
 		(dnp no)
-		(property "Reference" "R25"
+		(property "Reference" "R26"
 			(at 133.35 78.74 90)
 			(effects
@@
 			(project "STM32XP"
 				(path "/1f1b32b0-2877-4942-afdb-ad5dc4634e8b/f17fb096-3b39-4a0e-96ae-7df73a2ffb98"
-					(reference "R25")
+					(reference "R26")
 					(unit 1)
 				)
@@
 		(on_board yes)
 		(dnp no)
-		(property "Reference" "R37"
+		(property "Reference" "R40"
 			(at 120.65 154.94 90)
 			(effects
@@
 			(project "STM32XP"
 				(path "/1f1b32b0-2877-4942-afdb-ad5dc4634e8b/f17fb096-3b39-4a0e-96ae-7df73a2ffb98"
-					(reference "R37")
+					(reference "R40")
 					(unit 1)
 				)
@@
 		(on_board yes)
 		(dnp no)
-		(property "Reference" "R36"
+		(property "Reference" "R39"
 			(at 120.65 116.84 90)
 			(effects
@@
 			(project "STM32XP"
 				(path "/1f1b32b0-2877-4942-afdb-ad5dc4634e8b/f17fb096-3b39-4a0e-96ae-7df73a2ffb98"
-					(reference "R36")
+					(reference "R39")
 					(unit 1)
 				)
@@
 		(on_board yes)
 		(dnp no)
-		(property "Reference" "R33"
+		(property "Reference" "R35"
 			(at 133.35 116.84 90)
 			(effects
@@
 			(project "STM32XP"
 				(path "/1f1b32b0-2877-4942-afdb-ad5dc4634e8b/f17fb096-3b39-4a0e-96ae-7df73a2ffb98"
-					(reference "R33")
+					(reference "R35")
 					(unit 1)
 				)
@@
 		(on_board yes)
 		(dnp no)
-		(property "Reference" "R23"
+		(property "Reference" "R24"
 			(at 120.65 78.74 90)
 			(effects
@@
 			(project "STM32XP"
 				(path "/1f1b32b0-2877-4942-afdb-ad5dc4634e8b/f17fb096-3b39-4a0e-96ae-7df73a2ffb98"
-					(reference "R23")
+					(reference "R24")
 					(unit 1)
 				)
@@
 		(on_board yes)
 		(dnp no)
-		(property "Reference" "R26"
+		(property "Reference" "R27"
 			(at 133.35 40.64 90)
 			(effects
@@
 			(project "STM32XP"
 				(path "/1f1b32b0-2877-4942-afdb-ad5dc4634e8b/f17fb096-3b39-4a0e-96ae-7df73a2ffb98"
-					(reference "R26")
+					(reference "R27")
 					(unit 1)
 				)
@@
 		(on_board yes)
 		(dnp no)
-		(property "Reference" "R34"
+		(property "Reference" "R36"
 			(at 133.35 154.94 90)
 			(effects
@@
 			(project "STM32XP"
 				(path "/1f1b32b0-2877-4942-afdb-ad5dc4634e8b/f17fb096-3b39-4a0e-96ae-7df73a2ffb98"
-					(reference "R34")
+					(reference "R36")
 					(unit 1)
 				)
@@
 		(on_board yes)
 		(dnp no)
-		(property "Reference" "R24"
+		(property "Reference" "R25"
 			(at 120.65 40.64 90)
 			(effects
@@
 			(project "STM32XP"
 				(path "/1f1b32b0-2877-4942-afdb-ad5dc4634e8b/f17fb096-3b39-4a0e-96ae-7df73a2ffb98"
-					(reference "R24")
+					(reference "R25")
 					(unit 1)
 				)
