File: HARDWARE/KICAD/IO.kicad_sch (KiCad schematic)
At the start: 16 parts, among them J1 USB_C_Receptacle_USB2.0_16P, J2 Micro_SD_Card, J3 Conn_01x20_Socket, J4 Conn_01x20_Socket, U5 USBLC6-2SC6

Commit message: Continuing layout and routing.
Parts:
- added C39: 10uF 25V, Capacitor_SMD:C_0805_2012Metric_Pad1.18x1.45mm_HandSolder, symbol Device:C_Small
Connections:
- net +VBUS: now also C39.1
- net GND: now also J1.S1 (SHIELD), J2.9 (SHIELD), C39.2
- net USB OTG ID: now reaches J3.18 (Pin_18)
- no-connect marks 0 -> 4
Other:
- company: (none) -> Mechatronix Lab
- title: (none) -> STM32 EXPLORER BOARD
- moved on the sheet: C16, C17, C18, J1, J2, J3, J4, L2, R11, R19, R20, R21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

Commit message: Trying to solve all errors on DRC, but some depend on finishing other tasks.
Parts:
- renumbered C39 to C12, C16 to C20, C18 to C38, C17 to C39, J4 to J1, J1 to J4, J2 to J5, J3 to J6, L2 to L3, R20 to R33, R11 to R4, R19 to R40, R21 to R43, R9 to R5, R8 to R6
Changed lines of the file:
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@@
 		(on_board yes)
 		(dnp no)
-		(property "Reference" "L2"
+		(property "Reference" "L3"
 			(at 177.8 58.42 0)
 			(effects
@@
 			(project "STM32XP"
 				(path "/1f1b32b0-2877-4942-afdb-ad5dc4634e8b/9b01c2f9-465b-4787-acfa-c3351aa61c9e"
-					(reference "L2")
+					(reference "L3")
 					(unit 1)
 				)
@@
 		(on_board yes)
 		(dnp no)
-		(property "Reference" "J4"
+		(property "Reference" "J1"
 			(at 124.46 93.9799 0)
 			(effects
@@
 			(project "STM32XP"
 				(path "/1f1b32b0-2877-4942-afdb-ad5dc4634e8b/9b01c2f9-465b-4787-acfa-c3351aa61c9e"
-					(reference "J4")
+					(reference "J1")
 					(unit 1)
 				)
@@
 		(on_board yes)
 		(dnp no)
-		(property "Reference" "R21"
+		(property "Reference" "R43"
 			(at 196.85 118.11 90)
 			(effects
@@
 			(project "STM32XP"
 				(path "/1f1b32b0-2877-4942-afdb-ad5dc4634e8b/9b01c2f9-465b-4787-acfa-c3351aa61c9e"
-					(reference "R21")
+					(reference "R43")
 					(unit 1)
 				)
@@
 		(on_board yes)
 		(dnp no)
-		(property "Reference" "C16"
+		(property "Reference" "C20"
 			(at 217.17 49.53 90)
 			(effects
@@
 			(project "STM32XP"
 				(path "/1f1b32b0-2877-4942-afdb-ad5dc4634e8b/9b01c2f9-465b-4787-acfa-c3351aa61c9e"
-					(reference "C16")
+					(reference "C20")
 					(unit 1)
 				)
@@
 		(on_board yes)
 		(dnp no)
-		(property "Reference" "C39"
+		(property "Reference" "C12"
 			(at 217.17 40.64 90)
 			(effects
@@
 			(project "STM32XP"
 				(path "/1f1b32b0-2877-4942-afdb-ad5dc4634e8b/9b01c2f9-465b-4787-acfa-c3351aa61c9e"
-					(reference "C39")
+					(reference "C12")
 					(unit 1)
 				)
@@
 		(on_board yes)
 		(dnp no)
-		(property "Reference" "C17"
+		(property "Reference" "C39"
 			(at 223.52 104.14 90)
 			(effects
@@
 			(project "STM32XP"
 				(path "/1f1b32b0-2877-4942-afdb-ad5dc4634e8b/9b01c2f9-465b-4787-acfa-c3351aa61c9e"
-					(reference "C17")
+					(reference "C39")
 					(unit 1)
 				)
@@
 		(on_board yes)
 		(dnp no)
-		(property "Reference" "J1"
+		(property "Reference" "J4"
 			(at 256.54 43.18 0)
 			(effects
@@
 			(project "STM32XP"
 				(path "/1f1b32b0-2877-4942-afdb-ad5dc4634e8b/9b01c2f9-465b-4787-acfa-c3351aa61c9e"
-					(reference "J1")
+					(reference "J4")
 					(unit 1)
 				)
@@
 		(on_board yes)
 		(dnp no)
-		(property "Reference" "R11"
+		(property "Reference" "R4"
 			(at 90.17 82.55 90)
 			(effects
@@
 			(project "STM32XP"
 				(path "/1f1b32b0-2877-4942-afdb-ad5dc4634e8b/9b01c2f9-465b-4787-acfa-c3351aa61c9e"
-					(reference "R11")
+					(reference "R4")
 					(unit 1)
 				)
@@
 		(on_board yes)
 		(dnp no)
-		(property "Reference" "R9"
+		(property "Reference" "R5"
 			(at 90.17 80.01 90)
 			(effects
@@
 			(project "STM32XP"
 				(path "/1f1b32b0-2877-4942-afdb-ad5dc4634e8b/9b01c2f9-465b-4787-acfa-c3351aa61c9e"
-					(reference "R9")
+					(reference "R5")
 					(unit 1)
 				)
@@
 		(on_board yes)
 		(dnp no)
-		(property "Reference" "R19"
+		(property "Reference" "R40"
 			(at 173.99 138.43 90)
 			(effects
@@
 			(project "STM32XP"
 				(path "/1f1b32b0-2877-4942-afdb-ad5dc4634e8b/9b01c2f9-465b-4787-acfa-c3351aa61c9e"
-					(reference "R19")
+					(reference "R40")
 					(unit 1)
 				)
@@
 		(on_board yes)
 		(dnp no)
-		(property "Reference" "J3"
+		(property "Reference" "J6"
 			(at 27.94 93.9799 0)
 			(effects
@@
 			(project "STM32XP"
 				(path "/1f1b32b0-2877-4942-afdb-ad5dc4634e8b/9b01c2f9-465b-4787-acfa-c3351aa61c9e"
-					(reference "J3")
+					(reference "J6")
 					(unit 1)
 				)
@@
 		(on_board yes)
 		(dnp no)
-		(property "Reference" "C18"
+		(property "Reference" "C38"
 			(at 223.52 113.03 90)
 			(effects
@@
 			(project "STM32XP"
 				(path "/1f1b32b0-2877-4942-afdb-ad5dc4634e8b/9b01c2f9-465b-4787-acfa-c3351aa61c9e"
-					(reference "C18")
+					(reference "C38")
 					(unit 1)
 				)
@@
 		(on_board yes)
 		(dnp no)
-		(property "Reference" "R20"
+		(property "Reference" "R33"
 			(at 204.47 110.49 90)
 			(effects
@@
 			(project "STM32XP"
 				(path "/1f1b32b0-2877-4942-afdb-ad5dc4634e8b/9b01c2f9-465b-4787-acfa-c3351aa61c9e"
-					(reference "R20")
+					(reference "R33")
 					(unit 1)
 				)
@@
 		(dnp no)
 		(fields_autoplaced yes)
-		(property "Reference" "J2"
+		(property "Reference" "J5"
 			(at 241.935 113.03 0)
 			(effects
@@
 			(project "STM32XP"
 				(path "/1f1b32b0-2877-4942-afdb-ad5dc4634e8b/9b01c2f9-465b-4787-acfa-c3351aa61c9e"
-					(reference "J2")
+					(reference "J5")
 					(unit 1)
 				)
@@
 		(on_board yes)
 		(dnp no)
-		(property "Reference" "R8"
+		(property "Reference" "R6"
 			(at 90.17 77.47 90)
 			(effects
@@
 			(project "STM32XP"
 				(path "/1f1b32b0-2877-4942-afdb-ad5dc4634e8b/9b01c2f9-465b-4787-acfa-c3351aa61c9e"
-					(reference "R8")
-					(unit 1)
-				)
+					(reference "R6")
+					(unit 1)
+				)

Commit message: Changed tactile switch model; had to enlarge board and adjust positioning of components; added some 3D models and comments with PNs for further reference; general layout and routing improvements.
Parts:
- added R50: 10K 1%, Resistor_SMD:R_0603_1608Metric_Pad0.98x0.95mm_HandSolder, symbol Device:R_US
Connections:
- net SD DAT1 SPI is gone; now on net SPI SCK: J5.8 (DAT1), R43.1
- net +3.3V: now also R50.2
- new net SD CARD ~{IN}: R50.1
Other:
- note added: "PIN 9 - CARD DETECTOR"
- note added: "WE 629722000214 https://www.we-online.com/en/components/products/WR-COM_USB_20_TYPE_C_RECEPTACLE_HORIZONTAL_SMT#629722000214"
- note added: "WE 693071020811 https://www.we-online.com/en/components/products/CRD_SD_MICRO_PUSH_AND_PULL_8_PINS#693071020811"
- moved on the sheet: R40

Commit message: More improvements. Added 3D models. Added legends.
Connections:
- net SPI SCK: no longer J5.8 (DAT1), R43.1
- new net SD DAT1 SPI: J5.8 (DAT1), R43.1
Other:
- note added: "WE 744232090 https://www.we-online.com/en/components/products/WE-CNSW#/articles/WE-CNSW-1206"
- note added: "WE Filter Bag USB 2.0 Type A EMC https://www.we-online.com/en/components/products/EMC_FILTER_BAGS_STICKS_USB_2_0_FILTER_BAG#744232090"
Changed lines of the file:
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@@
-	)
-	(junction
-		(at 199.39 134.62)
-		(diameter 0)
-		(color 0 0 0 0)
 	)
 	(junction
@@
 	(wire
 		(pts
-			(xy 199.39 134.62) (xy 218.44 134.62)
+			(xy 196.85 134.62) (xy 218.44 134.62)
 		)
 		(stroke
@@
 	(wire
 		(pts
+			(xy 199.39 121.92) (xy 199.39 142.24)
+		)
+		(stroke
+			(width 0)
+			(type default)
+		)
+	)
+	(wire
+		(pts
 			(xy 241.3 46.99) (xy 238.76 46.99)
 		)
@@
 	(wire
 		(pts
-			(xy 199.39 134.62) (xy 199.39 142.24)
-		)
-		(stroke
-			(width 0)
-			(type default)
-		)
-	)
-	(wire
-		(pts
 			(xy 231.14 76.2) (xy 231.14 64.77)
 		)
@@
 	(wire
 		(pts
-			(xy 196.85 134.62) (xy 199.39 134.62)
-		)
-		(stroke
-			(width 0)
-			(type default)
-		)
-	)
-	(wire
-		(pts
 			(xy 191.77 137.16) (xy 191.77 114.3)
 		)
@@
 		(pts
 			(xy 196.85 132.08) (xy 196.85 134.62)
-		)
-		(stroke
-			(width 0)
-			(type default)
-		)
-	)
-	(wire
-		(pts
-			(xy 199.39 121.92) (xy 199.39 134.62)
 		)
 		(stroke
@@
 			)
 			(justify left)
+		)
+	)
+	(text "WE Filter Bag USB 2.0 Type A EMC\nhttps://www.we-online.com/en/components/products/EMC_FILTER_BAGS_STICKS_USB_2_0_FILTER_BAG#744232090"
+		(exclude_from_sim no)
+		(at 179.07 46.99 0)
+		(effects
+			(font
+				(size 1.27 1.27)
+			)
+			(justify right)
 		)
 	)
@@
 		)
 	)
+	(text "WE 744232090\nhttps://www.we-online.com/en/components/products/WE-CNSW#/articles/WE-CNSW-1206"
+		(exclude_from_sim no)
+		(at 179.07 54.61 0)
+		(effects
+			(font
+				(size 1.27 1.27)
+			)
+			(justify right)
+		)
+	)

Commit message: Improvements to layout. Fixed most of errors and warnings. Added correct footprint for Micro SD socket. Added markings and symbols to legend.
Parts:
- removed J5: Micro_SD_Card, Connector_Card:microSD_HC_Wuerth_693072010801, symbol Connector:Micro_SD_Card
- added J5: MICRO SD, STM32XP:WE 693071020811, symbol STM32XP:WE_693071020811
Connections:
- net +3.3V: now also J5.4 (VDD)
- net GND: now also J5.10 (SHIELD), J5.11 (SHIELD), J5.12 (SHIELD), J5.13 (SHIELD), J5.6 (VSS)
- net SD CARD ~{IN}: now also J5.9 (DET)
- net SD DAT0 SPI: now also J5.7 (DAT0)
- net SD DAT1 SPI: now also J5.8 (DAT1)
- net SD DAT2 SPI: now also J5.1 (DAT2)
- net SPI MOSI: now also J5.3 (CMD)
- net SPI NSS: now also J5.2 (DAT3/CD)
- net SPI SCK: now also J5.5 (CLK)
Other:
- note removed: "PIN 9 - CARD DETECTOR"
- note removed: "WE 693071020811 https://www.we-online.com/en/components/products/CRD_SD_MICRO_PUSH_AND_PULL_8_PINS#693071020811"
- moved on the sheet: C12, C20, C38, C39, J4, L3, R33, R40, R43, R50, U5

Commit message: Finished PCB design, but needs to be reviewed. Added all components and PNs that were missing or incorrect. Added draft of STM32 EXPLORER logo.
Parts:
- removed L3: CMF3216F-900-2P-T, Inductor_SMD:L_CommonModeChoke_TDK_ACM2520-2P, symbol Device:EMI_Filter_LL_1423
- added C16: 680nF 16V, Capacitor_SMD:C_0603_1608Metric_Pad1.08x0.95mm_HandSolder, symbol Device:C_Small
- added FB2, FB3: 600R, Inductor_SMD:L_0603_1608Metric_Pad1.05x0.95mm_HandSolder, symbol Device:L_Small
- added L2: 744232090, STM32XP:WE 744232090, symbol STM32XP:WE_744232090
- added TP8: +VBUS, TestPoint:TestPoint_Keystone_5000-5004_Miniature, symbol Connector:TestPoint
- J4: value USB_C_Receptacle_USB2.0_16P -> USB TYPE C; Manufacturer (none) -> Würth Elektronik; PN (none) -> WE 629722000214
- renumbered C12 to C19, C20 to C26, C39 to C40, C38 to C45, R33 to R38, R40 to R41, R43 to R42, R50 to R45
Connections:
- net +VBUS: now also FB3.2, TP8.1
- net GND: now also C16.2
- net USB D+: now also L2.4
- net USB D-: now also L2.1
- net USB FILTERED D+: now also L2.3
- net USB FILTERED D-: now also L2.2
- new net +VBUSF: FB2.1
- new net USB FILTERED POWER: C16.1, FB2.2, FB3.1
Other:
- note removed: "WE 629722000214 https://www.we-online.com/en/components/products/WR-COM_USB_20_TYPE_C_RECEPTACLE_HORIZONTAL_SMT#629722000214"
- note removed: "WE 744232090 https://www.we-online.com/en/components/products/WE-CNSW#/articles/WE-CNSW-1206"
- note removed: "WE Filter Bag USB 2.0 Type A EMC https://www.we-online.com/en/components/products/EMC_FILTER_BAGS_STICKS_USB_2_0_FILTER_BAG#744232090"
- moved on the sheet: C19, C26, J1, J4, J6, R4, R5, R6, R7, U5

Commit message: Finished Revision 0 design. Used plugin to make manufacturing files. Purchased 5 units in JLCPCB. Let's wait to check the results! :D
Parts:
- added R23, R28: 5.1K 1%, Resistor_SMD:R_0603_1608Metric_Pad0.98x0.95mm_HandSolder, symbol Device:R_US
- added R37: 10K 1%, Resistor_SMD:R_0603_1608Metric_Pad0.98x0.95mm_HandSolder, symbol Device:R_US
- renumbered R38 to R41, R41 to R44, R42 to R45, R45 to R48
Connections:
- net +3.3V: now also R37.2
- net GND: now also R23.1, R28.1
- net SPI NSS: now also R37.1
- net SWDIO CONN: now reaches J1.3 (Pin_3), R7.2
- net SWCLK CONN: now reaches J1.4 (Pin_4), R6.2
- net SWO CONN: now reaches J1.5 (Pin_5), R5.2
- net NRST CONN: now reaches J1.6 (Pin_6), R4.2
- net USB CC1: now reaches J4.A5 (CC1)
- net USB CC1: now also R28.2
- net USB CC2: now reaches J4.B5 (CC2)
- net USB CC2: now also R23.2
- no-connect marks 4 -> 2
Other:
- title: STM32 EXPLORER BOARD -> STM32 EXPLORER BOARD PROTOTYPE
- moved on the sheet: C16, C19, C26, C40, C45, FB2, FB3, J1, J4, J5, J6, L2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
