File: HARDWARE/KICAD/MCU.kicad_sch (KiCad schematic)
At the start: 38 parts, among them Q2 2N7002, Q3 2N7002, SW3 RST, U1 STM32F411RETx, Y1 32.768kHz, Y2 8MHz xpF

Commit message: Continuing layout and routing.
Other:
- company: (none) -> Mechatronix Lab
- title: (none) -> STM32 EXPLORER BOARD
Changed lines of the file:
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@@
 	(generator_version "8.0")
 	(paper "A4")
+	(title_block
+		(title "STM32 EXPLORER BOARD")
+		(date "2024-04-26")
+		(rev "00")
+		(company "Mechatronix Lab")
+		(comment 1 "Eng. André A. M. Araújo")
+	)
 	(junction
 		(at 109.22 149.86)

Commit message: Trying to solve all errors on DRC, but some depend on finishing other tasks.
Parts:
- added TP12: +VCORE, TestPoint:TestPoint_Keystone_5000-5004_Miniature, symbol Connector:TestPoint
- renumbered C8 to C10, C1 to C11, C2 to C18, C10 to C19, C9 to C25, C13 to C26, C5 to C29, C6 to C32, C7 to C33, C4 to C34, C3 to C35, C14 to C36, C11 to C37, L1 to L4, Q2 to Q1, Q3 to Q2, R5 to R11, R4 to R12, R3 to R13, R6 to R14, R1 to R15, R12 to R16, R13 to R17, R41 to R18, R40 to R19, R2 to R25, R33 to R27, R32 to R29, R10 to R30, R30 to R32, R16 to R36, R17 to R39, R18 to R42, SW3 to SW1, U1 to U8
Connections:
- net VCORE renamed +VCORE
- net +VCORE: now also TP12.1
Other:
- moved on the sheet: C36, C37

Commit message: Changed tactile switch model; had to enlarge board and adjust positioning of components; added some 3D models and comments with PNs for further reference; general layout and routing improvements.
Parts:
- added C40, C41: 100nF 50V, Capacitor_SMD:C_0603_1608Metric_Pad1.08x0.95mm_HandSolder, symbol Device:C_Small
- added C42, C43: 10pF 50V, Capacitor_SMD:C_0603_1608Metric_Pad1.08x0.95mm_HandSolder, symbol Device:C_Small
- SW1: footprint Button_Switch_SMD:SW_SPST_CK_KXT3 -> Button_Switch_SMD:SW_Push_1P1T_NO_CK_KSC6xxJ
Connections:
- net +3.3V: now also C40.2
- net +5V: now also C41.1
- net GND: now also C40.1, C41.2, C42.1, C43.1
- net at U8.3 (PC14), Y1.2: now also C42.2
- net at U8.4 (PC15), Y1.1: now also C43.2
- net SD CARD ~{IN}: now reaches U8.51 (PC10)
Other:
- note added: "SEIKO SC-32S32.768kHz20PPM12.5pF https://www.lcsc.com/datasheet/lcsc_datasheet_1811151435_Seiko-SC-32S32-768kHz20PPM12-5pF_C97606.pdf SEIKO EPSON Q13FC13500004 https://www.lcsc.com/datasheet/lcsc_datasheet_2404180925_Seiko-Epson-Q13FC13500004_C32346.pdf"
- note added: "WE 830055295 12 MHz 20 ppm 18pF https://www.we-online.com/en/components/products/WE-XTAL#/articles/CFPX-180"
- moved on the sheet: C19, C25, C26, C37, Q1, Q2, R11, R14, R15, R18, R19, R25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

Commit message: Finished PCB design, but needs to be reviewed. Added all components and PNs that were missing or incorrect. Added draft of STM32 EXPLORER logo.
Parts:
- renumbered C40 to C11, C43 to C14, C42 to C15, C10 to C17, C11 to C18, C18 to C24, C19 to C25, C25 to C31, C26 to C32, C29 to C35, C32 to C36, C33 to C37, C34 to C41, C35 to C42, C36 to C43, C37 to C44, C41 to C5, L4 to L3, Q1 to Q2, Q2 to Q3, R18 to R11, R11 to R12, R19 to R14, R14 to R15, R12 to R16, R13 to R17, R15 to R18, R16 to R19, R17 to R20, R25 to R27, R27 to R28, R36 to R35, R42 to R40, TP12 to TP11

Commit message: Finished Revision 0 design. Used plugin to make manufacturing files. Purchased 5 units in JLCPCB. Let's wait to check the results! :D
Parts:
- added TP10: +3.3VA, TestPoint:TestPoint_Keystone_5000-5004_Miniature, symbol Connector:TestPoint
- added TP15: PD2, TestPoint:TestPoint_THTPad_D1.0mm_Drill0.5mm, symbol Connector:TestPoint
- added TP16: PC11, TestPoint:TestPoint_THTPad_D1.0mm_Drill0.5mm, symbol Connector:TestPoint
- added TP17: PC12, TestPoint:TestPoint_THTPad_D1.0mm_Drill0.5mm, symbol Connector:TestPoint
- added TP18: PB5, TestPoint:TestPoint_THTPad_D1.0mm_Drill0.5mm, symbol Connector:TestPoint
- added TP19: PB4, TestPoint:TestPoint_THTPad_D1.0mm_Drill0.5mm, symbol Connector:TestPoint
- added TP20: PC13, TestPoint:TestPoint_THTPad_D1.0mm_Drill0.5mm, symbol Connector:TestPoint
- added TP21: PB10, TestPoint:TestPoint_THTPad_D1.0mm_Drill0.5mm, symbol Connector:TestPoint
- Y2: value 8MHz xpF -> 12MHz 20Pppm 18pF
- renumbered R27 to R29, R28 to R30, R29 to R31, R30 to R32, R31 to R33, R32 to R34, R35 to R38, R39 to R42, R40 to R43, TP11 to TP12
Connections:
- net +3.3VA: now also TP10.1
- net +5V: now also C5.2; no longer C5.1
- net GND: now also C5.1; no longer C5.2
- net HSE OUT: now reaches C31.2, R29.1, Y2.1
- net BOOT0: now reaches R18.2, U8.60 (BOOT0)
- net PH0: now reaches C25.2, U8.5 (PH0), Y2.3
- net PC13: now reaches U8.2 (PC13)
- net PC13: now also TP20.1
- net PB10: now reaches U8.29 (PB10)
- net PB10: now also TP21.1
- net LSE IN: now reaches C15.2, U8.3 (PC14), Y1.2
- net LSE OUT: now reaches C14.2, U8.4 (PC15), Y1.1
- net PC11: now reaches U8.52 (PC11)
- net PC11: now also TP16.1
- net PC12: now reaches U8.53 (PC12)
- net PC12: now also TP17.1
- net PD2: now reaches U8.54 (PD2)
- net PD2: now also TP15.1
- net PB4: now reaches U8.56 (PB4)
- net PB4: now also TP19.1
- net PB5: now reaches U8.57 (PB5)
- net PB5: now also TP18.1
- net PB6: now reaches R19.1, U8.58 (PB6)
- net PH1: now reaches R29.2, U8.6 (PH1)
- net MCU PA15 renamed PA15
- net MCU PB12 SPI renamed PB12 SPI
- net MCU PB13 SPI renamed PB13 SPI
- net MCU PB15 SPI renamed PB15 SPI
- net MCU PB8 renamed PB8
- net MCU PB9 renamed PB9
Other:
- note added: "FB4"
- note removed: "CHECK IF USB PULLUPS ARE NECESSARY"
- title: STM32 EXPLORER BOARD -> STM32 EXPLORER BOARD PROTOTYPE
- moved on the sheet: C11, C17, C25, C31, C5, Q2, Q3, R11, R12, R14, R15, Y2
