File: HARDWARE/KICAD/POWER.kicad_sch (KiCad schematic)
At the start: 21 parts, among them J5 Jack-DC, U4 AMS1117-3.3, U7 AMS1117-5.0, U8 AP3012

Commit message: Continuing layout and routing.
Parts:
- added D5, D6, D7, D8, D9: LED, LED_SMD:LED_0603_1608Metric_Pad1.05x0.95mm_HandSolder, symbol Device:LED
- added R45, R46: 10K 1%, Resistor_SMD:R_0603_1608Metric_Pad0.98x0.95mm_HandSolder, symbol Device:R_US
- added R47, R48, R49: 1K 1%, Resistor_SMD:R_0603_1608Metric_Pad0.98x0.95mm_HandSolder, symbol Device:R_US
- added TP1: +3.3V, TestPoint:TestPoint_Keystone_5000-5004_Miniature, symbol Connector:TestPoint
- added TP10, TP11, TP9: GND, TestPoint:TestPoint_Keystone_5000-5004_Miniature, symbol Connector:TestPoint
- added TP2: +5VA, TestPoint:TestPoint_Keystone_5000-5004_Miniature, symbol Connector:TestPoint
- added TP3: +9V, TestPoint:TestPoint_Keystone_5000-5004_Miniature, symbol Connector:TestPoint
- added TP4: +VSEL, TestPoint:TestPoint_Keystone_5000-5004_Miniature, symbol Connector:TestPoint
- added TP5: +VEXT, TestPoint:TestPoint_Keystone_5000-5004_Miniature, symbol Connector:TestPoint
- added TP6: +3VBAT, TestPoint:TestPoint_Keystone_5000-5004_Miniature, symbol Connector:TestPoint
- added TP7: +5V, TestPoint:TestPoint_Keystone_5000-5004_Miniature, symbol Connector:TestPoint
- added TP8: +VBUS, TestPoint:TestPoint_Keystone_5000-5004_Miniature, symbol Connector:TestPoint
Connections:
- net +3.3V: now also D7.2 (A), TP1.1
- net +3VBAT: now also TP6.1
- net +5V: now also D8.2 (A), TP7.1
- net +5VA: now also TP2.1
- net +9V: now also D6.2 (A), TP3.1
- net +VBUS: now also D5.2 (A), TP8.1
- net +VEXT: now also D9.2 (A), TP5.1
- net +VSEL: now also TP4.1
- net GND: now also R45.1, R46.1, R47.1, R48.1, R49.1, TP10.1, TP11.1, TP9.1
- new net: D7.1 (K), R47.2
- new net: D6.1 (K), R46.2
- new net: D9.1 (K), R49.2
- new net: D5.1 (K), R45.2
- new net: D8.1 (K), R48.2
Other:
- company: (none) -> Mechatronix Lab
- title: (none) -> STM32 EXPLORER BOARD
- moved on the sheet: BT1, C12, C31, C34, C35, C36, C37, C38, D3, D4, J5, JP1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

Commit message: Added new PNs for some components. Overall improvements in schematic and layout.
Parts:
- removed D3: 1N5819WS, Diode_SMD:D_SOD-323, symbol Diode:1N5819WS
- removed L3: L_Small, Inductor_SMD:L_0603_1608Metric_Pad1.05x0.95mm_HandSolder, symbol Device:L_Small
- added D3: STPS1L40-Y, Diode_SMD:D_SOD-123, symbol STM32XP:STPS1L40-Y
- added L3: 10uH, STM32XP:WE 74404024100, symbol STM32XP:WE_74404024100
Connections:
- net BOOST IN: now also L3.1
- net BOOST OUT: now also D3.1 (K)
- net BOOST SW: now also D3.2 (A), L3.2
Changed lines of the file:
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@@
 	)
 	(junction
-		(at 127 73.66)
+		(at 241.3 134.62)
 		(diameter 0)
 		(color 0 0 0 0)
 	)
 	(junction
-		(at 241.3 134.62)
+		(at 101.6 121.92)
 		(diameter 0)
 		(color 0 0 0 0)
 	)
 	(junction
-		(at 101.6 121.92)
+		(at 127 73.66)
 		(diameter 0)
 		(color 0 0 0 0)
@@
 	(wire
 		(pts
+			(xy 127 73.66) (xy 135.89 73.66)
+		)
+		(stroke
+			(width 0)
+			(type default)
+		)
+	)
+	(wire
+		(pts
 			(xy 114.3 134.62) (xy 127 134.62)
 		)
@@
 	(wire
 		(pts
-			(xy 127 73.66) (xy 137.16 73.66)
-		)
-		(stroke
-			(width 0)
-			(type default)
-		)
-	)
-	(wire
-		(pts
 			(xy 190.5 71.12) (xy 190.5 73.66)
 		)
@@
 	(wire
 		(pts
-			(xy 142.24 73.66) (xy 152.4 73.66)
+			(xy 143.51 73.66) (xy 152.4 73.66)
 		)
 		(stroke
@@
 	)
 	(symbol
-		(lib_id "Diode:1N5819WS")
-		(at 158.75 73.66 0)
-		(mirror y)
+		(lib_id "Device:LED")
+		(at 139.7 128.27 90)
 		(unit 1)
 		(exclude_from_sim no)
@@
 		(on_board yes)
 		(dnp no)
-		(property "Reference" "D3"
-			(at 158.75 71.12 0)
+		(property "Reference" "D7"
+			(at 134.62 127 90)
 			(effects
 				(font
 					(size 1.27 1.27)
 				)
+				(justify right)
 			)
 		)
-		(property "Value" "1N5819WS"
-			(at 159.0675 76.2 0)
+		(property "Value" "LED"
+			(at 133.35 129.54 90)
 			(effects
 				(font
 					(size 1.27 1.27)
 				)
+				(justify right)
 			)
 		)
-		(property "Footprint" "Diode_SMD:D_SOD-323"
-			(at 158.75 78.105 0)
+		(property "Footprint" "LED_SMD:LED_0603_1608Metric_Pad1.05x0.95mm_HandSolder"
+			(at 139.7 128.27 0)
 			(effects
 				(font
@@
 			)
 		)
-		(property "Datasheet" "https://datasheet.lcsc.com/lcsc/2204281430_Guangdong-Hottech-1N5819WS_C191023.pdf"
-			(at 158.75 73.66 0)
+		(property "Datasheet" "~"
+			(at 139.7 128.27 0)
 			(effects
 				(font
@@
 			)
 		)
-		(property "Description" "40V 600mV@1A 1A SOD-323 Schottky Barrier Diodes, SOD-323"
-			(at 158.75 73.66 0)
+		(property "Description" "Light emitting diode"
+			(at 139.7 128.27 0)
 			(effects
 				(font
@@
 			)
 		)
-		(pin "1"
-		)
 		(pin "2"
 		)
+		(pin "1"
+		)
 		(instances
 			(project "STM32XP"
 				(path "/1f1b32b0-2877-4942-afdb-ad5dc4634e8b/c5d90769-1771-42f2-86df-749a2f175e63"
-					(reference "D3")
+					(reference "D7")
 					(unit 1)
 				)
@@
 	)
 	(symbol
-		(lib_id "Device:LED")
-		(at 139.7 128.27 90)
+		(lib_id "STM32XP:WE_74404024100")
+		(at 139.7 73.66 90)
 		(unit 1)
 		(exclude_from_sim no)
@@
 		(on_board yes)
 		(dnp no)
-		(property "Reference" "D7"
-			(at 134.62 127 90)
+		(property "Reference" "L3"
+			(at 139.7 71.12 90)
 			(effects
 				(font
 					(size 1.27 1.27)
 				)
-				(justify right)
 			)
 		)
-		(property "Value" "LED"
-			(at 133.35 129.54 90)
+		(property "Value" "10uH"
+			(at 139.7 74.93 90)
 			(effects
 				(font
 					(size 1.27 1.27)
 				)
-				(justify right)
 			)
 		)
-		(property "Footprint" "LED_SMD:LED_0603_1608Metric_Pad1.05x0.95mm_HandSolder"
-			(at 139.7 128.27 0)
+		(property "Footprint" "STM32XP:WE 74404024100"
+			(at 139.7 73.66 0)
 			(effects
 				(font
@@
 			)
 		)
-		(property "Datasheet" "~"
-			(at 139.7 128.27 0)
+		(property "Datasheet" "https://www.we-online.com/components/products/datasheet/74404024100.pdf"
+			(at 139.7 73.66 0)
 			(effects
 				(font
@@
 			)
 		)
-		(property "Description" "Light emitting diode"
-			(at 139.7 128.27 0)
+		(property "Description" "SEMI SHIELDED POWER INDUCTOR WE WÜRTH ELEKTRONIK WE-LQS"
+			(at 139.7 73.66 0)
 			(effects
 				(font
@@
 			(project "STM32XP"
 				(path "/1f1b32b0-2877-4942-afdb-ad5dc4634e8b/c5d90769-1771-42f2-86df-749a2f175e63"
-					(reference "D7")
+					(reference "L3")
 					(unit 1)
 				)
@@
 	)
 	(symbol
+		(lib_id "STM32XP:STPS1L40-Y")
+		(at 158.75 73.66 180)
+		(unit 1)
+		(exclude_from_sim no)
+		(in_bom yes)
+		(on_board yes)
+		(dnp no)
+		(property "Reference" "D3"
+			(at 158.75 71.12 0)
+			(effects
+				(font
+					(size 1.27 1.27)
+				)
+			)
+		)
+		(property "Value" "STPS1L40-Y"
+			(at 158.75 76.2 0)
+			(effects
+				(font
+					(size 1.27 1.27)
+				)
+			)
+		)
+		(property "Footprint" "Diode_SMD:D_SOD-123"
+			(at 158.75 73.66 0)
+			(effects
+				(font
+					(size 1.27 1.27)
+				)
+				(hide yes)
+			)
+		)
+		(property "Datasheet" "https://www.st.com/resource/en/datasheet/stps1l40-y.pdf"
+			(at 158.75 73.66 0)
+			(effects
+				(font
+					(size 1.27 1.27)
+				)
+				(hide yes)
+			)
+		)
+		(property "Description" "1A 40V 0.37V"
+			(at 158.75 73.66 0)
+			(effects
+				(font
+					(size 1.27 1.27)
+				)
+				(hide yes)
+			)
+		)
+		(pin "2"
+		)
+		(pin "1"
+		)
+		(instances
+			(project "STM32XP"
+				(path "/1f1b32b0-2877-4942-afdb-ad5dc4634e8b/c5d90769-1771-42f2-86df-749a2f175e63"
+					(reference "D3")
+					(unit 1)
+				)
+			)
+		)
+	)
+	(symbol
 		(lib_id "Device:C_Small")
 		(at 177.8 86.36 180)
@@
 	)
 	(symbol
-		(lib_id "Device:L_Small")
-		(at 139.7 73.66 90)
-		(unit 1)
-		(exclude_from_sim no)
-		(in_bom yes)
-		(on_board yes)
-		(dnp no)
-		(fields_autoplaced yes)
-		(property "Reference" "L3"
-			(at 139.7 68.58 90)
-			(effects
-				(font
-					(size 1.27 1.27)
-				)
-			)
-		)
-		(property "Value" "L_Small"
-			(at 139.7 71.12 90)
-			(effects
-				(font
-					(size 1.27 1.27)
-				)
-			)
-		)
-		(property "Footprint" "Inductor_SMD:L_0603_1608Metric_Pad1.05x0.95mm_HandSolder"
-			(at 139.7 73.66 0)
-			(effects
-				(font
-					(size 1.27 1.27)
-				)
-				(hide yes)
-			)
-		)
-		(property "Datasheet" "~"
-			(at 139.7 73.66 0)
-			(effects
-				(font
-					(size 1.27 1.27)
-				)
-				(hide yes)
-			)
-		)
-		(property "Description" "Inductor, small symbol"
-			(at 139.7 73.66 0)
-			(effects
-				(font
-					(size 1.27 1.27)
-				)
-				(hide yes)
-			)
-		)
-		(pin "1"
-		)
-		(pin "2"
-		)
-		(instances
-			(project "STM32XP"
-				(path "/1f1b32b0-2877-4942-afdb-ad5dc4634e8b/c5d90769-1771-42f2-86df-749a2f175e63"
-					(reference "L3")
-					(unit 1)
-				)
-			)
-		)
-	)
-	(symbol
 		(lib_id "Device:R_US")
 		(at 121.92 80.01 180)
@@
 		(dnp no)
 		(property "Reference" "U8"
-			(at 139.7 77.47 0)
+			(at 133.35 77.47 0)
 			(effects
 				(font

Commit message: Continuing layout and routing.
Other:
- note removed: "WE 74404024100 https://www.we-online.com/components/products/datasheet/74404024100.pdf"
- moved on the sheet: TP3
Changed lines of the file:
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@@
 	)
 	(junction
-		(at 190.5 71.12)
+		(at 190.5 66.04)
 		(diameter 0)
 		(color 0 0 0 0)
@@
 	)
 	(junction
+		(at 190.5 73.66)
+		(diameter 0)
+		(color 0 0 0 0)
+	)
+	(junction
 		(at 114.3 134.62)
 		(diameter 0)
@@
 	)
 	(junction
-		(at 190.5 73.66)
-		(diameter 0)
-		(color 0 0 0 0)
-	)
-	(junction
 		(at 101.6 73.66)
 		(diameter 0)
@@
 	(wire
 		(pts
-			(xy 190.5 71.12) (xy 193.04 71.12)
+			(xy 190.5 66.04) (xy 193.04 66.04)
 		)
 		(stroke
@@
 	(wire
 		(pts
-			(xy 35.56 104.14) (xy 38.1 104.14)
+			(xy 190.5 66.04) (xy 190.5 73.66)
 		)
 		(stroke
@@
 	(wire
 		(pts
-			(xy 190.5 71.12) (xy 190.5 73.66)
+			(xy 35.56 104.14) (xy 38.1 104.14)
 		)
 		(stroke
@@
 	(wire
 		(pts
-			(xy 190.5 73.66) (xy 190.5 76.2)
-		)
-		(stroke
-			(width 0)
-			(type default)
-		)
-	)
-	(wire
-		(pts
 			(xy 165.1 83.82) (xy 165.1 86.36)
 		)
@@
 	(wire
 		(pts
-			(xy 190.5 73.66) (xy 187.96 73.66)
+			(xy 187.96 73.66) (xy 190.5 73.66)
 		)
 		(stroke
@@
 	(wire
 		(pts
-			(xy 190.5 68.58) (xy 190.5 71.12)
+			(xy 190.5 63.5) (xy 190.5 66.04)
 		)
 		(stroke
@@
 	(wire
 		(pts
-			(xy 76.2 40.64) (xy 76.2 73.66)
+			(xy 190.5 73.66) (xy 190.5 76.2)
 		)
 		(stroke
@@
 		)
 	)
-	(text "WE 74404024100\nhttps://www.we-online.com/components/products/datasheet/74404024100.pdf"
-		(exclude_from_sim no)
-		(at 152.4 62.23 0)
-		(effects
-			(font
-				(size 1.27 1.27)
-			)
+	(wire
+		(pts
+			(xy 76.2 40.64) (xy 76.2 73.66)
+		)
+		(stroke
+			(width 0)
+			(type default)
 		)
 	)
@@
 	(symbol
 		(lib_id "Connector:TestPoint")
-		(at 193.04 71.12 270)
+		(at 193.04 66.04 270)
 		(unit 1)
 		(exclude_from_sim no)
@@
 		(fields_autoplaced yes)
 		(property "Reference" "TP3"
-			(at 198.12 69.8499 90)
+			(at 198.12 64.7699 90)
 			(effects
 				(font
@@
 		)
 		(property "Value" "+9V"
-			(at 198.12 72.3899 90)
+			(at 198.12 67.3099 90)
 			(effects
 				(font
@@
 		)
 		(property "Footprint" "TestPoint:TestPoint_Keystone_5000-5004_Miniature"
-			(at 193.04 76.2 0)
+			(at 193.04 71.12 0)
 			(effects
 				(font
@@
 		)
 		(property "Datasheet" "~"
-			(at 193.04 76.2 0)
+			(at 193.04 71.12 0)
 			(effects
 				(font
@@
 		)
 		(property "Description" "test point"
-			(at 193.04 71.12 0)
+			(at 193.04 66.04 0)
 			(effects
 				(font
@@
 	(symbol
 		(lib_id "power:VCC")
-		(at 190.5 68.58 0)
+		(at 190.5 63.5 0)
 		(unit 1)
 		(exclude_from_sim no)
@@
 		(dnp no)
 		(property "Reference" "#PWR079"
-			(at 190.5 72.39 0)
+			(at 190.5 67.31 0)
 			(effects
 				(font
@@
 		)
 		(property "Value" "+9V"
-			(at 190.5 64.77 0)
+			(at 190.5 59.69 0)
 			(effects
 				(font
@@
 		)
 		(property "Footprint" ""
-			(at 190.5 68.58 0)
+			(at 190.5 63.5 0)
 			(effects
 				(font
@@
 		)
 		(property "Datasheet" ""
-			(at 190.5 68.58 0)
+			(at 190.5 63.5 0)
 			(effects
 				(font
@@
 		)
 		(property "Description" "Power symbol creates a global label with name \"VCC\""
-			(at 190.5 68.58 0)
+			(at 190.5 63.5 0)
 			(effects
 				(font

Commit message: Trying to solve all errors on DRC, but some depend on finishing other tasks.
Parts:
- renumbered C35 to C1, C36 to C15, C34 to C5, C31 to C6, C37 to C7, C12 to C8, C38 to C9, D6 to D1, D3 to D2, D8 to D3, D7 to D4, D4 to D6, D9 to D7, D5 to D9, J5 to J2, L3 to L1, L4 to L2, R46 to R1, R44 to R10, R43 to R2, R49 to R24, R45 to R28, R42 to R3, R48 to R8, R47 to R9, TP9 to TP1, TP2 to TP10, TP6 to TP2, TP7 to TP3, TP1 to TP4, TP3 to TP5, TP10 to TP6, TP4 to TP7, TP5 to TP8, TP8 to TP9, U7 to U1, U4 to U2, U8 to U3

Commit message: Changed tactile switch model; had to enlarge board and adjust positioning of components; added some 3D models and comments with PNs for further reference; general layout and routing improvements.
Parts:
- added TP13: GND, TestPoint:TestPoint_Keystone_5000-5004_Miniature, symbol Connector:TestPoint
Connections:
- net GND: now also TP13.1
Other:
- note added: "WE 694106301002 chrome-extension://efaidnbmnnnibpcajpcglclefindmkaj/https://www.we-online.com/components/products/datasheet/694106301002.pdf https://www.we-online.com/en/components/products/DC_RIGHT_ANGLED_6_4_69410X301002 CONFIRM ID 2mm OR 2.5mm"
- note added: "WE 79527141 https://www.we-online.com/en/components/products/BCPH_BATTERY_HOLDER"
- moved on the sheet: R8
Changed lines of the file:
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@@
 	)
 	(junction
+		(at 241.3 139.7)
+		(diameter 0)
+		(color 0 0 0 0)
+	)
+	(junction
 		(at 203.2 134.62)
 		(diameter 0)
@@
 	(wire
 		(pts
-			(xy 228.6 144.78) (xy 228.6 147.32)
+			(xy 228.6 143.51) (xy 228.6 147.32)
 		)
 		(stroke
@@
 	(wire
 		(pts
+			(xy 241.3 139.7) (xy 243.84 139.7)
+		)
+		(stroke
+			(width 0)
+			(type default)
+		)
+	)
+	(wire
+		(pts
 			(xy 38.1 109.22) (xy 38.1 111.76)
 		)
@@
 	(wire
 		(pts
-			(xy 228.6 132.08) (xy 228.6 137.16)
+			(xy 228.6 132.08) (xy 228.6 135.89)
 		)
 		(stroke
@@
 	(wire
 		(pts
+			(xy 241.3 139.7) (xy 241.3 144.78)
+		)
+		(stroke
+			(width 0)
+			(type default)
+		)
+	)
+	(wire
+		(pts
 			(xy 129.54 81.28) (xy 127 81.28)
 		)
@@
 	(wire
 		(pts
-			(xy 241.3 134.62) (xy 241.3 144.78)
+			(xy 241.3 134.62) (xy 241.3 139.7)
 		)
 		(stroke
@@
 		)
 	)
+	(text "WE 694106301002\nchrome-extension://efaidnbmnnnibpcajpcglclefindmkaj/https://www.we-online.com/components/products/datasheet/694106301002.pdf\nhttps://www.we-online.com/en/components/products/DC_RIGHT_ANGLED_6_4_69410X301002\n\nCONFIRM ID 2mm OR 2.5mm"
+		(exclude_from_sim no)
+		(at 33.02 86.36 0)
+		(effects
+			(font
+				(size 1.27 1.27)
+			)
+			(justify right)
+		)
+	)
 	(text "VOUT = 1.25 * (R42/R43)\nhttps://jansson.us/resistors.html"
 		(exclude_from_sim no)
@@
 		)
 	)
+	(text "WE 	79527141\nhttps://www.we-online.com/en/components/products/BCPH_BATTERY_HOLDER"
+		(exclude_from_sim no)
+		(at 41.91 146.05 0)
+		(effects
+			(font
+				(size 1.27 1.27)
+			)
+			(justify left)
+		)
+	)
 	(label "BOOST SW"
 		(at 146.05 73.66 0)
@@
 	(symbol
 		(lib_id "Device:R_US")
-		(at 228.6 140.97 180)
+		(at 228.6 139.7 180)
 		(unit 1)
 		(exclude_from_sim no)
@@
 		(dnp no)
 		(property "Reference" "R8"
-			(at 226.06 140.97 90)
+			(at 226.06 139.7 90)
 			(effects
 				(font
@@
 		)
 		(property "Value" "1K 1%"
-			(at 231.14 140.97 90)
+			(at 231.14 139.7 90)
 			(effects
 				(font
@@
 		)
 		(property "Footprint" "Resistor_SMD:R_0603_1608Metric_Pad0.98x0.95mm_HandSolder"
-			(at 227.584 140.716 90)
+			(at 227.584 139.446 90)
 			(effects
 				(font
@@
 		)
 		(property "Datasheet" "~"
-			(at 228.6 140.97 0)
+			(at 228.6 139.7 0)
 			(effects
 				(font
@@
 		)
 		(property "Description" "Resistor, US symbol"
-			(at 228.6 140.97 0)
+			(at 228.6 139.7 0)
 			(effects
 				(font
@@
 					(unit 1)
 				)
+			)
+		)
+	)
+	(symbol
+		(lib_id "Connector:TestPoint")
+		(at 243.84 139.7 270)
+		(unit 1)
+		(exclude_from_sim no)
+		(in_bom yes)
+		(on_board yes)
+		(dnp no)
+		(fields_autoplaced yes)
+		(property "Reference" "TP13"
+			(at 248.92 138.4299 90)
+			(effects
+				(font
+					(size 1.27 1.27)
+				)
+				(justify left)
+			)
+		)
+		(property "Value" "GND"
+			(at 248.92 140.9699 90)
+			(effects
+				(font
+					(size 1.27 1.27)
+				)
+				(justify left)
+			)
+		)
+		(property "Footprint" "TestPoint:TestPoint_Keystone_5000-5004_Miniature"
+			(at 243.84 144.78 0)
+			(effects
+				(font
+					(size 1.27 1.27)
+				)
+				(hide yes)
+			)
+		)
+		(property "Datasheet" "~"
+			(at 243.84 144.78 0)
+			(effects
+				(font
+					(size 1.27 1.27)
+				)
+				(hide yes)
+			)
+		)
+		(property "Description" "test point"
+			(at 243.84 139.7 0)
+			(effects
+				(font
+					(size 1.27 1.27)
+				)
+				(hide yes)
+			)
+		)
+		(pin "1"
+		)
+		(instances
+			(project "STM32XP"
+				(path "/1f1b32b0-2877-4942-afdb-ad5dc4634e8b/c5d90769-1771-42f2-86df-749a2f175e63"
+					(reference "TP13")
+					(unit 1)
+				)

Commit message: More improvements. Added 3D models. Added legends.
Parts:
- BT1: footprint Battery:BatteryHolder_Multicomp_BC-2001_1x2032 -> Battery:BatteryHolder_Keystone_1060_1x2032
Changed lines of the file:
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@@
 			)
 		)
-		(property "Footprint" "Battery:BatteryHolder_Multicomp_BC-2001_1x2032"
+		(property "Footprint" "Battery:BatteryHolder_Keystone_1060_1x2032"
 			(at 38.1 139.446 90)
 			(effects

Commit message: Finished PCB design, but needs to be reviewed. Added all components and PNs that were missing or incorrect. Added draft of STM32 EXPLORER logo.
Parts:
- removed TP9: +VBUS, TestPoint:TestPoint_Keystone_5000-5004_Miniature, symbol Connector:TestPoint
- FB1: renamed from L2; value L_Small -> 600R; Manufacturer (none) -> Würth Elektronik; PN (none) -> 742792651
- J2: MANUFACTURER (none) -> Würth Elektronik; PN (none) -> 694106301002
- renumbered C9 to C10, C15 to C13, C1 to C2, C5 to C4, C6 to C7, C7 to C8, C8 to C9, D9 to D7, D7 to D8, R9 to R10, R10 to R13, R28 to R21, R24 to R22, R8 to R9, TP6 to TP1, TP11 to TP12, TP3 to TP2, TP4 to TP3, TP1 to TP4, TP7 to TP6, TP8 to TP7, TP2 to TP9
Connections:
- net +VBUS renamed +VBUSF
Other:
- note removed: "WE 694106301002 chrome-extension://efaidnbmnnnibpcajpcglclefindmkaj/https://www.we-online.com/components/products/datasheet/694106301002.pdf https://www.we-online.com/en/components/products/DC_RIGHT_ANGLED_6_4_69410X301002 CONFIRM ID 2mm OR 2.5mm"

Commit message: Finished Revision 0 design. Used plugin to make manufacturing files. Purchased 5 units in JLCPCB. Let's wait to check the results! :D
Parts:
- renumbered TP10 to TP11, TP12 to TP13, TP13 to TP14
Connections:
- net +3.3V LED: now reaches D4.1 (K), R10.2
- net +9V LED: now reaches D1.1 (K), R1.2
- net +VEXT LED: now reaches D8.1 (K), R22.2
- net +VBUSF LED: now reaches D7.1 (K), R21.2
- net +5V LED: now reaches D3.1 (K), R9.2
- no-connect marks 0 -> 1
Other:
- title: STM32 EXPLORER BOARD -> STM32 EXPLORER BOARD PROTOTYPE
Changed lines of the file:
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@@
 	(paper "A4")
 	(title_block
-		(title "STM32 EXPLORER BOARD")
-		(date "2024-04-26")
+		(title "STM32 EXPLORER BOARD PROTOTYPE")
+		(date "2024-07-21")
 		(rev "00")
 		(company "Mechatronix Lab")
@@
 		(color 0 0 0 0)
 	)
+	(no_connect
+		(at 35.56 101.6)
+	)
 	(wire
 		(pts
@@
 	(wire
 		(pts
-			(xy 38.1 143.51) (xy 38.1 149.86)
+			(xy 38.1 143.51) (xy 38.1 147.32)
 		)
 		(stroke
@@
 		)
 	)
+	(label "+9V LED"
+		(at 190.5 86.36 180)
+		(fields_autoplaced yes)
+		(effects
+			(font
+				(size 0.635 0.635)
+			)
+			(justify right bottom)
+		)
+	)
 	(label "BOOST SW"
 		(at 146.05 73.66 0)
@@
 		)
 	)
+	(label "+VBUSF LED"
+		(at 88.9 48.26 180)
+		(fields_autoplaced yes)
+		(effects
+			(font
+				(size 0.635 0.635)
+			)
+			(justify right bottom)
+		)
+	)
+	(label "+5V LED"
+		(at 228.6 134.62 180)
+		(fields_autoplaced yes)
+		(effects
+			(font
+				(size 0.635 0.635)
+			)
+			(justify right bottom)
+		)
+	)
+	(label "+3.3V LED"
+		(at 139.7 134.62 180)
+		(fields_autoplaced yes)
+		(effects
+			(font
+				(size 0.635 0.635)
+			)
+			(justify right bottom)
+		)
+	)
+	(label "+VEXT LED"
+		(at 63.5 48.26 180)
+		(fields_autoplaced yes)
+		(effects
+			(font
+				(size 0.635 0.635)
+			)
+			(justify right bottom)
+		)
+	)
 	(label "BOOST FB"
 		(at 151.13 86.36 0)
@@
 		(dnp no)
 		(fields_autoplaced yes)
-		(property "Reference" "TP12"
+		(property "Reference" "TP13"
 			(at 248.92 143.5099 90)
 			(effects
@@
 			(project "STM32XP"
 				(path "/1f1b32b0-2877-4942-afdb-ad5dc4634e8b/c5d90769-1771-42f2-86df-749a2f175e63"
-					(reference "TP12")
+					(reference "TP13")
 					(unit 1)
 				)
@@
 		(dnp no)
 		(fields_autoplaced yes)
-		(property "Reference" "TP10"
+		(property "Reference" "TP11"
 			(at 248.92 118.1099 90)
 			(effects
@@
 			(project "STM32XP"
 				(path "/1f1b32b0-2877-4942-afdb-ad5dc4634e8b/c5d90769-1771-42f2-86df-749a2f175e63"
-					(reference "TP10")
+					(reference "TP11")
 					(unit 1)
 				)
@@
 	(symbol
 		(lib_id "power:GND")
-		(at 38.1 149.86 0)
+		(at 38.1 147.32 0)
 		(unit 1)
 		(exclude_from_sim no)
@@
 		(fields_autoplaced yes)
 		(property "Reference" "#PWR023"
-			(at 38.1 156.21 0)
+			(at 38.1 153.67 0)
 			(effects
 				(font
@@
 		)
 		(property "Value" "GND"
-			(at 38.1 154.94 0)
+			(at 38.1 152.4 0)
 			(effects
 				(font
@@
 		)
 		(property "Footprint" ""
-			(at 38.1 149.86 0)
+			(at 38.1 147.32 0)
 			(effects
 				(font
@@
 		)
 		(property "Datasheet" ""
-			(at 38.1 149.86 0)
+			(at 38.1 147.32 0)
 			(effects
 				(font
@@
 		)
 		(property "Description" "Power symbol creates a global label with name \"GND\" , ground"
-			(at 38.1 149.86 0)
+			(at 38.1 147.32 0)
 			(effects
 				(font
@@
 		(dnp no)
 		(property "Reference" "D6"
-			(at 76.2 33.02 0)
+			(at 76.2 30.48 0)
 			(effects
 				(font
@@
 		)
 		(property "Value" "BAT54C"
-			(at 81.28 38.1 0)
+			(at 76.2 33.02 0)
 			(effects
 				(font
@@
 		(dnp no)
 		(fields_autoplaced yes)
-		(property "Reference" "TP13"
+		(property "Reference" "TP14"
 			(at 248.92 138.4299 90)
 			(effects
@@
 			(project "STM32XP"
 				(path "/1f1b32b0-2877-4942-afdb-ad5dc4634e8b/c5d90769-1771-42f2-86df-749a2f175e63"
-					(reference "TP13")
+					(reference "TP14")
 					(unit 1)
 				)
