File: HARDWARE/KICAD/POWER.kicad_sch (KiCad schematic)
At the start: 42 parts, among them J2 Jack-DC, U1 AMS1117-5.0, U2 AMS1117-3.3, U3 AP3012

Commit message: Added comments about minor adjustments needed after board assembly.
Other:
- note added: "2024.08.09: R2 = 3.6K // 3.6K R3 = 10K VOUT = 1.25 * (1 + R3/R2) = 8.2V"
Changed lines of the file:
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@@
+		)
+	)
+	(text "2024.08.09:\nR2 = 3.6K // 3.6K\nR3 = 10K\nVOUT = 1.25 * (1 + R3/R2) = 8.2V"
+		(exclude_from_sim no)
+		(at 139.7 63.5 0)
+		(effects
+			(font
+				(size 1.27 1.27)
+				(thickness 0.254)
+				(bold yes)
+				(italic yes)
+				(color 194 0 0 1)
+			)
+			(justify left)
 		)
 	)
