File: HARDWARE/KICAD/INTERFACE.kicad_sch (KiCad schematic)
At the start: 22 parts, among them Q1 MMBT3904, SW1 SW_Push, SW2 SW_Push, SW4 SW_Push, SW5 SW_Push, SW6 SW_Push, SW7 SW_Push, SW8 SW_Push, U6 OLED 128x64 1.3"

Commit message: Continuing layout and routing.
Connections:
- net +3.3V: now also U6.1 (VCC); no longer U6.2 (VCC)
- net GND: now also U6.2 (GND); no longer U6.1 (GND)
Other:
- company: (none) -> Mechatronix Lab
- title: (none) -> STM32 EXPLORER BOARD
- moved on the sheet: C15, C32
Changed lines of the file:
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@@
 	(generator_version "8.0")
 	(paper "A4")
+	(title_block
+		(title "STM32 EXPLORER BOARD")
+		(date "2024-04-26")
+		(rev "00")
+		(company "Mechatronix Lab")
+		(comment 1 "Eng. André A. M. Araújo")
+	)
 	(junction
 		(at 50.8 58.42)
@@
 	)
 	(junction
-		(at 127 102.87)
+		(at 124.46 97.79)
+		(diameter 0)
+		(color 0 0 0 0)
+	)
+	(junction
+		(at 137.16 97.79)
 		(diameter 0)
 		(color 0 0 0 0)
@@
 	)
 	(junction
-		(at 139.7 102.87)
-		(diameter 0)
-		(color 0 0 0 0)
-	)
-	(junction
-		(at 139.7 93.98)
+		(at 137.16 88.9)
 		(diameter 0)
 		(color 0 0 0 0)
@@
 	)
 	(junction
-		(at 127 107.95)
-		(diameter 0)
-		(color 0 0 0 0)
-	)
-	(junction
 		(at 76.2 58.42)
 		(diameter 0)
@@
 	(wire
 		(pts
-			(xy 139.7 91.44) (xy 139.7 93.98)
+			(xy 137.16 86.36) (xy 137.16 88.9)
 		)
 		(stroke
@@
 	(wire
 		(pts
+			(xy 139.7 97.79) (xy 139.7 110.49)
+		)
+		(stroke
+			(width 0)
+			(type default)
+		)
+	)
+	(wire
+		(pts
 			(xy 127 55.88) (xy 127 58.42)
 		)
@@
 	(wire
 		(pts
-			(xy 130.81 93.98) (xy 127 93.98)
-		)
-		(stroke
-			(width 0)
-			(type default)
-		)
-	)
-	(wire
-		(pts
-			(xy 127 102.87) (xy 130.81 102.87)
+			(xy 128.27 88.9) (xy 124.46 88.9)
+		)
+		(stroke
+			(width 0)
+			(type default)
+		)
+	)
+	(wire
+		(pts
+			(xy 124.46 97.79) (xy 128.27 97.79)
+		)
+		(stroke
+			(width 0)
+			(type default)
+		)
+	)
+	(wire
+		(pts
+			(xy 142.24 97.79) (xy 142.24 100.33)
 		)
 		(stroke
@@
 	(wire
 		(pts
+			(xy 137.16 97.79) (xy 137.16 110.49)
+		)
+		(stroke
+			(width 0)
+			(type default)
+		)
+	)
+	(wire
+		(pts
 			(xy 227.33 99.06) (xy 227.33 101.6)
 		)
@@
 	(wire
 		(pts
-			(xy 139.7 93.98) (xy 139.7 102.87)
+			(xy 137.16 88.9) (xy 137.16 97.79)
 		)
 		(stroke
@@
 	(wire
 		(pts
-			(xy 135.89 93.98) (xy 139.7 93.98)
+			(xy 133.35 88.9) (xy 137.16 88.9)
 		)
 		(stroke
@@
 	(wire
 		(pts
-			(xy 127 107.95) (xy 137.16 107.95)
-		)
-		(stroke
-			(width 0)
-			(type default)
-		)
-	)
-	(wire
-		(pts
 			(xy 101.6 58.42) (xy 101.6 60.96)
 		)
@@
 	(wire
 		(pts
-			(xy 137.16 107.95) (xy 137.16 110.49)
+			(xy 139.7 97.79) (xy 142.24 97.79)
 		)
 		(stroke
@@
 	(wire
 		(pts
-			(xy 127 93.98) (xy 127 102.87)
-		)
-		(stroke
-			(width 0)
-			(type default)
-		)
-	)
-	(wire
-		(pts
 			(xy 142.24 105.41) (xy 142.24 110.49)
 		)
@@
 	(wire
 		(pts
+			(xy 124.46 97.79) (xy 124.46 100.33)
+		)
+		(stroke
+			(width 0)
+			(type default)
+		)
+	)
+	(wire
+		(pts
 			(xy 229.87 96.52) (xy 229.87 99.06)
 		)
@@
 	(wire
 		(pts
-			(xy 139.7 102.87) (xy 139.7 110.49)
-		)
-		(stroke
-			(width 0)
-			(type default)
-		)
-	)
-	(wire
-		(pts
 			(xy 50.8 40.64) (xy 50.8 48.26)
 		)
@@
 	(wire
 		(pts
-			(xy 127 107.95) (xy 127 110.49)
-		)
-		(stroke
-			(width 0)
-			(type default)
-		)
-	)
-	(wire
-		(pts
 			(xy 227.33 111.76) (xy 229.87 111.76)
 		)
@@
 	(wire
 		(pts
-			(xy 135.89 102.87) (xy 139.7 102.87)
+			(xy 133.35 97.79) (xy 137.16 97.79)
 		)
 		(stroke
@@
 	(wire
 		(pts
-			(xy 127 102.87) (xy 127 107.95)
+			(xy 124.46 88.9) (xy 124.46 97.79)
 		)
 		(stroke
@@
 				(path "/1f1b32b0-2877-4942-afdb-ad5dc4634e8b/f228163b-b634-4755-ba71-ac87e0adbab4"
 					(reference "R15")
+					(unit 1)
+				)
+			)
+		)
+	)
+	(symbol
+		(lib_id "power:GND")
+		(at 142.24 100.33 0)
+		(unit 1)
+		(exclude_from_sim no)
+		(in_bom yes)
+		(on_board yes)
+		(dnp no)
+		(fields_autoplaced yes)
+		(property "Reference" "#PWR084"
+			(at 142.24 106.68 0)
+			(effects
+				(font
+					(size 1.27 1.27)
+				)
+				(hide yes)
+			)
+		)
+		(property "Value" "GND"
+			(at 142.24 105.41 0)
+			(effects
+				(font
+					(size 1.27 1.27)
+				)
+				(hide yes)
+			)
+		)
+		(property "Footprint" ""
+			(at 142.24 100.33 0)
+			(effects
+				(font
+					(size 1.27 1.27)
+				)
+				(hide yes)
+			)
+		)
+		(property "Datasheet" ""
+			(at 142.24 100.33 0)
+			(effects
+				(font
+					(size 1.27 1.27)
+				)
+				(hide yes)
+			)
+		)
+		(property "Description" "Power symbol creates a global label with name \"GND\" , ground"
+			(at 142.24 100.33 0)
+			(effects
+				(font
+					(size 1.27 1.27)
+				)
+				(hide yes)
+			)
+		)
+		(pin "1"
+		)
+		(instances
+			(project "STM32XP"
+				(path "/1f1b32b0-2877-4942-afdb-ad5dc4634e8b/f228163b-b634-4755-ba71-ac87e0adbab4"
+					(reference "#PWR084")
 					(unit 1)
 				)
@@
 	(symbol
 		(lib_id "Device:C_Small")
-		(at 133.35 102.87 90)
+		(at 130.81 97.79 90)
 		(unit 1)
 		(exclude_from_sim no)
@@
 		(dnp no)
 		(property "Reference" "C32"
-			(at 132.08 100.33 90)
+			(at 129.54 95.25 90)
 			(effects
 				(font
@@
 		)
 		(property "Value" "100nF 50V"
-			(at 128.27 105.41 90)
+			(at 125.73 100.33 90)
 			(effects
 				(font
@@
 		)
 		(property "Footprint" "Capacitor_SMD:C_0603_1608Metric_Pad1.08x0.95mm_HandSolder"
-			(at 133.35 102.87 0)
+			(at 130.81 97.79 0)
 			(effects
 				(font
@@
 		)
 		(property "Datasheet" "~"
-			(at 133.35 102.87 0)
+			(at 130.81 97.79 0)
 			(effects
 				(font
@@
 		)
 		(property "Description" "Unpolarized capacitor, small symbol"
-			(at 133.35 102.87 0)
+			(at 130.81 97.79 0)
 			(effects
 				(font
@@
 	(symbol
 		(lib_id "Device:C_Small")
-		(at 133.35 93.98 90)
+		(at 130.81 88.9 90)
 		(unit 1)
 		(exclude_from_sim no)
@@
 		(dnp no)
 		(property "Reference" "C15"
-			(at 132.08 91.44 90)
+			(at 129.54 86.36 90)
 			(effects
 				(font
@@
 		)
 		(property "Value" "10uF 25V"
-			(at 128.27 96.52 90)
+			(at 125.73 91.44 90)
 			(effects
 				(font
@@
 		)
 		(property "Footprint" "Capacitor_SMD:C_0805_2012Metric_Pad1.18x1.45mm_HandSolder"
-			(at 133.35 93.98 0)
+			(at 130.81 88.9 0)
 			(effects
 				(font
@@
 		)
 		(property "Datasheet" "~"
-			(at 133.35 93.98 0)
+			(at 130.81 88.9 0)
 			(effects
 				(font
@@
 		)
 		(property "Description" "Unpolarized capacitor, small symbol"
-			(at 133.35 93.98 0)
+			(at 130.81 88.9 0)
 			(effects
 				(font
@@
 	(symbol
 		(lib_id "power:GND")
-		(at 127 110.49 0)
+		(at 124.46 100.33 0)
 		(unit 1)
 		(exclude_from_sim no)
@@
 		(fields_autoplaced yes)
 		(property "Reference" "#PWR026"
-			(at 127 116.84 0)
+			(at 124.46 106.68 0)
 			(effects
 				(font
@@
 		)
 		(property "Value" "GND"
-			(at 127 115.57 0)
+			(at 124.46 105.41 0)
 			(effects
 				(font
@@
 		)
 		(property "Footprint" ""
-			(at 127 110.49 0)
+			(at 124.46 100.33 0)
 			(effects
 				(font
@@
 		)
 		(property "Datasheet" ""
-			(at 127 110.49 0)
+			(at 124.46 100.33 0)
 			(effects
 				(font
@@
 		)
 		(property "Description" "Power symbol creates a global label with name \"GND\" , ground"
-			(at 127 110.49 0)
+			(at 124.46 100.33 0)
 			(effects
 				(font
@@
 	(symbol
 		(lib_id "power:VCC")
-		(at 139.7 91.44 0)
+		(at 137.16 86.36 0)
 		(unit 1)
 		(exclude_from_sim no)
@@
 		(dnp no)
 		(property "Reference" "#PWR028"
-			(at 139.7 95.25 0)
+			(at 137.16 90.17 0)
 			(effects
 				(font
@@
 		)
 		(property "Value" "+3.3V"
-			(at 139.7 87.63 0)
+			(at 137.16 82.55 0)
 			(effects
 				(font
@@
 		)
 		(property "Footprint" ""
-			(at 139.7 91.44 0)
+			(at 137.16 86.36 0)
 			(effects
 				(font
@@
 		)
 		(property "Datasheet" ""
-			(at 139.7 91.44 0)
+			(at 137.16 86.36 0)
 			(effects
 				(font
@@
 		)
 		(property "Description" "Power symbol creates a global label with name \"VCC\""
-			(at 139.7 91.44 0)
-			(effects
-				(font
+			(at 137.16 86.36 0)
+			(effects
+				(font

Commit message: Trying to solve all errors on DRC, but some depend on finishing other tasks.
Parts:
- removed Q1: MMBT3904, Package_TO_SOT_SMD:SOT-23, symbol Transistor_BJT:MMBT3904
- added Q3: 2N7002, Package_TO_SOT_SMD:SOT-23, symbol Transistor_FET:2N7002
- renumbered C33 to C2, C15 to C3, C32 to C4, D1 to D5, R39 to R26, R34 to R41, R36 to R44, R38 to R45, R37 to R46, R14 to R47, R15 to R48, R35 to R49, SW4 to SW2, SW6 to SW3, SW8 to SW4, SW7 to SW5, SW1 to SW6, SW2 to SW7, SW5 to SW8, U6 to U4
Connections:
- net GND: now also Q3.2 (S)
- net PWM BUZZER: now also Q3.1 (G)
- net at LS1.2, R26.1: now also Q3.3 (D)
Changed lines of the file:
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@@
 		(on_board yes)
 		(dnp no)
-		(property "Reference" "R15"
+		(property "Reference" "R48"
 			(at 240.03 55.88 90)
 			(effects
@@
 			(project "STM32XP"
 				(path "/1f1b32b0-2877-4942-afdb-ad5dc4634e8b/f228163b-b634-4755-ba71-ac87e0adbab4"
-					(reference "R15")
+					(reference "R48")
 					(unit 1)
 				)
@@
 		(dnp no)
 		(fields_autoplaced yes)
-		(property "Reference" "SW4"
+		(property "Reference" "SW2"
 			(at 52.07 64.7699 90)
 			(effects
@@
 			(project "STM32XP"
 				(path "/1f1b32b0-2877-4942-afdb-ad5dc4634e8b/f228163b-b634-4755-ba71-ac87e0adbab4"
-					(reference "SW4")
+					(reference "SW2")
 					(unit 1)
 				)
@@
 		(on_board yes)
 		(dnp no)
-		(property "Reference" "D1"
+		(property "Reference" "D5"
 			(at 81.28 110.49 0)
 			(effects
@@
 			(project "STM32XP"
 				(path "/1f1b32b0-2877-4942-afdb-ad5dc4634e8b/f228163b-b634-4755-ba71-ac87e0adbab4"
-					(reference "D1")
+					(reference "D5")
 					(unit 1)
 				)
@@
 		(on_board yes)
 		(dnp no)
-		(property "Reference" "R36"
+		(property "Reference" "R44"
 			(at 100.33 55.88 90)
 			(effects
@@
 			(project "STM32XP"
 				(path "/1f1b32b0-2877-4942-afdb-ad5dc4634e8b/f228163b-b634-4755-ba71-ac87e0adbab4"
-					(reference "R36")
+					(reference "R44")
 					(unit 1)
 				)
@@
 		(on_board yes)
 		(dnp no)
-		(property "Reference" "C33"
+		(property "Reference" "C2"
 			(at 69.85 106.68 90)
 			(effects
@@
 			(project "STM32XP"
 				(path "/1f1b32b0-2877-4942-afdb-ad5dc4634e8b/f228163b-b634-4755-ba71-ac87e0adbab4"
-					(reference "C33")
+					(reference "C2")
 					(unit 1)
 				)
@@
 		(on_board yes)
 		(dnp no)
-		(property "Reference" "C32"
+		(property "Reference" "C4"
 			(at 129.54 95.25 90)
 			(effects
@@
 			(project "STM32XP"
 				(path "/1f1b32b0-2877-4942-afdb-ad5dc4634e8b/f228163b-b634-4755-ba71-ac87e0adbab4"
-					(reference "C32")
+					(reference "C4")
 					(unit 1)
 				)
@@
 	)
 	(symbol
+		(lib_id "Transistor_FET:2N7002")
+		(at 227.33 119.38 0)
+		(unit 1)
+		(exclude_from_sim no)
+		(in_bom yes)
+		(on_board yes)
+		(dnp no)
+		(property "Reference" "Q3"
+			(at 233.68 118.11 0)
+			(effects
+				(font
+					(size 1.27 1.27)
+				)
+			)
+		)
+		(property "Value" "2N7002"
+			(at 236.22 120.65 0)
+			(effects
+				(font
+					(size 1.27 1.27)
+				)
+			)
+		)
+		(property "Footprint" "Package_TO_SOT_SMD:SOT-23"
+			(at 232.41 121.285 0)
+			(effects
+				(font
+					(size 1.27 1.27)
+					(italic yes)
+				)
+				(justify left)
+				(hide yes)
+			)
+		)
+		(property "Datasheet" "https://www.onsemi.com/pub/Collateral/NDS7002A-D.PDF"
+			(at 232.41 123.19 0)
+			(effects
+				(font
+					(size 1.27 1.27)
+				)
+				(justify left)
+				(hide yes)
+			)
+		)
+		(property "Description" "0.115A Id, 60V Vds, N-Channel MOSFET, SOT-23"
+			(at 227.33 119.38 0)
+			(effects
+				(font
+					(size 1.27 1.27)
+				)
+				(hide yes)
+			)
+		)
+		(pin "1"
+		)
+		(pin "2"
+		)
+		(pin "3"
+		)
+		(instances
+			(project "STM32XP"
+				(path "/1f1b32b0-2877-4942-afdb-ad5dc4634e8b/f228163b-b634-4755-ba71-ac87e0adbab4"
+					(reference "Q3")
+					(unit 1)
+				)
+			)
+		)
+	)
+	(symbol
 		(lib_id "power:GND")
 		(at 152.4 73.66 0)
@@
 		(on_board yes)
 		(dnp no)
-		(property "Reference" "C15"
+		(property "Reference" "C3"
 			(at 129.54 86.36 90)
 			(effects
@@
 			(project "STM32XP"
 				(path "/1f1b32b0-2877-4942-afdb-ad5dc4634e8b/f228163b-b634-4755-ba71-ac87e0adbab4"
-					(reference "C15")
+					(reference "C3")
 					(unit 1)
 				)
@@
 		(dnp no)
 		(fields_autoplaced yes)
-		(property "Reference" "SW5"
+		(property "Reference" "SW8"
 			(at 77.47 64.7699 90)
 			(effects
@@
 			(project "STM32XP"
 				(path "/1f1b32b0-2877-4942-afdb-ad5dc4634e8b/f228163b-b634-4755-ba71-ac87e0adbab4"
-					(reference "SW5")
+					(reference "SW8")
 					(unit 1)
 				)
@@
 		(on_board yes)
 		(dnp no)
-		(property "Reference" "R38"
+		(property "Reference" "R45"
 			(at 151.13 55.88 90)
 			(effects
@@
 			(project "STM32XP"
 				(path "/1f1b32b0-2877-4942-afdb-ad5dc4634e8b/f228163b-b634-4755-ba71-ac87e0adbab4"
-					(reference "R38")
+					(reference "R45")
 					(unit 1)
 				)
@@
 		(dnp no)
 		(fields_autoplaced yes)
-		(property "Reference" "SW2"
+		(property "Reference" "SW7"
 			(at 242.57 64.7699 90)
 			(effects
@@
 			(project "STM32XP"
 				(path "/1f1b32b0-2877-4942-afdb-ad5dc4634e8b/f228163b-b634-4755-ba71-ac87e0adbab4"
-					(reference "SW2")
+					(reference "SW7")
 					(unit 1)
 				)
@@
 		(on_board yes)
 		(dnp no)
-		(property "Reference" "R39"
+		(property "Reference" "R26"
 			(at 224.79 105.41 90)
 			(effects
@@
 			(project "STM32XP"
 				(path "/1f1b32b0-2877-4942-afdb-ad5dc4634e8b/f228163b-b634-4755-ba71-ac87e0adbab4"
-					(reference "R39")
+					(reference "R26")
 					(unit 1)
 				)
@@
 		(on_board yes)
 		(dnp no)
-		(property "Reference" "R35"
+		(property "Reference" "R49"
 			(at 74.93 55.88 90)
 			(effects
@@
 			(project "STM32XP"
 				(path "/1f1b32b0-2877-4942-afdb-ad5dc4634e8b/f228163b-b634-4755-ba71-ac87e0adbab4"
-					(reference "R35")
+					(reference "R49")
 					(unit 1)
 				)
@@
 		(dnp no)
 		(fields_autoplaced yes)
-		(property "Reference" "U6"
+		(property "Reference" "U4"
 			(at 152.4 119.3799 0)
 			(effects
@@
 			(project "STM32XP"
 				(path "/1f1b32b0-2877-4942-afdb-ad5dc4634e8b/f228163b-b634-4755-ba71-ac87e0adbab4"
-					(reference "U6")
+					(reference "U4")
 					(unit 1)
 				)
@@
 	)
 	(symbol
-		(lib_id "Transistor_BJT:MMBT3904")
-		(at 227.33 119.38 0)
-		(unit 1)
-		(exclude_from_sim no)
-		(in_bom yes)
-		(on_board yes)
-		(dnp no)
-		(fields_autoplaced yes)
-		(property "Reference" "Q1"
-			(at 232.41 118.1099 0)
-			(effects
-				(font
-					(size 1.27 1.27)
-				)
-				(justify left)
-			)
-		)
-		(property "Value" "MMBT3904"
-			(at 232.41 120.6499 0)
-			(effects
-				(font
-					(size 1.27 1.27)
-				)
-				(justify left)
-			)
-		)
-		(property "Footprint" "Package_TO_SOT_SMD:SOT-23"
-			(at 232.41 121.285 0)
-			(effects
-				(font
-					(size 1.27 1.27)
-					(italic yes)
-				)
-				(justify left)
-				(hide yes)
-			)
-		)
-		(property "Datasheet" "https://www.onsemi.com/pdf/datasheet/pzt3904-d.pdf"
-			(at 227.33 119.38 0)
-			(effects
-				(font
-					(size 1.27 1.27)
-				)
-				(justify left)
-				(hide yes)
-			)
-		)
-		(property "Description" "0.2A Ic, 40V Vce, Small Signal NPN Transistor, SOT-23"
-			(at 227.33 119.38 0)
-			(effects
-				(font
-					(size 1.27 1.27)
-				)
-				(hide yes)
-			)
-		)
-		(pin "1"
-		)
-		(pin "3"
-		)
-		(pin "2"
-		)
-		(instances
-			(project "STM32XP"
-				(path "/1f1b32b0-2877-4942-afdb-ad5dc4634e8b/f228163b-b634-4755-ba71-ac87e0adbab4"
-					(reference "Q1")
-					(unit 1)
-				)
-			)
-		)
-	)
-	(symbol
 		(lib_id "power:VCC")
 		(at 101.6 40.64 0)
@@
 		(dnp no)
 		(fields_autoplaced yes)
-		(property "Reference" "SW1"
+		(property "Reference" "SW6"
 			(at 217.17 64.7699 90)
 			(effects
@@
 			(project "STM32XP"
 				(path "/1f1b32b0-2877-4942-afdb-ad5dc4634e8b/f228163b-b634-4755-ba71-ac87e0adbab4"
-					(reference "SW1")
+					(reference "SW6")
 					(unit 1)
 				)
@@
 		(on_board yes)
 		(dnp no)
-		(property "Reference" "R14"
+		(property "Reference" "R47"
 			(at 214.63 55.88 90)
 			(effects
@@
 			(project "STM32XP"
 				(path "/1f1b32b0-2877-4942-afdb-ad5dc4634e8b/f228163b-b634-4755-ba71-ac87e0adbab4"
-					(reference "R14")
+					(reference "R47")
 					(unit 1)
 				)
@@
 		(dnp no)
 		(fields_autoplaced yes)
-		(property "Reference" "SW8"
+		(property "Reference" "SW4"
 			(at 153.67 64.7699 90)
 			(effects
@@
 			(project "STM32XP"
 				(path "/1f1b32b0-2877-4942-afdb-ad5dc4634e8b/f228163b-b634-4755-ba71-ac87e0adbab4"
-					(reference "SW8")
+					(reference "SW4")
 					(unit 1)
 				)
@@
 		(dnp no)
 		(fields_autoplaced yes)
-		(property "Reference" "SW7"
+		(property "Reference" "SW5"
 			(at 128.27 64.7699 90)
 			(effects
@@
 			(project "STM32XP"
 				(path "/1f1b32b0-2877-4942-afdb-ad5dc4634e8b/f228163b-b634-4755-ba71-ac87e0adbab4"
-					(reference "SW7")
+					(reference "SW5")
 					(unit 1)
 				)
@@
 		(on_board yes)
 		(dnp no)
-		(property "Reference" "R34"
+		(property "Reference" "R41"
 			(at 49.53 55.88 90)
 			(effects
@@
 			(project "STM32XP"
 				(path "/1f1b32b0-2877-4942-afdb-ad5dc4634e8b/f228163b-b634-4755-ba71-ac87e0adbab4"
-					(reference "R34")
+					(reference "R41")
 					(unit 1)
 				)
@@
 		(dnp no)
 		(fields_autoplaced yes)
-		(property "Reference" "SW6"
+		(property "Reference" "SW3"
 			(at 102.87 64.7699 90)
 			(effects
@@
 			(project "STM32XP"
 				(path "/1f1b32b0-2877-4942-afdb-ad5dc4634e8b/f228163b-b634-4755-ba71-ac87e0adbab4"
-					(reference "SW6")
+					(reference "SW3")
 					(unit 1)
 				)
@@
 		(on_board yes)
 		(dnp no)
-		(property "Reference" "R37"
+		(property "Reference" "R46"
 			(at 125.73 55.88 90)
 			(effects
@@
 			(project "STM32XP"
 				(path "/1f1b32b0-2877-4942-afdb-ad5dc4634e8b/f228163b-b634-4755-ba71-ac87e0adbab4"
-					(reference "R37")
-					(unit 1)
-				)
+					(reference "R46")
+					(unit 1)
+				)

Commit message: Changed tactile switch model; had to enlarge board and adjust positioning of components; added some 3D models and comments with PNs for further reference; general layout and routing improvements.
Parts:
- SW2: value SW_Push -> UP; footprint Button_Switch_SMD:SW_SPST_CK_KXT3 -> Button_Switch_SMD:SW_Push_1P1T_NO_CK_KSC6xxJ
- SW3: value SW_Push -> LEFT; footprint Button_Switch_SMD:SW_SPST_CK_KXT3 -> Button_Switch_SMD:SW_Push_1P1T_NO_CK_KSC6xxJ
- SW4: value SW_Push -> CENTER; footprint Button_Switch_SMD:SW_SPST_CK_KXT3 -> Button_Switch_SMD:SW_Push_1P1T_NO_CK_KSC6xxJ
- SW5: value SW_Push -> RIGHT; footprint Button_Switch_SMD:SW_SPST_CK_KXT3 -> Button_Switch_SMD:SW_Push_1P1T_NO_CK_KSC6xxJ
- SW6: value SW_Push -> BUTTON 1; footprint Button_Switch_SMD:SW_SPST_CK_KXT3 -> Button_Switch_SMD:SW_Push_1P1T_NO_CK_KSC6xxJ
- SW7: value SW_Push -> BUTTON 2; footprint Button_Switch_SMD:SW_SPST_CK_KXT3 -> Button_Switch_SMD:SW_Push_1P1T_NO_CK_KSC6xxJ
- SW8: value SW_Push -> DOWN; footprint Button_Switch_SMD:SW_SPST_CK_KXT3 -> Button_Switch_SMD:SW_Push_1P1T_NO_CK_KSC6xxJ

Commit message: Finished PCB design, but needs to be reviewed. Added all components and PNs that were missing or incorrect. Added draft of STM32 EXPLORER logo.
Parts:
- removed LS1: Speaker_Crystal, Buzzer_Beeper:MagneticBuzzer_PUI_AT-0927-TT-6-R, symbol Device:Speaker_Crystal
- added C1: 10uF 25V, Capacitor_SMD:C_0805_2012Metric_Pad1.18x1.45mm_HandSolder, symbol Device:C_Small
- added D10: 150505M173300, STM32XP:WE 150505M173300, symbol STM32XP:WE 50505M173300
- added LS1: 78dB 4kHz, STM32XP:PKM13EPYH4000-A0, symbol STM32XP:PKM13EPYH4000-A0
- renumbered C4 to C12, C2 to C3, C3 to C6, Q3 to Q1, R41 to R43, R45 to R44, R44 to R49, R49 to R50, R26 to R8
Connections:
- net GND: now also C1.1, D10.1 (KB), D10.3 (KR), D10.5 (KG)
- net PWM BLUE: now also D10.2 (AB)
- net PWM GREEN: now also D10.6 (AG)
- net PWM RED: now also D10.4 (AR)
- net at Q1.3 (D), R8.1: now also LS1.2
- net +VSEL renamed +9V
- net +9V: now also C1.2, LS1.1
Other:
- moved on the sheet: C12, C3, C6, D5, Q1, R43, R44, R46, R47, R48, R49, R50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

Commit message: Finished Revision 0 design. Used plugin to make manufacturing files. Purchased 5 units in JLCPCB. Let's wait to check the results! :D
Parts:
- renumbered R43 to R46, R44 to R47, R46 to R49, R47 to R50, R48 to R51, R49 to R52, R50 to R53
Connections:
- net BUZZER DRAIN: now reaches LS1.2, Q1.3 (D), R8.1
Other:
- title: STM32 EXPLORER BOARD -> STM32 EXPLORER BOARD PROTOTYPE
- moved on the sheet: C1, C12, C6, D10, LS1, Q1, R8, U4

Commit message: Added comments about minor adjustments needed after board assembly.
Other:
- note added: "2024.08.09: 10K PULL-DOWN RESISTOR ADDED TO GATE, TO PREVENTE NOISE WHEN HANDLING THE BOARD"
Changed lines of the file:
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@@
+		)
+	)
+	(text "2024.08.09:\n10K PULL-DOWN RESISTOR ADDED TO GATE,\nTO PREVENTE NOISE WHEN HANDLING THE BOARD"
+		(exclude_from_sim no)
+		(at 226.06 60.96 0)
+		(effects
+			(font
+				(size 1.27 1.27)
+				(thickness 0.254)
+				(bold yes)
+				(italic yes)
+				(color 194 0 0 1)
+			)
+			(justify right)
 		)
 	)

Commit message: Added updated PDF with comments after corrections in the prototype.
Other:
- note added: "2024.08.09: 10K PULL-DOWN RESISTOR ADDED TO GATE, TO PREVENT NOISE WHEN HANDLING THE BOARD"
- note removed: "2024.08.09: 10K PULL-DOWN RESISTOR ADDED TO GATE, TO PREVENTE NOISE WHEN HANDLING THE BOARD"
Changed lines of the file:
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@@
 		)
 	)
-	(text "2024.08.09:\n10K PULL-DOWN RESISTOR ADDED TO GATE,\nTO PREVENTE NOISE WHEN HANDLING THE BOARD"
+	(text "2024.08.09:\n10K PULL-DOWN RESISTOR ADDED TO GATE,\nTO PREVENT NOISE WHEN HANDLING THE BOARD"
 		(exclude_from_sim no)
 		(at 226.06 60.96 0)
